File: hardware/PowerDistributionUnit_Mk1/Indicators.kicad_sch (KiCad schematic)
At the start: 60 parts, among them J13 Logic Analyzer, SW1 JS202011SCQN, U27 74LVC594APW,118, U28 74LVC594APW,118, U29 74AUP1G04GW-Q100H, U30 NL27WZ17DFT2G-Q

Commit message: update all symbols with LCSC P/N
Parts:
- C108, C109, C110, C111, C112, C113: LCSC P/N (none) -> C15849
- D18, D19, D20, D21, D22, D23, D24, D25, D26, D27, D28, D29, D30, D31, D32, D33: LCSC P/N (none) -> C5628891
- R19, R20: LCSC P/N (none) -> C22808
- R21: LCSC P/N (none) -> C23179
- R280: LCSC P/N (none) -> C25804
- R281: LCSC P/N (none) -> C844548
- R32: LCSC P/N (none) -> C21189
- SW1: LCSC P/N (none) -> C221666
- U27, U28: LCSC P/N (none) -> C548830
- U29: LCSC P/N (none) -> C458145
- U30: LCSC P/N (none) -> C152467
