File: hardware/PowerDistributionUnit_Mk1/PowerDistributionUnit_Mk1.kicad_pcb (KiCad board)
At the start: 4 copper layers, 80.4 x 206 mm, 768 parts, among them J1 XT-30, J10 Logic Analyzer, J11 Logic Analyzer, J12 Logic Analyzer, J13 Logic Analyzer, J2 Molex_NanoFit_2x8, J3 Molex_NanoFit_1x6, J4 Molex_NanoFit_1x2, J5 Molex_NanoFit_1x2, J6 Conn_01x01, J8 Molex_NanoFit_1x2, J9 Molex_NanoFit_1x2, Q1 NVMFWS1D7N04XMT1G, Q2 NVMFWS1D7N04XMT1G, SW1 JS202011SCQN, U1 LeaderSOM, U10 74LVC594AD,118, U11 TPS27SA08CQPWPRQ1, U12 TPS27SA08CQPWPRQ1, U13 TPS27SA08CQPWPRQ1, U14 TPS27SA08CQPWPRQ1, U15 TPS27SA08CQPWPRQ1, U16 TPS27SA08CQPWPRQ1, U17 TPS27SA08CQPWPRQ1, U18 TPS27SA08CQPWPRQ1, U19 TPS27SA08CQPWPRQ1, U2 LM74502HDDFR, U20 TPS27SA08CQPWPRQ1, U21 TPS27SA08CQPWPRQ1, U22 MCP23S17-E/SO, U23 ADS131M08QPBSRQ1, U24 ADS131M08QPBSRQ1, U25 NL17SZS11DFT2G-Q, U26 TLV9002QDRQ1, U27 74LVC594AD,118, U28 74LVC594AD,118, U29 74AUP1G04GW-Q100H, U3 TPS27SA08CQPWPRQ1, U30 NL27WZ17DFT2G-Q, U31 74LVC594AD,118, U32 ACS37042KLHBLT-010B3, U33 ACS37042KLHBLT-010B3, U34 ACS37042KLHBLT-010B3, U35 ACS37042KLHBLT-010B3, U36 ACS37042KLHBLT-010B3, U37 ACS37042KLHBLT-010B3, U38 ACS37042KLHBLT-010B3, U39 ACS37042KLHBLT-010B3, U4 TPS27SA08CQPWPRQ1, U40 ACS37042KLHBLT-010B3, U41 ACS37042KLHBLT-010B3, U42 ACS37042KLHBLT-010B3, U43 ACS37042KLHBLT-010B3, U44 ACS37042KLHBLT-010B3, U45 ACS37042KLHBLT-010B3, U46 ACS37042KLHBLT-010B3, U47 ACS37042KLHBLT-010B3, U5 TPS27SA08CQPWPRQ1, U6 TPS27SA08CQPWPRQ1, U7 74LVC594AD,118, U8 74LVC594AD,118, U9 TPS27SA08CQPWPRQ1, Y1 ABM3-8.000MHZ-D2Y-T, Y2 ABM3-8.000MHZ-D2Y-T

Commit message: NC the mounting holes (because Lakshay Gupta)
Connections:
- H1 pad 1: GND -> unconnected-(H1-Pad1)
- H2 pad 1: GND -> unconnected-(H2-Pad1)
- H3 pad 1: GND -> unconnected-(H3-Pad1)
- H4 pad 1: GND -> unconnected-(H4-Pad1)
Changed lines of the file:
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@@
 	(net 498 "unconnected-(R9-Pad2)")
 	(net 499 "unconnected-(R11-Pad2)")
+	(net 500 "unconnected-(H1-Pad1)")
+	(net 501 "unconnected-(H2-Pad1)")
+	(net 502 "unconnected-(H3-Pad1)")
+	(net 503 "unconnected-(H4-Pad1)")
 	(footprint "Capacitor_SMD:C_0805_2012Metric"
 		(layer "F.Cu")
@@
 			(layers "*.Cu" "*.Mask")
 			(remove_unused_layers no)
-			(net 7 "GND")
+			(net 501 "unconnected-(H2-Pad1)")
 			(pinfunction "1")
-			(pintype "input")
+			(pintype "input+no_connect")
 			(zone_connect 2)
 		)
@@
 			(layers "*.Cu" "*.Mask")
 			(remove_unused_layers no)
-			(net 7 "GND")
+			(net 502 "unconnected-(H3-Pad1)")
 			(pinfunction "1")
-			(pintype "input")
+			(pintype "input+no_connect")
 			(zone_connect 2)
 		)
@@
 			(layers "*.Cu" "*.Mask")
 			(remove_unused_layers no)
-			(net 7 "GND")
+			(net 503 "unconnected-(H4-Pad1)")
 			(pinfunction "1")
-			(pintype "input")
+			(pintype "input+no_connect")
 			(zone_connect 2)
 		)
@@
 			(layers "*.Cu" "*.Mask")
 			(remove_unused_layers no)
-			(net 7 "GND")
+			(net 500 "unconnected-(H1-Pad1)")
 			(pinfunction "1")
-			(pintype "input")
+			(pintype "input+no_connect")
 			(zone_connect 2)
 		)
