File: hardware/PowerDistributionTestBreakout_Mk1/PowerDistributionTestBreakout_Mk1.kicad_sch (KiCad schematic)
At the start: 0 parts

Commit message: schematic, add symbol/footprint for screw terminal and banana connector
Parts:
- added H1, H2, H3, H4: M3, MountingHole:MountingHole_3.2mm_M3_Pad, symbol Mechanical:MountingHole_Pad
- added J1: Molex_NanoFit_2x8, PowerDistributionUnitLib:CONN_SD-105312-100_16_MOL, symbol PowerDistributionUnitLib:Molex_NanoFit_2x8
- added J10, J11, J12, J13, J14, J15, J16, J17, J18, J19, J20, J21, J22, J23, J24, J25, J26, J27, J28, J29, J3, J30, J31, J32, J33, J34, J4, J5, J6, J7, J8, J9: 575-4, PowerDistributionUnitLib:5754, symbol PowerDistributionUnitLib:575-4
- added J2: Molex_NanoFit_1x6, PowerDistributionUnitLib:CONN_SD-105309-100_06_MOL, symbol PowerDistributionUnitLib:Molex_NanoFit_1x6
- added J35, J36, J37, J38, J39, J40, J41, J42, J43, J44, J45, J46, J47, J48, J49, J50: TB002-500-02BE, PowerDistributionUnitLib:CUI_TB002-500-02BE, symbol PowerDistributionUnitLib:TB002-500-02BE
- added TP1, TP10, TP11, TP12, TP13, TP14, TP15, TP16, TP17, TP18, TP19, TP2, TP20, TP21, TP22, TP23, TP24, TP3, TP4, TP5, TP6, TP7, TP8, TP9: TestPoint, Connector_PinHeader_2.54mm:PinHeader_1x01_P2.54mm_Vertical, symbol Connector:TestPoint
Connections:
- new net GND: J10.1 (Pin_1), J15.1 (Pin_1), J16.1 (Pin_1), J17.1 (Pin_1), J18.1 (Pin_1), J2.1 (Pin_1), J2.2 (Pin_2), J2.3 (Pin_3), J2.4 (Pin_4), J2.5 (Pin_5), J2.6 (Pin_6), J27.1 (Pin_1), J28.1 (Pin_1), J29.1 (Pin_1), J30.1 (Pin_1), J31.1 (Pin_1), J32.1 (Pin_1), J33.1 (Pin_1), J34.1 (Pin_1), J35.2 (Pin_2), J36.2 (Pin_2), J37.2 (Pin_2), J38.2 (Pin_2), J39.2 (Pin_2), J4.1 (Pin_1), J40.2 (Pin_2), J41.2 (Pin_2), J42.2 (Pin_2), J43.2 (Pin_2), J44.2 (Pin_2), J45.2 (Pin_2), J46.2 (Pin_2), J47.2 (Pin_2), J48.2 (Pin_2), J49.2 (Pin_2), J50.2 (Pin_2), J6.1 (Pin_1), J9.1 (Pin_1), TP17.1, TP18.1, TP19.1, TP20.1, TP21.1, TP22.1, TP23.1, TP24.1
- new net LV_OUT.0: J1.8 (Pin_9), J3.1 (Pin_1), J35.1 (Pin_1), TP1.1
- new net LV_OUT.1: J1.7 (Pin_10), J36.1 (Pin_1), J5.1 (Pin_1), TP2.1
- new net LV_OUT.10: J1.14 (Pin_6), J21.1 (Pin_1), J45.1 (Pin_1), TP11.1
- new net LV_OUT.11: J1.13 (Pin_5), J22.1 (Pin_1), J46.1 (Pin_1), TP12.1
- new net LV_OUT.12: J1.12 (Pin_4), J23.1 (Pin_1), J47.1 (Pin_1), TP13.1
- new net LV_OUT.13: J1.11 (Pin_3), J24.1 (Pin_1), J48.1 (Pin_1), TP14.1
- new net LV_OUT.14: J1.10 (Pin_2), J25.1 (Pin_1), J49.1 (Pin_1), TP15.1
- new net LV_OUT.15: J1.9 (Pin_1), J26.1 (Pin_1), J50.1 (Pin_1), TP16.1
- new net LV_OUT.2: J1.6 (Pin_11), J37.1 (Pin_1), J7.1 (Pin_1), TP3.1
- new net LV_OUT.3: J1.5, J38.1 (Pin_1), J8.1 (Pin_1), TP4.1
- new net LV_OUT.4: J1.4 (Pin_13), J11.1 (Pin_1), J39.1 (Pin_1), TP5.1
- new net LV_OUT.5: J1.3 (Pin_14), J12.1 (Pin_1), J40.1 (Pin_1), TP6.1
- new net LV_OUT.6: J1.2 (Pin_15), J13.1 (Pin_1), J41.1 (Pin_1), TP7.1
- new net LV_OUT.7: J1.1 (Pin_16), J14.1 (Pin_1), J42.1 (Pin_1), TP8.1
- new net LV_OUT.8: J1.16 (Pin_8), J19.1 (Pin_1), J43.1 (Pin_1), TP9.1
- new net LV_OUT.9: J1.15 (Pin_7), J20.1 (Pin_1), J44.1 (Pin_1), TP10.1
- no-connect marks 0 -> 4
Other:
- company: (none) -> Longhorn Racing Solar
- title: (none) -> PDU Mk1 Test Breakout
