File: hardware/PS-PowerDistributionUnit.kicad_sch (KiCad schematic)
At the start: 5 parts, among them J1 XT-30, J2 Molex_NanoFit_1x2, J3 Molex_NanoFit_1x2

Commit message: init schem super simple..
Parts:
- added R49: 10k, symbol Device:R_US
Connections:
- net +3V3: now also R49.1
- net 48PinMCU/PG10-NRST: now also R49.2
Other:
- added sheet Indicators (Indicators.kicad_sch)
- sheet 48PinMCU ports: added PA8; removed none
- sheet Pair1: file untitled.kicad_sch -> Pair1.kicad_sch
- sheet Pair2: file untitled.kicad_sch -> Pair2.kicad_sch
- sheet Pair3: file untitled.kicad_sch -> Pair3.kicad_sch
- sheet Pair4: file untitled.kicad_sch -> Pair4.kicad_sch
- sheet Pair5: file untitled.kicad_sch -> Pair5.kicad_sch
- sheet Pair6: file untitled.kicad_sch -> Pair6.kicad_sch
- sheet Pair7: file untitled.kicad_sch -> Pair7.kicad_sch
- sheet Pair8: file untitled.kicad_sch -> Pair8.kicad_sch
- moved on the sheet: R8

Commit message: updated kicad and started on gamer led
Other:
- added sheet 5VBuck (5VBuck.kicad_sch)
