File: hardware/PS-PowerDistributionUnit.kicad_sch (KiCad schematic)
At the start: 25 parts, among them J1 LV_IN, J10 Conn_01x02, J11 Conn_01x02, J12 Conn_01x02, J13 Conn_01x02, J14 Conn_01x02, J15 Conn_01x02, J3 LV_0UT2

Commit message: before update design block
Parts:
- added TP17: DI_TP, Connector_PinHeader_2.54mm:PinHeader_1x01_P2.54mm_Vertical, symbol Connector:TestPoint
- added TP18: CS_TP1, Connector_PinHeader_2.54mm:PinHeader_1x01_P2.54mm_Vertical, symbol Connector:TestPoint
- added TP19: FLT_TP1, Connector_PinHeader_2.54mm:PinHeader_1x01_P2.54mm_Vertical, symbol Connector:TestPoint
- added TP20: FLT_TP2, Connector_PinHeader_2.54mm:PinHeader_1x01_P2.54mm_Vertical, symbol Connector:TestPoint
- added TP21: CS_TP2, Connector_PinHeader_2.54mm:PinHeader_1x01_P2.54mm_Vertical, symbol Connector:TestPoint
- added TP22: FLT_TP3, Connector_PinHeader_2.54mm:PinHeader_1x01_P2.54mm_Vertical, symbol Connector:TestPoint
- added TP23: CS_TP3, Connector_PinHeader_2.54mm:PinHeader_1x01_P2.54mm_Vertical, symbol Connector:TestPoint
- added TP24: FLT_TP4, Connector_PinHeader_2.54mm:PinHeader_1x01_P2.54mm_Vertical, symbol Connector:TestPoint
- added TP25: CS_TP4, Connector_PinHeader_2.54mm:PinHeader_1x01_P2.54mm_Vertical, symbol Connector:TestPoint
- added TP26: FLT_TP5, Connector_PinHeader_2.54mm:PinHeader_1x01_P2.54mm_Vertical, symbol Connector:TestPoint
- added TP27: CS_TP5, Connector_PinHeader_2.54mm:PinHeader_1x01_P2.54mm_Vertical, symbol Connector:TestPoint
- added TP28: FLT_TP6, Connector_PinHeader_2.54mm:PinHeader_1x01_P2.54mm_Vertical, symbol Connector:TestPoint
- added TP29: CS_TP6, Connector_PinHeader_2.54mm:PinHeader_1x01_P2.54mm_Vertical, symbol Connector:TestPoint
- added TP32: 24V_PHSS, TestPoint:TestPoint_THTPad_D3.0mm_Drill1.5mm, symbol Connector:TestPoint
- added TP45, TP46: GND, TestPoint:TestPoint_THTPad_D3.0mm_Drill1.5mm, symbol Connector:TestPoint
- TP6: value TestPoint -> MISO_TP; footprint (none) -> Connector_PinHeader_2.54mm:PinHeader_1x01_P2.54mm_Vertical
- TP7: value TestPoint -> SCLK_TP; footprint (none) -> Connector_PinHeader_2.54mm:PinHeader_1x01_P2.54mm_Vertical
- TP8: value TestPoint -> MOSI_TP; footprint (none) -> Connector_PinHeader_2.54mm:PinHeader_1x01_P2.54mm_Vertical
- TP9: value TestPoint -> LIMP_TP; footprint (none) -> Connector_PinHeader_2.54mm:PinHeader_1x01_P2.54mm_Vertical
Connections:
- net +24V_HSS: now also TP32.1
- net 48PinMCU/PA15: now also TP21.1
- net 48PinMCU/PA3: now also TP23.1
- net 48PinMCU/PA4: now also TP18.1
- net 48PinMCU/PA7: no longer TP8.1
- net 48PinMCU/PA8: now also TP25.1
- net 48PinMCU/PA9: now also TP20.1
- net 48PinMCU/PB1: now also TP27.1
- net 48PinMCU/PB10: now also TP19.1
- net 48PinMCU/PB11: now also TP22.1
- net 48PinMCU/PB3: now also TP29.1
- net 48PinMCU/PB4: now also TP24.1
- net 48PinMCU/PC13: now also TP28.1
- net 48PinMCU/PC14: now also TP26.1
- net DI_MODE: now also TP17.1
- net GND: now also TP45.1, TP46.1
- net MOSI: now also TP8.1
- no-connect marks 13 -> 14
Other:
- note added: "TODO: -need more calc for specific Rsns and Csns -fix indicators, more debug led -switch to 12V versions of design blocks once they're made -after 12V switch: It looks like the indicator LEDs have a max rating of 5.3V. Once we switch the buck passives, make sure that the output of the buck is within the acceptable range"
- note removed: "TODO: -need more calc for specific Rsns and Csns -fix indicators, more debug led -logic analyzer need? -switch to 12V versions of design blocks once they're made -after 12V switch: It looks like the indicator LEDs have a max rating of 5.3V. Once we switch the buck passives, make sure that the output of the buck is within the acceptable range"
- moved on the sheet: F1, H1, H2, H3, H4, J1, J10, J11, J12, J13, J14, J15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

Commit message: added p/n and footprints
Parts:
- F1: footprint (none) -> LHRS_Power:Fuse-3557-2
- H1, H2, H3, H4: footprint (none) -> MountingHole:MountingHole_3.2mm_M3_Pad
- J10, J11, J12, J13, J14, J15: footprint (none) -> Connector_Molex:Molex_Nano-Fit_105309-xx02_1x02_P2.50mm_Vertical; LCSC P/N (none) -> C2938824; P/N (none) -> 1053091102
- J3: LCSC P/N (none) -> C485572; P/N (none) -> 430451212
- R1, R2, R3, R4, R5, R6: footprint (none) -> Resistor_SMD:R_0603_1608Metric; P/N (none) -> CRCW060310K0FKEI
- R10, R9: footprint (none) -> Resistor_SMD:R_0603_1608Metric; LCSC P/N (none) -> C107701; P/N (none) -> RC0603FR-0722RL
- TP17, TP18, TP19, TP20, TP21, TP22, TP23, TP24, TP25, TP26, TP27, TP28, TP29, TP6, TP7, TP8, TP9: LCSC P/N (none) -> C41426955; P/N (none) -> A254N01-0B1P51-H25A60
