File: hardware/untitled.kicad_sch (KiCad schematic)
At the start: 3 parts, among them IC2 TPS2HCS08AQPWPRQ1

Commit message: added hss and driving back from houston
Parts:
- added C: C_SNS, symbol Device:C
- added D, D3: D_TVS, symbol Device:D_TVS
- added F2: C1F_8, Fuse:Fuse_1206_3216Metric, symbol PowerDistributionUnitLib:C1F_8
- added R: 10k, symbol Device:R_US
- R: renamed from R9; value R_US -> R_SNS
- renumbered IC2 to IC
Connections:
- net GND: now also R.2, C.2, D.1 (A1), D3.1 (A1)
- net at IC.10 (VOUT2_2): now also IC.11 (VOUT2_3), IC.9 (VOUT2_1), F2.2
- net at IC.2 (SNS): now also R.1, C.1
- net at IC.4 (DI): now also R.1
- net at F1.1: now also D.2 (A2)
- new net: D3.2 (A2), F2.1
- new net DI_MODE: R.2
Other:
- note added: "R and C should be placed close to sns pin"
- note added: "recommended: 0.2-1.5kΩ and 1 - 4.7nF"
- note removed: "R should be placed close to sns pin"
- note removed: "recommended: 0.2-1.5kΩ"
- moved on the sheet: F1, IC, R

Commit message: before sleep progress-added out put and current reverse stuff for elcon
Parts:
- added D20: D_Schottky, symbol Device:D_Schottky
- added J12, J4: Conn_01x02, symbol Connector_Generic:Conn_01x02
- renumbered C to C21, D to D13, IC to IC6, R to R21, R to R24
Connections:
- net GND: now also J12.1 (Pin_1), J4.2 (Pin_2); no longer D13.1 (A1), D3.1 (A1)
- new net: D20.2 (A), D3.1 (A1)
- new net: D13.1 (A1), J12.2 (Pin_2)
- new net elcon: D20.1 (K), J4.1 (Pin_1)
