File: hardware/3V3Buck.kicad_sch (KiCad schematic)
At the start: 12 parts, among them U1 LMR51635XDDCR

Commit message: progress
Parts:
- U1: footprint breh:DDC0006A-MFG -> LHRS_ICs:DDC0006A-MFG
- renumbered TP18 to TP?, TP19 to TP?, TP17 to TP?, TP16 to TP?
Changed lines of the file:
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@@
 			)
 			(project "PS-Buck"
-				(path "/eb16378f-e371-46a9-bfab-b0d9404d0362/bf74a586-cb4a-4ae5-9c2d-204be6a4ff19"
+				(path "/eb16378f-e371-46a9-bfab-b0d9404d0362/5dad52f3-6f13-4043-9864-0ec1f6c2175f"
 					(reference "C7")
 					(unit 1)
@@
 			)
 			(project "PS-Buck"
-				(path "/eb16378f-e371-46a9-bfab-b0d9404d0362/bf74a586-cb4a-4ae5-9c2d-204be6a4ff19"
+				(path "/eb16378f-e371-46a9-bfab-b0d9404d0362/5dad52f3-6f13-4043-9864-0ec1f6c2175f"
 					(reference "R6")
 					(unit 1)
@@
 		(on_board yes)
 		(dnp no)
-		(property "Reference" "TP18"
+		(property "Reference" "TP?"
 			(at 222.25 119.8879 0)
 			(effects
@@
 		)
 		(instances
+			(project "3V3Buck"
+				(path "/39da07fa-d2fd-433c-a855-3c74e2086fee"
+					(reference "TP?")
+					(unit 1)
+				)
+			)
 			(project "PowerPath"
 				(path "/ad6c7df0-eb90-4670-9aa8-3e2007aefc2d/1dff8fcf-47f2-40bd-a8d2-72c78139361d"
@@
 				)
 			)
-			(project "PowerPath"
-				(path "/eb16378f-e371-46a9-bfab-b0d9404d0362/bf74a586-cb4a-4ae5-9c2d-204be6a4ff19"
-					(reference "TP18")
+			(project "3V3Buck"
+				(path "/eb16378f-e371-46a9-bfab-b0d9404d0362/5dad52f3-6f13-4043-9864-0ec1f6c2175f"
+					(reference "TP?")
 					(unit 1)
 				)
@@
 			)
 			(project "PS-Buck"
-				(path "/eb16378f-e371-46a9-bfab-b0d9404d0362/bf74a586-cb4a-4ae5-9c2d-204be6a4ff19"
+				(path "/eb16378f-e371-46a9-bfab-b0d9404d0362/5dad52f3-6f13-4043-9864-0ec1f6c2175f"
 					(reference "C6")
 					(unit 1)
@@
 			)
 			(project "PS-Buck"
-				(path "/eb16378f-e371-46a9-bfab-b0d9404d0362/bf74a586-cb4a-4ae5-9c2d-204be6a4ff19"
+				(path "/eb16378f-e371-46a9-bfab-b0d9404d0362/5dad52f3-6f13-4043-9864-0ec1f6c2175f"
 					(reference "#FLG04")
 					(unit 1)
@@
 			)
 			(project "PS-Buck"
-				(path "/eb16378f-e371-46a9-bfab-b0d9404d0362/bf74a586-cb4a-4ae5-9c2d-204be6a4ff19"
+				(path "/eb16378f-e371-46a9-bfab-b0d9404d0362/5dad52f3-6f13-4043-9864-0ec1f6c2175f"
 					(reference "L1")
 					(unit 1)
@@
 			)
 		)
-		(property "Footprint" "breh:DDC0006A-MFG"
+		(property "Footprint" "LHRS_ICs:DDC0006A-MFG"
 			(at 97.79 76.2 0)
 			(effects
@@
 			)
 			(project "PS-Buck"
-				(path "/eb16378f-e371-46a9-bfab-b0d9404d0362/bf74a586-cb4a-4ae5-9c2d-204be6a4ff19"
+				(path "/eb16378f-e371-46a9-bfab-b0d9404d0362/5dad52f3-6f13-4043-9864-0ec1f6c2175f"
 					(reference "U1")
 					(unit 1)
@@
 		(on_board yes)
 		(dnp no)
-		(property "Reference" "TP19"
+		(property "Reference" "TP?"
 			(at 222.25 132.5879 0)
 			(effects
@@
 		)
 		(instances
+			(project "3V3Buck"
+				(path "/39da07fa-d2fd-433c-a855-3c74e2086fee"
+					(reference "TP?")
+					(unit 1)
+				)
+			)
 			(project "PowerPath"
 				(path "/ad6c7df0-eb90-4670-9aa8-3e2007aefc2d/1dff8fcf-47f2-40bd-a8d2-72c78139361d"
@@
 				)
 			)
-			(project "PowerPath"
-				(path "/eb16378f-e371-46a9-bfab-b0d9404d0362/bf74a586-cb4a-4ae5-9c2d-204be6a4ff19"
-					(reference "TP19")
+			(project "3V3Buck"
+				(path "/eb16378f-e371-46a9-bfab-b0d9404d0362/5dad52f3-6f13-4043-9864-0ec1f6c2175f"
+					(reference "TP?")
 					(unit 1)
 				)
@@
 			)
 			(project "PS-Buck"
-				(path "/eb16378f-e371-46a9-bfab-b0d9404d0362/bf74a586-cb4a-4ae5-9c2d-204be6a4ff19"
+				(path "/eb16378f-e371-46a9-bfab-b0d9404d0362/5dad52f3-6f13-4043-9864-0ec1f6c2175f"
 					(reference "C3")
 					(unit 1)
@@
 		(on_board yes)
 		(dnp no)
-		(property "Reference" "TP17"
+		(property "Reference" "TP?"
 			(at 209.55 132.5879 0)
 			(effects
@@
 		)
 		(instances
+			(project "3V3Buck"
+				(path "/39da07fa-d2fd-433c-a855-3c74e2086fee"
+					(reference "TP?")
+					(unit 1)
+				)
+			)
 			(project "PowerPath"
 				(path "/ad6c7df0-eb90-4670-9aa8-3e2007aefc2d/1dff8fcf-47f2-40bd-a8d2-72c78139361d"
@@
 				)
 			)
-			(project "PowerPath"
-				(path "/eb16378f-e371-46a9-bfab-b0d9404d0362/bf74a586-cb4a-4ae5-9c2d-204be6a4ff19"
-					(reference "TP17")
+			(project "3V3Buck"
+				(path "/eb16378f-e371-46a9-bfab-b0d9404d0362/5dad52f3-6f13-4043-9864-0ec1f6c2175f"
+					(reference "TP?")
 					(unit 1)
 				)
@@
 		(on_board yes)
 		(dnp no)
-		(property "Reference" "TP16"
+		(property "Reference" "TP?"
 			(at 209.55 119.8879 0)
 			(effects
@@
 		)
 		(instances
+			(project "3V3Buck"
+				(path "/39da07fa-d2fd-433c-a855-3c74e2086fee"
+					(reference "TP?")
+					(unit 1)
+				)
+			)
 			(project "PowerPath"
 				(path "/ad6c7df0-eb90-4670-9aa8-3e2007aefc2d/1dff8fcf-47f2-40bd-a8d2-72c78139361d"
@@
 				)
 			)
-			(project "PowerPath"
-				(path "/eb16378f-e371-46a9-bfab-b0d9404d0362/bf74a586-cb4a-4ae5-9c2d-204be6a4ff19"
-					(reference "TP16")
+			(project "3V3Buck"
+				(path "/eb16378f-e371-46a9-bfab-b0d9404d0362/5dad52f3-6f13-4043-9864-0ec1f6c2175f"
+					(reference "TP?")
 					(unit 1)
 				)
@@
 			)
 			(project "PS-Buck"
-				(path "/eb16378f-e371-46a9-bfab-b0d9404d0362/bf74a586-cb4a-4ae5-9c2d-204be6a4ff19"
+				(path "/eb16378f-e371-46a9-bfab-b0d9404d0362/5dad52f3-6f13-4043-9864-0ec1f6c2175f"
 					(reference "#FLG03")
 					(unit 1)
@@
 			)
 			(project "PS-Buck"
-				(path "/eb16378f-e371-46a9-bfab-b0d9404d0362/bf74a586-cb4a-4ae5-9c2d-204be6a4ff19"
+				(path "/eb16378f-e371-46a9-bfab-b0d9404d0362/5dad52f3-6f13-4043-9864-0ec1f6c2175f"
 					(reference "C4")
 					(unit 1)
@@
 			)
 			(project "PS-Buck"
-				(path "/eb16378f-e371-46a9-bfab-b0d9404d0362/bf74a586-cb4a-4ae5-9c2d-204be6a4ff19"
+				(path "/eb16378f-e371-46a9-bfab-b0d9404d0362/5dad52f3-6f13-4043-9864-0ec1f6c2175f"
 					(reference "R7")
 					(unit 1)
