File: hardware/Pair1.kicad_sch (KiCad schematic)
At the start: 11 parts, among them J12 Conn_01x02, J4 Conn_01x02

Commit message: aesthetic added
Parts:
- removed D3, D?: D_TVS, symbol Device:D_TVS
- removed F1, F2: C1F_8, Fuse:Fuse_1206_3216Metric, symbol PowerDistributionUnitLib:C1F_8
- removed J12, J4: Conn_01x02, symbol Connector_Generic:Conn_01x02
- removed R?: 10k, symbol Device:R_US
- removed R?: R_SNS, symbol Device:R_US
- added C30, C31: 100n, symbol Device:C
- added D39, D40: D_TVS, symbol Device:D_TVS
- added F17, F18: C1F_8, Fuse:Fuse_1206_3216Metric, symbol PowerDistributionUnitLib:C1F_8
- added J20, J21: Conn_01x02, symbol Connector_Generic:Conn_01x02
- added R50: 10k, symbol Device:R_US
- added R51: R_SNS, symbol Device:R_US
Connections:
- net DI_MODE: now also R50.2
- net GND: now also D20.2 (A), C30.1, C31.1, D39.1 (A1), D40.1 (A1), J20.1 (Pin_1), J21.1 (Pin_1), R51.2
- net at IC?.10 (VOUT2_2), IC?.11 (VOUT2_3), IC?.9 (VOUT2_1): now also F17.2
- net at C?.1, IC?.2 (SNS): now also R51.1
- net at IC?.4 (DI): now also R50.1
- net at IC?.6 (VOUT1_1), IC?.7 (VOUT1_2), IC?.8 (VOUT1_3): now also F18.2
- net at D20.1 (K): now also C30.2, D39.2 (A2), F17.1, J20.2 (Pin_2)
- new net: C31.2, D40.2 (A2), F18.1, J21.2 (Pin_2)
Other:
- moved on the sheet: C?, IC?

Commit message: progress
Parts:
- removed F17, F18: C1F_8, Fuse:Fuse_1206_3216Metric, symbol PowerDistributionUnitLib:C1F_8
- added F1, F9: Fuse_3557_2, LHRS_Power:Fuse-3557-2, symbol lhrs_power:Fuse_3557_2
Connections:
- net GND: no longer D20.2 (A)
- net at C31.2, D40.2 (A2), J21.2 (Pin_2): now also F1.2
- net at IC?.10 (VOUT2_2), IC?.11 (VOUT2_3), IC?.9 (VOUT2_1): now also F9.1
- net at IC?.6 (VOUT1_1), IC?.7 (VOUT1_2), IC?.8 (VOUT1_3): now also F1.1
- new net: D20.2 (A), F9.2
Other:
- moved on the sheet: C30, D20, D39, J20

Commit message: discrete cs
Parts:
- gave numbers to parts that had none: 2
- renumbered C31 to C25, C30 to C26, D40 to D21, D20 to D22, D39 to D23, F9 to F2, J21 to J4, J20 to J5, R50 to R12, R51 to R13
Connections:
- net SDI renamed SPI_MOSI
- net SDO renamed SPI_MISO

Commit message: surahbi comment mostly done except led
Parts:
- removed C25, C26: 100n, symbol Device:C
- removed D21, D23: D_TVS, symbol Device:D_TVS
- removed D22: D_Schottky, symbol Device:D_Schottky
- removed F1, F2: Fuse_3557_2, LHRS_Power:Fuse-3557-2, symbol lhrs_power:Fuse_3557_2
- removed J4, J5: Conn_01x02, symbol Connector_Generic:Conn_01x02
- removed R12: 10k, symbol Device:R_US
- removed R13: R_SNS, symbol Device:R_US
- added C28, C32: 100n, symbol Device:C
- added C47: 1000n, symbol Device:C
- added C6: 1n, symbol Device:C
- added C62: 470n, symbol Device:C
- added D24, D26, D41: D_TVS, symbol Device:D_TVS
- added D50: D_Schottky, symbol Device:D_Schottky
- added F3, F6: 7.5A, LHRS_Power:Fuse-3557-2, symbol lhrs_power:Fuse_3557_2
- added R12, R64: 10k, symbol Device:R
- added R13: 1k, symbol Device:R
- added R19, R36: 4.7k, symbol Device:R
- added R28, R40, R47, R58: 22, symbol Device:R
- added R77: 10, symbol Device:R
- C24: value C_SNS -> 2.2n
Connections:
- net +24V: now also C47.1, C6.1, D41.2 (A2)
- net +3V3: now also R36.1, R77.1; no longer IC2.3 (VDD)
- net DI_MODE: now also R12.1
- net FLT_WAKE: now also R36.2, R64.1, R64.2
- net GND: now also C28.1, C32.1, C47.2, C6.2, C62.2, D24.1 (A1), D26.1 (A1), D41.1 (A1), D50.1 (K), R19.2; no longer C24.2, IC2.1 (GND)
- net SPI_CS: now also R47.1; no longer IC2.15 (NCS)
- net SPI_MISO: now also R40.1; no longer IC2.14 (SDO)
- net SPI_MOSI: now also R28.1; no longer IC2.13 (SDI)
- net SPI_SCLK: now also R58.1; no longer IC2.16 (SCLK)
- net VOUT2: now reaches IC2.10 (VOUT2_2), IC2.11 (VOUT2_3), IC2.9 (VOUT2_1)
- net VOUT2: now also F6.1
- net at C24.1, IC2.2 (SNS): now also R13.2
- net at IC2.4 (DI): now also R12.2
- net VOUT1: now reaches IC2.6 (VOUT1_1), IC2.7 (VOUT1_2), IC2.8 (VOUT1_3)
- net VOUT1: now also F3.1
- new net: IC2.15 (NCS), R47.2
- new net: C24.2, D50.2 (A), IC2.1 (GND), R13.1, R19.1
- new net: IC2.13 (SDI), R28.2
- new net: IC2.14 (SDO), R40.2
- new net: IC2.16 (SCLK), R58.2
- new net OUTPUT1: C28.2, D24.2 (A2), F3.2
- new net OUTPUT2: C32.2, D26.2 (A2), F6.2
- new net VDD: C62.1, IC2.3 (VDD), R77.2
Other:
- note added: "Battery Voltage"
- note added: "FLT/WAKE SIGNAL"
- note added: "Output"
- note added: "Voltage at Drain"
- note removed: "recommended: 0.2-1.5kΩ and 1 - 4.7nF"
- moved on the sheet: C24, IC2
