File: hardware/Pair1.kicad_sch (KiCad schematic)
At the start: 23 parts, among them IC2 TPS2HCS08AQPWPRQ1

Commit message: added hss physical fuse
Connections:
- net +24V renamed +24V_HSS
Changed lines of the file:
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@@
 	(wire
 		(pts
-			(xy 118.745 84.455) (xy 125.095 84.455)
+			(xy 119.38 84.455) (xy 125.095 84.455)
 		)
 		(stroke
@@
 	(wire
 		(pts
-			(xy 118.745 81.915) (xy 118.745 84.455)
-		)
-		(stroke
-			(width 0)
-			(type default)
-		)
-	)
-	(wire
-		(pts
 			(xy 157.48 50.8) (xy 157.48 53.34)
 		)
@@
 	(wire
 		(pts
-			(xy 115.57 86.995) (xy 125.095 86.995)
+			(xy 120.015 86.995) (xy 125.095 86.995)
 		)
 		(stroke
@@
 	)
 	(label "VDD"
-		(at 115.57 86.995 0)
+		(at 120.015 86.995 0)
 		(effects
 			(font
@@
 		)
 	)
+	(hierarchical_label "+24V_HSS"
+		(shape input)
+		(at 119.38 84.455 180)
+		(effects
+			(font
+				(size 1.27 1.27)
+			)
+			(justify right)
+		)
+	)
 	(hierarchical_label "OUTPUT2"
 		(shape output)
@@
 		)
 	)
-	(symbol
-		(lib_id "power:+24V")
-		(at 118.745 81.915 0)
-		(unit 1)
-		(body_style 1)
-		(exclude_from_sim no)
-		(in_bom yes)
-		(on_board yes)
-		(in_pos_files yes)
-		(dnp no)
-		(fields_autoplaced yes)
-		(property "Reference" "#PWR052"
-			(at 118.745 85.725 0)
-			(hide yes)
-			(show_name no)
-			(do_not_autoplace no)
-			(effects
-				(font
-					(size 1.27 1.27)
-				)
-			)
-		)
-		(property "Value" "+24V"
-			(at 118.745 77.47 0)
-			(show_name no)
-			(do_not_autoplace no)
-			(effects
-				(font
-					(size 1.27 1.27)
-				)
-			)
-		)
-		(property "Footprint" ""
-			(at 118.745 81.915 0)
-			(hide yes)
-			(show_name no)
-			(do_not_autoplace no)
-			(effects
-				(font
-					(size 1.27 1.27)
-				)
-			)
-		)
-		(property "Datasheet" ""
-			(at 118.745 81.915 0)
-			(hide yes)
-			(show_name no)
-			(do_not_autoplace no)
-			(effects
-				(font
-					(size 1.27 1.27)
-				)
-			)
-		)
-		(property "Description" "Power symbol creates a global label with name \"+24V\""
-			(at 118.745 81.915 0)
-			(hide yes)
-			(show_name no)
-			(do_not_autoplace no)
-			(effects
-				(font
-					(size 1.27 1.27)
-				)
-			)
-		)
-		(pin "1"
-		)
-		(instances
-			(project "PS-PowerDistributionUnit"
-				(path "/eb16378f-e371-46a9-bfab-b0d9404d0362/3909f681-ed21-4f6c-997f-d0f5d9a50140"
-					(reference "#PWR087")
-					(unit 1)
-				)
-				(path "/eb16378f-e371-46a9-bfab-b0d9404d0362/91ab2e5b-361c-4f6e-96f4-249ed894cf88"
-					(reference "#PWR080")
-					(unit 1)
-				)
-				(path "/eb16378f-e371-46a9-bfab-b0d9404d0362/95650361-8e3d-4fb9-aeae-766234533dc0"
-					(reference "#PWR066")
-					(unit 1)
-				)
-				(path "/eb16378f-e371-46a9-bfab-b0d9404d0362/ac45b9fd-4ce8-4391-9e98-0dd18286737f"
-					(reference "#PWR052")
-					(unit 1)
-				)
-				(path "/eb16378f-e371-46a9-bfab-b0d9404d0362/cb13da7e-067a-493c-b3b5-481ca6e5952d"
-					(reference "#PWR059")
-					(unit 1)
-				)
-				(path "/eb16378f-e371-46a9-bfab-b0d9404d0362/deedd56c-6817-40a7-b528-032192f149d8"
-					(reference "#PWR073")
-					(unit 1)
-				)
-			)
-		)
-	)

Commit message: addressed review and pushing
Parts:
- added D18, D39: LED, symbol Device:LED
- added R5, R85: 4.7k, symbol Device:R
Connections:
- net OUTPUT1: now also D18.1 (K)
- net OUTPUT2: now also D39.1 (K)
- net VOUT1: now also R5.1
- net VOUT2: now also R85.1
- new net: D39.2 (A), R85.2
- new net: D18.2 (A), R5.2
Other:
- note added: "Output with blown fuse indicator"
- note removed: "Output"
- moved on the sheet: C28, C32, D24, D26, F3, F6

Commit message: some reviews done
Parts:
- C47: value 1000n -> 1u
- F3, F6: value 7.5A -> 5A
Changed lines of the file:
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@@
 			)
 		)
-		(property "Value" "7.5A"
+		(property "Value" "5A"
 			(at 201.93 63.5 90)
 			(show_name no)
@@
 			)
 		)
-		(property "Value" "1000n"
+		(property "Value" "1u"
 			(at 142.24 48.2599 0)
 			(show_name no)
@@
 			)
 		)
-		(property "Value" "7.5A"
+		(property "Value" "5A"
 			(at 201.93 36.83 90)
 			(show_name no)
