File: hardware/PowerProtection.kicad_sch (KiCad schematic)
At the start: 17 parts, among them U7 LM76202QPWPRQ1

Commit message: progress
Parts:
- removed C20, C23: 10uF, Capacitor_SMD:C_0805_2012Metric_Pad1.18x1.45mm_HandSolder, symbol Device:C
- removed C25: 100nF, Capacitor_SMD:C_0603_1608Metric_Pad1.08x0.95mm_HandSolder, symbol Device:C
- removed D10: TVS, Diode_SMD:D_SOD-123F, symbol Device:D_Zener
- removed D2: TVS, Diode_SMD:D_SOD-323_HandSoldering, symbol Diode:SD12_SOD323
- removed R12: 45.3k, Resistor_SMD:R_0603_1608Metric_Pad0.98x0.95mm_HandSolder, symbol Device:R
- removed R13: 590, Resistor_SMD:R_0603_1608Metric_Pad0.98x0.95mm_HandSolder, symbol Device:R
- removed R15: 2.1k, Resistor_SMD:R_0603_1608Metric_Pad0.98x0.95mm_HandSolder, symbol Device:R
- removed R20: 402k, Resistor_SMD:R_0603_1608Metric_Pad0.98x0.95mm_HandSolder, symbol Device:R
- removed R23, R27: 10k, Resistor_SMD:R_0603_1608Metric_Pad0.98x0.95mm_HandSolder, symbol Device:R
- removed R30: 24m, Resistor_SMD:R_0603_1608Metric_Pad0.98x0.95mm_HandSolder, symbol Device:R
- removed R31: 100k, Resistor_SMD:R_0603_1608Metric_Pad0.98x0.95mm_HandSolder, symbol Device:R
- removed U7: LM76202QPWPRQ1, UTSVT_Power:LM76202QPWPRQ1, symbol utsvt_power:LM76202QPWPRQ1
- added C3: 220n, Capacitor_SMD:C_0603_1608Metric_Pad1.08x0.95mm_HandSolder, symbol Device:C
- added C4: 10n, Capacitor_SMD:C_0603_1608Metric_Pad1.08x0.95mm_HandSolder, symbol ECE319H:C
- added C5: 10u, Capacitor_SMD:C_0805_2012Metric_Pad1.18x1.45mm_HandSolder, symbol Device:C
- added D1: SMAF4758A, LHRS_Passives:SODFL5026X125N, symbol Device:D_Zener
- added D2: SMBJ30CD, Diode_SMD:D_SMB, symbol Device:D_Zener
- added IC1: LM74502DDFR, LHRS_Power:LM74502DDFR, symbol LHRS_ICs:LM74502HDDFR
- added Q1, Q2: PSMN012-100YS, Package_TO_SOT_SMD:LFPAK56, symbol lhrs_power:PSMN012-100YS
- added R3: 33, Resistor_SMD:R_0603_1608Metric_Pad0.98x0.95mm_HandSolder, symbol Device:R
- added R4: 221k, Resistor_SMD:R_0603_1608Metric_Pad0.98x0.95mm_HandSolder, symbol Device:R
- added R5, R7: 10k, Resistor_SMD:R_0603_1608Metric_Pad0.98x0.95mm_HandSolder, symbol Device:R
- added R6: 137k, Resistor_SMD:R_0603_1608Metric_Pad0.98x0.95mm_HandSolder, symbol Device:R
- C1: value 1uF -> 0.1u; LCSC P/N (none) -> C14663; P/N MLASU168SB5105KTNA01 -> MLASH168SB7104KTNA01
- C2: value 1uF -> 1u; LCSC P/N (none) -> C15849
- R1: LCSC P/N (none) -> C25804; Mouser Part Number (none) -> 71-CRCW060310K0FKEI; P/N CRCW060310K0FKEI -> CRCW060310K0FKEI
Connections:
- net Fault is gone; now on net Vin: R1.2
- net GND: now also C2.1, C4.2, C5.2, D1.2 (A), D2.2 (A2), IC1.2 (GND), R5.2, R7.2; no longer C2.2
- net +24V: no longer names the net of R1.1
- net +24V: now also C2.2, C3.1, D1.1 (K), IC1.5 (VS); no longer C2.1
- net 24V_Ext renamed Vin
- net Vin: now also D2.1 (A1), Q1.5, R4.1, R6.2
- new net: C3.2, IC1.4 (VCAP)
- new net: C4.1, R3.1
- new net EN/UVLO: IC1.1 (EN/UVLO), R6.1, R7.1
- new net OV: IC1.7 (OV), R4.2, R5.1
- new net Vout: C5.1, Q2.5
- new net gate: IC1.6 (GATE), Q1.4, Q2.4, R3.2
- new net source: IC1.8 (SRC), Q1.1, Q1.2, Q1.3, Q2.1, Q2.2, Q2.3
- no-connect marks 2 -> 0
Other:
- note added: "1.235 is Enable/UVLO falling threshold on data sheet"
- note added: "4.84ms = 75us + 220nF * 6.5V/300uA 6.5V recommended on datasheet 4.84ms power up delay"
- note added: "Kell Harpole"
- note added: "Overvoltage Protection: 29.03V Vovr = (R2 * Vov)/(R1 + R2) Vov = Vovr * (R1 + R2) / R2 28.875 = 1.25 * (221k + 10k) / 10k"
- note removed: "20.88 ms ramp time"
- note removed: "Current Monitoring"
- note removed: "DNP until validated"
- note removed: "Functional Mode Selection"
- note removed: "ILim(A) = 12/R(k) 1.2A = 12/10kΩ"
- note removed: "OVP set to 27v for buck max voltage of 28v"
- note removed: "Overcurrent Protection"
- note removed: "Pullups"
- note removed: "RTN!=GND Conecting GND to RTN turns off RPP!"
- note removed: "SHDN has weak internal pullup - pulled up to MCU voltage after initial power on"
- note removed: "Set to circuit breaker (latchoff) Use 0 ohm resistor for auto-retry (540ms)"
- note removed: "Typical gain: 78.28 uA/A Vout @ 1.3A = 2.407v R(imon) = 23.7 mΩ"
- note removed: "Under/Overvoltage Protection"

Commit message: added kell pp block
Parts:
- renumbered C1 to C16, C2 to C17, C3 to C18, C4 to C19, C5 to C20, D2 to D21, D1 to D22, IC1 to IC2, R3 to R10, R4 to R11, R5 to R12, R7 to R13, R6 to R14, R1 to R9
Changed lines of the file:
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@@
 		(dnp no)
 		(fields_autoplaced yes)
-		(property "Reference" "C3"
+		(property "Reference" "C18"
 			(at 57.785 80.0099 0)
 			(show_name no)
@@
 				(path "/a968d2b9-0c0e-491c-a5a4-aacd8448ff64"
 					(reference "C3")
+					(unit 1)
+				)
+			)
+			(project "PS-PowerDistributionUnit"
+				(path "/eb16378f-e371-46a9-bfab-b0d9404d0362/57719e66-c5b1-466c-b4ff-7913976ad99e"
+					(reference "C18")
 					(unit 1)
 				)
@@
 		(dnp no)
 		(fields_autoplaced yes)
-		(property "Reference" "R1"
+		(property "Reference" "R9"
 			(at 45.72 60.9599 0)
 			(show_name no)
@@
 				(path "/a968d2b9-0c0e-491c-a5a4-aacd8448ff64"
 					(reference "R1")
+					(unit 1)
+				)
+			)
+			(project "PS-PowerDistributionUnit"
+				(path "/eb16378f-e371-46a9-bfab-b0d9404d0362/57719e66-c5b1-466c-b4ff-7913976ad99e"
+					(reference "R9")
 					(unit 1)
 				)
@@
 		(in_pos_files yes)
 		(dnp no)
-		(property "Reference" "R7"
+		(property "Reference" "R13"
 			(at 125.73 77.47 90)
 			(show_name no)
@@
 				(path "/a968d2b9-0c0e-491c-a5a4-aacd8448ff64"
 					(reference "R7")
+					(unit 1)
+				)
+			)
+			(project "PS-PowerDistributionUnit"
+				(path "/eb16378f-e371-46a9-bfab-b0d9404d0362/57719e66-c5b1-466c-b4ff-7913976ad99e"
+					(reference "R13")
 					(unit 1)
 				)
@@
 		(in_pos_files yes)
 		(dnp no)
-		(property "Reference" "C1"
+		(property "Reference" "C16"
 			(at 38.1 49.5299 0)
 			(show_name no)
@@
 				(path "/a968d2b9-0c0e-491c-a5a4-aacd8448ff64"
 					(reference "C1")
+					(unit 1)
+				)
+			)
+			(project "PS-PowerDistributionUnit"
+				(path "/eb16378f-e371-46a9-bfab-b0d9404d0362/57719e66-c5b1-466c-b4ff-7913976ad99e"
+					(reference "C16")
 					(unit 1)
 				)
@@
 		(in_pos_files yes)
 		(dnp no)
-		(property "Reference" "R6"
+		(property "Reference" "R14"
 			(at 125.984 87.63 90)
 			(show_name no)
@@
 				(path "/a968d2b9-0c0e-491c-a5a4-aacd8448ff64"
 					(reference "R6")
+					(unit 1)
+				)
+			)
+			(project "PS-PowerDistributionUnit"
+				(path "/eb16378f-e371-46a9-bfab-b0d9404d0362/57719e66-c5b1-466c-b4ff-7913976ad99e"
+					(reference "R14")
 					(unit 1)
 				)
@@
 		(in_pos_files yes)
 		(dnp no)
-		(property "Reference" "R3"
+		(property "Reference" "R10"
 			(at 67.31 54.61 90)
 			(show_name no)
@@
 				(path "/a968d2b9-0c0e-491c-a5a4-aacd8448ff64"
 					(reference "R3")
+					(unit 1)
+				)
+			)
+			(project "PS-PowerDistributionUnit"
+				(path "/eb16378f-e371-46a9-bfab-b0d9404d0362/57719e66-c5b1-466c-b4ff-7913976ad99e"
+					(reference "R10")
 					(unit 1)
 				)
@@
 		(in_pos_files yes)
 		(dnp no)
-		(property "Reference" "IC1"
+		(property "Reference" "IC2"
 			(at 75.184 73.66 0)
 			(show_name no)
@@
 				(path "/a968d2b9-0c0e-491c-a5a4-aacd8448ff64"
 					(reference "IC1")
+					(unit 1)
+				)
+			)
+			(project "PS-PowerDistributionUnit"
+				(path "/eb16378f-e371-46a9-bfab-b0d9404d0362/57719e66-c5b1-466c-b4ff-7913976ad99e"
+					(reference "IC2")
 					(unit 1)
 				)
@@
 		(in_pos_files yes)
 		(dnp no)
-		(property "Reference" "D2"
+		(property "Reference" "D21"
 			(at 17.272 51.054 90)
 			(show_name no)
@@
 				(path "/a968d2b9-0c0e-491c-a5a4-aacd8448ff64"
 					(reference "D2")
+					(unit 1)
+				)
+			)
+			(project "PS-PowerDistributionUnit"
+				(path "/eb16378f-e371-46a9-bfab-b0d9404d0362/57719e66-c5b1-466c-b4ff-7913976ad99e"
+					(reference "D21")
 					(unit 1)
 				)
@@
 				)
 			)
+			(project "PS-PowerDistributionUnit"
+				(path "/eb16378f-e371-46a9-bfab-b0d9404d0362/57719e66-c5b1-466c-b4ff-7913976ad99e"
+					(reference "Q1")
+					(unit 1)
+				)
+			)
 		)
 	)
@@
 		(in_pos_files yes)
 		(dnp no)
-		(property "Reference" "C4"
+		(property "Reference" "C19"
 			(at 54.864 62.23 0)
 			(show_name no)
@@
 				(path "/a968d2b9-0c0e-491c-a5a4-aacd8448ff64"
 					(reference "C4")
+					(unit 1)
+				)
+			)
+			(project "PS-PowerDistributionUnit"
+				(path "/eb16378f-e371-46a9-bfab-b0d9404d0362/57719e66-c5b1-466c-b4ff-7913976ad99e"
+					(reference "C19")
 					(unit 1)
 				)
@@
 		(in_pos_files yes)
 		(dnp no)
-		(property "Reference" "C5"
+		(property "Reference" "C20"
 			(at 112.395 49.5299 0)
 			(show_name no)
@@
 				(path "/a968d2b9-0c0e-491c-a5a4-aacd8448ff64"
 					(reference "C5")
+					(unit 1)
+				)
+			)
+			(project "PS-PowerDistributionUnit"
+				(path "/eb16378f-e371-46a9-bfab-b0d9404d0362/57719e66-c5b1-466c-b4ff-7913976ad99e"
+					(reference "C20")
 					(unit 1)
 				)
@@
 				)
 			)
+			(project "PS-PowerDistributionUnit"
+				(path "/eb16378f-e371-46a9-bfab-b0d9404d0362/57719e66-c5b1-466c-b4ff-7913976ad99e"
+					(reference "Q2")
+					(unit 1)
+				)
+			)
 		)
 	)
@@
 		(in_pos_files yes)
 		(dnp no)
-		(property "Reference" "R5"
+		(property "Reference" "R12"
 			(at 114.808 87.884 90)
 			(show_name no)
@@
 				(path "/a968d2b9-0c0e-491c-a5a4-aacd8448ff64"
 					(reference "R5")
+					(unit 1)
+				)
+			)
+			(project "PS-PowerDistributionUnit"
+				(path "/eb16378f-e371-46a9-bfab-b0d9404d0362/57719e66-c5b1-466c-b4ff-7913976ad99e"
+					(reference "R12")
 					(unit 1)
 				)
@@
 		(in_pos_files yes)
 		(dnp no)
-		(property "Reference" "D1"
+		(property "Reference" "D22"
 			(at 46.228 84.074 90)
 			(show_name no)
@@
 				(path "/a968d2b9-0c0e-491c-a5a4-aacd8448ff64"
 					(reference "D1")
+					(unit 1)
+				)
+			)
+			(project "PS-PowerDistributionUnit"
+				(path "/eb16378f-e371-46a9-bfab-b0d9404d0362/57719e66-c5b1-466c-b4ff-7913976ad99e"
+					(reference "D22")
 					(unit 1)
 				)
@@
 		(in_pos_files yes)
 		(dnp no)
-		(property "Reference" "C2"
+		(property "Reference" "C17"
 			(at 33.02 80.0099 0)
 			(show_name no)
@@
 				(path "/a968d2b9-0c0e-491c-a5a4-aacd8448ff64"
 					(reference "C2")
+					(unit 1)
+				)
+			)
+			(project "PS-PowerDistributionUnit"
+				(path "/eb16378f-e371-46a9-bfab-b0d9404d0362/57719e66-c5b1-466c-b4ff-7913976ad99e"
+					(reference "C17")
 					(unit 1)
 				)
@@
 		(in_pos_files yes)
 		(dnp no)
-		(property "Reference" "R4"
+		(property "Reference" "R11"
 			(at 114.3 79.248 90)
 			(show_name no)
@@
 				)
 			)
+			(project "PS-PowerDistributionUnit"
+				(path "/eb16378f-e371-46a9-bfab-b0d9404d0362/57719e66-c5b1-466c-b4ff-7913976ad99e"
+					(reference "R11")
+					(unit 1)
+				)
+			)
 		)
 	)
-	(sheet_instances
-		(path "/"
-			(page "1")
-		)
-	)
-	(embedded_fonts no)
 )

Commit message: discrete cs
Parts:
- renumbered C16 to C50, C17 to C51, C18 to C52, C19 to C53, C20 to C54, D21 to D46, D22 to D47, IC2 to IC10, R9 to R28, R10 to R29, R11 to R30, R12 to R31, R13 to R32, R14 to R33
Changed lines of the file:
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@@
 		(dnp no)
 		(fields_autoplaced yes)
-		(property "Reference" "C18"
+		(property "Reference" "C52"
 			(at 57.785 80.0099 0)
 			(show_name no)
@@
 			(project "PS-PowerDistributionUnit"
 				(path "/eb16378f-e371-46a9-bfab-b0d9404d0362/57719e66-c5b1-466c-b4ff-7913976ad99e"
-					(reference "C18")
+					(reference "C52")
 					(unit 1)
 				)
@@
 		(dnp no)
 		(fields_autoplaced yes)
-		(property "Reference" "R9"
+		(property "Reference" "R28"
 			(at 45.72 60.9599 0)
 			(show_name no)
@@
 			(project "PS-PowerDistributionUnit"
 				(path "/eb16378f-e371-46a9-bfab-b0d9404d0362/57719e66-c5b1-466c-b4ff-7913976ad99e"
-					(reference "R9")
+					(reference "R28")
 					(unit 1)
 				)
@@
 		(in_pos_files yes)
 		(dnp no)
-		(property "Reference" "R13"
+		(property "Reference" "R32"
 			(at 125.73 77.47 90)
 			(show_name no)
@@
 			(project "PS-PowerDistributionUnit"
 				(path "/eb16378f-e371-46a9-bfab-b0d9404d0362/57719e66-c5b1-466c-b4ff-7913976ad99e"
-					(reference "R13")
+					(reference "R32")
 					(unit 1)
 				)
@@
 		(in_pos_files yes)
 		(dnp no)
-		(property "Reference" "C16"
+		(property "Reference" "C50"
 			(at 38.1 49.5299 0)
 			(show_name no)
@@
 			(project "PS-PowerDistributionUnit"
 				(path "/eb16378f-e371-46a9-bfab-b0d9404d0362/57719e66-c5b1-466c-b4ff-7913976ad99e"
-					(reference "C16")
+					(reference "C50")
 					(unit 1)
 				)
@@
 		(in_pos_files yes)
 		(dnp no)
-		(property "Reference" "R14"
+		(property "Reference" "R33"
 			(at 125.984 87.63 90)
 			(show_name no)
@@
 			(project "PS-PowerDistributionUnit"
 				(path "/eb16378f-e371-46a9-bfab-b0d9404d0362/57719e66-c5b1-466c-b4ff-7913976ad99e"
-					(reference "R14")
+					(reference "R33")
 					(unit 1)
 				)
@@
 		(in_pos_files yes)
 		(dnp no)
-		(property "Reference" "R10"
+		(property "Reference" "R29"
 			(at 67.31 54.61 90)
 			(show_name no)
@@
 			(project "PS-PowerDistributionUnit"
 				(path "/eb16378f-e371-46a9-bfab-b0d9404d0362/57719e66-c5b1-466c-b4ff-7913976ad99e"
-					(reference "R10")
+					(reference "R29")
 					(unit 1)
 				)
@@
 		(in_pos_files yes)
 		(dnp no)
-		(property "Reference" "IC2"
+		(property "Reference" "IC10"
 			(at 75.184 73.66 0)
 			(show_name no)
@@
 			(project "PS-PowerDistributionUnit"
 				(path "/eb16378f-e371-46a9-bfab-b0d9404d0362/57719e66-c5b1-466c-b4ff-7913976ad99e"
-					(reference "IC2")
+					(reference "IC10")
 					(unit 1)
 				)
@@
 		(in_pos_files yes)
 		(dnp no)
-		(property "Reference" "D21"
+		(property "Reference" "D46"
 			(at 17.272 51.054 90)
 			(show_name no)
@@
 			(project "PS-PowerDistributionUnit"
 				(path "/eb16378f-e371-46a9-bfab-b0d9404d0362/57719e66-c5b1-466c-b4ff-7913976ad99e"
-					(reference "D21")
+					(reference "D46")
 					(unit 1)
 				)
@@
 		(in_pos_files yes)
 		(dnp no)
-		(property "Reference" "C19"
+		(property "Reference" "C53"
 			(at 54.864 62.23 0)
 			(show_name no)
@@
 			(project "PS-PowerDistributionUnit"
 				(path "/eb16378f-e371-46a9-bfab-b0d9404d0362/57719e66-c5b1-466c-b4ff-7913976ad99e"
-					(reference "C19")
+					(reference "C53")
 					(unit 1)
 				)
@@
 		(in_pos_files yes)
 		(dnp no)
-		(property "Reference" "C20"
+		(property "Reference" "C54"
 			(at 112.395 49.5299 0)
 			(show_name no)
@@
 			(project "PS-PowerDistributionUnit"
 				(path "/eb16378f-e371-46a9-bfab-b0d9404d0362/57719e66-c5b1-466c-b4ff-7913976ad99e"
-					(reference "C20")
+					(reference "C54")
 					(unit 1)
 				)
@@
 		(in_pos_files yes)
 		(dnp no)
-		(property "Reference" "R12"
+		(property "Reference" "R31"
 			(at 114.808 87.884 90)
 			(show_name no)
@@
 			(project "PS-PowerDistributionUnit"
 				(path "/eb16378f-e371-46a9-bfab-b0d9404d0362/57719e66-c5b1-466c-b4ff-7913976ad99e"
-					(reference "R12")
+					(reference "R31")
 					(unit 1)
 				)
@@
 		(in_pos_files yes)
 		(dnp no)
-		(property "Reference" "D22"
+		(property "Reference" "D47"
 			(at 46.228 84.074 90)
 			(show_name no)
@@
 			(project "PS-PowerDistributionUnit"
 				(path "/eb16378f-e371-46a9-bfab-b0d9404d0362/57719e66-c5b1-466c-b4ff-7913976ad99e"
-					(reference "D22")
+					(reference "D47")
 					(unit 1)
 				)
@@
 		(in_pos_files yes)
 		(dnp no)
-		(property "Reference" "C17"
+		(property "Reference" "C51"
 			(at 33.02 80.0099 0)
 			(show_name no)
@@
 			(project "PS-PowerDistributionUnit"
 				(path "/eb16378f-e371-46a9-bfab-b0d9404d0362/57719e66-c5b1-466c-b4ff-7913976ad99e"
-					(reference "C17")
+					(reference "C51")
 					(unit 1)
 				)
@@
 		(in_pos_files yes)
 		(dnp no)
-		(property "Reference" "R11"
+		(property "Reference" "R30"
 			(at 114.3 79.248 90)
 			(show_name no)
@@
 			(project "PS-PowerDistributionUnit"
 				(path "/eb16378f-e371-46a9-bfab-b0d9404d0362/57719e66-c5b1-466c-b4ff-7913976ad99e"
-					(reference "R11")
-					(unit 1)
-				)
+					(reference "R30")
+					(unit 1)
+				)
