File: hardware/PowerProtection.kicad_sch (KiCad schematic)
At the start: 16 parts, among them IC10 LM74502DDFR, Q1 PSMN012-100YS, Q2 PSMN012-100YS

Commit message: surahbi comment mostly done except led
Parts:
- renumbered C50 to C55, C51 to C56, C52 to C57, C53 to C58, C54 to C59, D46 to D48, D47 to D49, IC10 to IC11, Q1 to Q3, Q2 to Q4, R28 to R42, R29 to R50, R30 to R51, R31 to R52, R32 to R53, R33 to R54
Changed lines of the file:
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@@
 		(dnp no)
 		(fields_autoplaced yes)
-		(property "Reference" "C52"
+		(property "Reference" "C57"
 			(at 57.785 80.0099 0)
 			(show_name no)
@@
 		)
 		(instances
-			(project "PowerProtection"
-				(path "/a968d2b9-0c0e-491c-a5a4-aacd8448ff64"
-					(reference "C3")
-					(unit 1)
-				)
-			)
 			(project "PS-PowerDistributionUnit"
-				(path "/eb16378f-e371-46a9-bfab-b0d9404d0362/57719e66-c5b1-466c-b4ff-7913976ad99e"
-					(reference "C52")
+				(path "/eb16378f-e371-46a9-bfab-b0d9404d0362/e5e6ee2e-1d09-4fff-9eef-bc055f220fc3/b0246900-e267-4919-ada7-b46927cdce75"
+					(reference "C57")
 					(unit 1)
 				)
@@
 		(dnp no)
 		(fields_autoplaced yes)
-		(property "Reference" "R28"
+		(property "Reference" "R42"
 			(at 45.72 60.9599 0)
 			(show_name no)
@@
 		)
 		(instances
-			(project "PowerProtection"
-				(path "/a968d2b9-0c0e-491c-a5a4-aacd8448ff64"
-					(reference "R1")
-					(unit 1)
-				)
-			)
 			(project "PS-PowerDistributionUnit"
-				(path "/eb16378f-e371-46a9-bfab-b0d9404d0362/57719e66-c5b1-466c-b4ff-7913976ad99e"
-					(reference "R28")
+				(path "/eb16378f-e371-46a9-bfab-b0d9404d0362/e5e6ee2e-1d09-4fff-9eef-bc055f220fc3/b0246900-e267-4919-ada7-b46927cdce75"
+					(reference "R42")
 					(unit 1)
 				)
@@
 		(in_pos_files yes)
 		(dnp no)
-		(property "Reference" "R32"
+		(property "Reference" "R53"
 			(at 125.73 77.47 90)
 			(show_name no)
@@
 		)
 		(instances
-			(project "PowerProtection"
-				(path "/a968d2b9-0c0e-491c-a5a4-aacd8448ff64"
-					(reference "R7")
-					(unit 1)
-				)
-			)
 			(project "PS-PowerDistributionUnit"
-				(path "/eb16378f-e371-46a9-bfab-b0d9404d0362/57719e66-c5b1-466c-b4ff-7913976ad99e"
-					(reference "R32")
+				(path "/eb16378f-e371-46a9-bfab-b0d9404d0362/e5e6ee2e-1d09-4fff-9eef-bc055f220fc3/b0246900-e267-4919-ada7-b46927cdce75"
+					(reference "R53")
 					(unit 1)
 				)
@@
 		(in_pos_files yes)
 		(dnp no)
-		(property "Reference" "C50"
+		(property "Reference" "C55"
 			(at 38.1 49.5299 0)
 			(show_name no)
@@
 		)
 		(instances
-			(project "PowerProtection"
-				(path "/a968d2b9-0c0e-491c-a5a4-aacd8448ff64"
-					(reference "C1")
-					(unit 1)
-				)
-			)
 			(project "PS-PowerDistributionUnit"
-				(path "/eb16378f-e371-46a9-bfab-b0d9404d0362/57719e66-c5b1-466c-b4ff-7913976ad99e"
-					(reference "C50")
+				(path "/eb16378f-e371-46a9-bfab-b0d9404d0362/e5e6ee2e-1d09-4fff-9eef-bc055f220fc3/b0246900-e267-4919-ada7-b46927cdce75"
+					(reference "C55")
 					(unit 1)
 				)
@@
 		(in_pos_files yes)
 		(dnp no)
-		(property "Reference" "R33"
+		(property "Reference" "R54"
 			(at 125.984 87.63 90)
 			(show_name no)
@@
 		)
 		(instances
-			(project "PowerProtection"
-				(path "/a968d2b9-0c0e-491c-a5a4-aacd8448ff64"
-					(reference "R6")
-					(unit 1)
-				)
-			)
 			(project "PS-PowerDistributionUnit"
-				(path "/eb16378f-e371-46a9-bfab-b0d9404d0362/57719e66-c5b1-466c-b4ff-7913976ad99e"
-					(reference "R33")
+				(path "/eb16378f-e371-46a9-bfab-b0d9404d0362/e5e6ee2e-1d09-4fff-9eef-bc055f220fc3/b0246900-e267-4919-ada7-b46927cdce75"
+					(reference "R54")
 					(unit 1)
 				)
@@
 		(in_pos_files yes)
 		(dnp no)
-		(property "Reference" "R29"
+		(property "Reference" "R50"
 			(at 67.31 54.61 90)
 			(show_name no)
@@
 		)
 		(instances
-			(project "PowerProtection"
-				(path "/a968d2b9-0c0e-491c-a5a4-aacd8448ff64"
-					(reference "R3")
-					(unit 1)
-				)
-			)
 			(project "PS-PowerDistributionUnit"
-				(path "/eb16378f-e371-46a9-bfab-b0d9404d0362/57719e66-c5b1-466c-b4ff-7913976ad99e"
-					(reference "R29")
+				(path "/eb16378f-e371-46a9-bfab-b0d9404d0362/e5e6ee2e-1d09-4fff-9eef-bc055f220fc3/b0246900-e267-4919-ada7-b46927cdce75"
+					(reference "R50")
 					(unit 1)
 				)
@@
 		(in_pos_files yes)
 		(dnp no)
-		(property "Reference" "IC10"
+		(property "Reference" "IC11"
 			(at 75.184 73.66 0)
 			(show_name no)
@@
 		)
 		(instances
-			(project "PowerProtection"
-				(path "/a968d2b9-0c0e-491c-a5a4-aacd8448ff64"
-					(reference "IC1")
-					(unit 1)
-				)
-			)
 			(project "PS-PowerDistributionUnit"
-				(path "/eb16378f-e371-46a9-bfab-b0d9404d0362/57719e66-c5b1-466c-b4ff-7913976ad99e"
-					(reference "IC10")
+				(path "/eb16378f-e371-46a9-bfab-b0d9404d0362/e5e6ee2e-1d09-4fff-9eef-bc055f220fc3/b0246900-e267-4919-ada7-b46927cdce75"
+					(reference "IC11")
 					(unit 1)
 				)
@@
 		(in_pos_files yes)
 		(dnp no)
-		(property "Reference" "D46"
+		(property "Reference" "D48"
 			(at 17.272 51.054 90)
 			(show_name no)
@@
 		)
 		(instances
-			(project "PowerProtection"
-				(path "/a968d2b9-0c0e-491c-a5a4-aacd8448ff64"
-					(reference "D2")
-					(unit 1)
-				)
-			)
 			(project "PS-PowerDistributionUnit"
-				(path "/eb16378f-e371-46a9-bfab-b0d9404d0362/57719e66-c5b1-466c-b4ff-7913976ad99e"
-					(reference "D46")
+				(path "/eb16378f-e371-46a9-bfab-b0d9404d0362/e5e6ee2e-1d09-4fff-9eef-bc055f220fc3/b0246900-e267-4919-ada7-b46927cdce75"
+					(reference "D48")
 					(unit 1)
 				)
@@
 		(in_pos_files yes)
 		(dnp no)
-		(property "Reference" "Q1"
+		(property "Reference" "Q3"
 			(at 51.816 38.608 90)
 			(show_name no)
@@
 		)
 		(instances
-			(project "PowerProtection"
-				(path "/a968d2b9-0c0e-491c-a5a4-aacd8448ff64"
-					(reference "Q1")
-					(unit 1)
-				)
-			)
 			(project "PS-PowerDistributionUnit"
-				(path "/eb16378f-e371-46a9-bfab-b0d9404d0362/57719e66-c5b1-466c-b4ff-7913976ad99e"
-					(reference "Q1")
+				(path "/eb16378f-e371-46a9-bfab-b0d9404d0362/e5e6ee2e-1d09-4fff-9eef-bc055f220fc3/b0246900-e267-4919-ada7-b46927cdce75"
+					(reference "Q3")
 					(unit 1)
 				)
@@
 		(in_pos_files yes)
 		(dnp no)
-		(property "Reference" "C53"
+		(property "Reference" "C58"
 			(at 54.864 62.23 0)
 			(show_name no)
@@
 		)
 		(instances
-			(project "PowerProtection"
-				(path "/a968d2b9-0c0e-491c-a5a4-aacd8448ff64"
-					(reference "C4")
-					(unit 1)
-				)
-			)
 			(project "PS-PowerDistributionUnit"
-				(path "/eb16378f-e371-46a9-bfab-b0d9404d0362/57719e66-c5b1-466c-b4ff-7913976ad99e"
-					(reference "C53")
+				(path "/eb16378f-e371-46a9-bfab-b0d9404d0362/e5e6ee2e-1d09-4fff-9eef-bc055f220fc3/b0246900-e267-4919-ada7-b46927cdce75"
+					(reference "C58")
 					(unit 1)
 				)
@@
 		(in_pos_files yes)
 		(dnp no)
-		(property "Reference" "C54"
+		(property "Reference" "C59"
 			(at 112.395 49.5299 0)
 			(show_name no)
@@
 		)
 		(instances
-			(project "PowerProtection"
-				(path "/a968d2b9-0c0e-491c-a5a4-aacd8448ff64"
-					(reference "C5")
-					(unit 1)
-				)
-			)
 			(project "PS-PowerDistributionUnit"
-				(path "/eb16378f-e371-46a9-bfab-b0d9404d0362/57719e66-c5b1-466c-b4ff-7913976ad99e"
-					(reference "C54")
+				(path "/eb16378f-e371-46a9-bfab-b0d9404d0362/e5e6ee2e-1d09-4fff-9eef-bc055f220fc3/b0246900-e267-4919-ada7-b46927cdce75"
+					(reference "C59")
 					(unit 1)
 				)
@@
 		(in_pos_files yes)
 		(dnp no)
-		(property "Reference" "Q2"
+		(property "Reference" "Q4"
 			(at 98.298 39.116 90)
 			(show_name no)
@@
 		)
 		(instances
-			(project "PowerProtection"
-				(path "/a968d2b9-0c0e-491c-a5a4-aacd8448ff64"
-					(reference "Q2")
-					(unit 1)
-				)
-			)
 			(project "PS-PowerDistributionUnit"
-				(path "/eb16378f-e371-46a9-bfab-b0d9404d0362/57719e66-c5b1-466c-b4ff-7913976ad99e"
-					(reference "Q2")
+				(path "/eb16378f-e371-46a9-bfab-b0d9404d0362/e5e6ee2e-1d09-4fff-9eef-bc055f220fc3/b0246900-e267-4919-ada7-b46927cdce75"
+					(reference "Q4")
 					(unit 1)
 				)
@@
 		(in_pos_files yes)
 		(dnp no)
-		(property "Reference" "R31"
+		(property "Reference" "R52"
 			(at 114.808 87.884 90)
 			(show_name no)
@@
 		)
 		(instances
-			(project "PowerProtection"
-				(path "/a968d2b9-0c0e-491c-a5a4-aacd8448ff64"
-					(reference "R5")
-					(unit 1)
-				)
-			)
 			(project "PS-PowerDistributionUnit"
-				(path "/eb16378f-e371-46a9-bfab-b0d9404d0362/57719e66-c5b1-466c-b4ff-7913976ad99e"
-					(reference "R31")
+				(path "/eb16378f-e371-46a9-bfab-b0d9404d0362/e5e6ee2e-1d09-4fff-9eef-bc055f220fc3/b0246900-e267-4919-ada7-b46927cdce75"
+					(reference "R52")
 					(unit 1)
 				)
@@
 		(in_pos_files yes)
 		(dnp no)
-		(property "Reference" "D47"
+		(property "Reference" "D49"
 			(at 46.228 84.074 90)
 			(show_name no)
@@
 		)
 		(instances
-			(project "PowerProtection"
-				(path "/a968d2b9-0c0e-491c-a5a4-aacd8448ff64"
-					(reference "D1")
-					(unit 1)
-				)
-			)
 			(project "PS-PowerDistributionUnit"
-				(path "/eb16378f-e371-46a9-bfab-b0d9404d0362/57719e66-c5b1-466c-b4ff-7913976ad99e"
-					(reference "D47")
+				(path "/eb16378f-e371-46a9-bfab-b0d9404d0362/e5e6ee2e-1d09-4fff-9eef-bc055f220fc3/b0246900-e267-4919-ada7-b46927cdce75"
+					(reference "D49")
 					(unit 1)
 				)
@@
 		(in_pos_files yes)
 		(dnp no)
-		(property "Reference" "C51"
+		(property "Reference" "C56"
 			(at 33.02 80.0099 0)
 			(show_name no)
@@
 		)
 		(instances
-			(project "PowerProtection"
-				(path "/a968d2b9-0c0e-491c-a5a4-aacd8448ff64"
-					(reference "C2")
-					(unit 1)
-				)
-			)
 			(project "PS-PowerDistributionUnit"
-				(path "/eb16378f-e371-46a9-bfab-b0d9404d0362/57719e66-c5b1-466c-b4ff-7913976ad99e"
-					(reference "C51")
+				(path "/eb16378f-e371-46a9-bfab-b0d9404d0362/e5e6ee2e-1d09-4fff-9eef-bc055f220fc3/b0246900-e267-4919-ada7-b46927cdce75"
+					(reference "C56")
 					(unit 1)
 				)
@@
 		(in_pos_files yes)
 		(dnp no)
-		(property "Reference" "R30"
+		(property "Reference" "R51"
 			(at 114.3 79.248 90)
 			(show_name no)
@@
 		)
 		(instances
-			(project "PowerProtection"
-				(path "/a968d2b9-0c0e-491c-a5a4-aacd8448ff64"
-					(reference "R4")
+			(project "PS-PowerDistributionUnit"
+				(path "/eb16378f-e371-46a9-bfab-b0d9404d0362/e5e6ee2e-1d09-4fff-9eef-bc055f220fc3/b0246900-e267-4919-ada7-b46927cdce75"
+					(reference "R51")
 					(unit 1)
 				)
-			)
-			(project "PS-PowerDistributionUnit"
-				(path "/eb16378f-e371-46a9-bfab-b0d9404d0362/57719e66-c5b1-466c-b4ff-7913976ad99e"
-					(reference "R30")
-					(unit 1)
-				)
