File: hardware/PowerProtection.kicad_sch (KiCad schematic)
At the start: 16 parts, among them IC11 LM74502DDFR, Q3 PSMN012-100YS, Q4 PSMN012-100YS

Commit message: maybe added tvs
Parts:
- renumbered C58 to C10, C59 to C11, C55 to C7, C56 to C8, C57 to C9, D48 to D2, D49 to D3, IC11 to IC1, Q3 to Q1, Q4 to Q2, R42 to R19, R50 to R20, R51 to R21, R52 to R22, R53 to R23, R54 to R24
Changed lines of the file:
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@@
 		(dnp no)
 		(fields_autoplaced yes)
-		(property "Reference" "C57"
+		(property "Reference" "C9"
 			(at 57.785 80.0099 0)
 			(show_name no)
@@
 			(project "PS-PowerDistributionUnit"
 				(path "/eb16378f-e371-46a9-bfab-b0d9404d0362/e5e6ee2e-1d09-4fff-9eef-bc055f220fc3/b0246900-e267-4919-ada7-b46927cdce75"
-					(reference "C57")
+					(reference "C9")
 					(unit 1)
 				)
@@
 		(dnp no)
 		(fields_autoplaced yes)
-		(property "Reference" "R42"
+		(property "Reference" "R19"
 			(at 45.72 60.9599 0)
 			(show_name no)
@@
 			(project "PS-PowerDistributionUnit"
 				(path "/eb16378f-e371-46a9-bfab-b0d9404d0362/e5e6ee2e-1d09-4fff-9eef-bc055f220fc3/b0246900-e267-4919-ada7-b46927cdce75"
-					(reference "R42")
+					(reference "R19")
 					(unit 1)
 				)
@@
 		(in_pos_files yes)
 		(dnp no)
-		(property "Reference" "R53"
+		(property "Reference" "R23"
 			(at 125.73 77.47 90)
 			(show_name no)
@@
 			(project "PS-PowerDistributionUnit"
 				(path "/eb16378f-e371-46a9-bfab-b0d9404d0362/e5e6ee2e-1d09-4fff-9eef-bc055f220fc3/b0246900-e267-4919-ada7-b46927cdce75"
-					(reference "R53")
+					(reference "R23")
 					(unit 1)
 				)
@@
 		(in_pos_files yes)
 		(dnp no)
-		(property "Reference" "C55"
+		(property "Reference" "C7"
 			(at 38.1 49.5299 0)
 			(show_name no)
@@
 			(project "PS-PowerDistributionUnit"
 				(path "/eb16378f-e371-46a9-bfab-b0d9404d0362/e5e6ee2e-1d09-4fff-9eef-bc055f220fc3/b0246900-e267-4919-ada7-b46927cdce75"
-					(reference "C55")
+					(reference "C7")
 					(unit 1)
 				)
@@
 		(in_pos_files yes)
 		(dnp no)
-		(property "Reference" "R54"
+		(property "Reference" "R24"
 			(at 125.984 87.63 90)
 			(show_name no)
@@
 			(project "PS-PowerDistributionUnit"
 				(path "/eb16378f-e371-46a9-bfab-b0d9404d0362/e5e6ee2e-1d09-4fff-9eef-bc055f220fc3/b0246900-e267-4919-ada7-b46927cdce75"
-					(reference "R54")
+					(reference "R24")
 					(unit 1)
 				)
@@
 		(in_pos_files yes)
 		(dnp no)
-		(property "Reference" "R50"
+		(property "Reference" "R20"
 			(at 67.31 54.61 90)
 			(show_name no)
@@
 			(project "PS-PowerDistributionUnit"
 				(path "/eb16378f-e371-46a9-bfab-b0d9404d0362/e5e6ee2e-1d09-4fff-9eef-bc055f220fc3/b0246900-e267-4919-ada7-b46927cdce75"
-					(reference "R50")
+					(reference "R20")
 					(unit 1)
 				)
@@
 		(in_pos_files yes)
 		(dnp no)
-		(property "Reference" "IC11"
+		(property "Reference" "IC1"
 			(at 75.184 73.66 0)
 			(show_name no)
@@
 			(project "PS-PowerDistributionUnit"
 				(path "/eb16378f-e371-46a9-bfab-b0d9404d0362/e5e6ee2e-1d09-4fff-9eef-bc055f220fc3/b0246900-e267-4919-ada7-b46927cdce75"
-					(reference "IC11")
+					(reference "IC1")
 					(unit 1)
 				)
@@
 		(in_pos_files yes)
 		(dnp no)
-		(property "Reference" "D48"
+		(property "Reference" "D2"
 			(at 17.272 51.054 90)
 			(show_name no)
@@
 			(project "PS-PowerDistributionUnit"
 				(path "/eb16378f-e371-46a9-bfab-b0d9404d0362/e5e6ee2e-1d09-4fff-9eef-bc055f220fc3/b0246900-e267-4919-ada7-b46927cdce75"
-					(reference "D48")
+					(reference "D2")
 					(unit 1)
 				)
@@
 		(in_pos_files yes)
 		(dnp no)
-		(property "Reference" "Q3"
+		(property "Reference" "Q1"
 			(at 51.816 38.608 90)
 			(show_name no)
@@
 			(project "PS-PowerDistributionUnit"
 				(path "/eb16378f-e371-46a9-bfab-b0d9404d0362/e5e6ee2e-1d09-4fff-9eef-bc055f220fc3/b0246900-e267-4919-ada7-b46927cdce75"
-					(reference "Q3")
+					(reference "Q1")
 					(unit 1)
 				)
@@
 		(in_pos_files yes)
 		(dnp no)
-		(property "Reference" "C58"
+		(property "Reference" "C10"
 			(at 54.864 62.23 0)
 			(show_name no)
@@
 			(project "PS-PowerDistributionUnit"
 				(path "/eb16378f-e371-46a9-bfab-b0d9404d0362/e5e6ee2e-1d09-4fff-9eef-bc055f220fc3/b0246900-e267-4919-ada7-b46927cdce75"
-					(reference "C58")
+					(reference "C10")
 					(unit 1)
 				)
@@
 		(in_pos_files yes)
 		(dnp no)
-		(property "Reference" "C59"
+		(property "Reference" "C11"
 			(at 112.395 49.5299 0)
 			(show_name no)
@@
 			(project "PS-PowerDistributionUnit"
 				(path "/eb16378f-e371-46a9-bfab-b0d9404d0362/e5e6ee2e-1d09-4fff-9eef-bc055f220fc3/b0246900-e267-4919-ada7-b46927cdce75"
-					(reference "C59")
+					(reference "C11")
 					(unit 1)
 				)
@@
 		(in_pos_files yes)
 		(dnp no)
-		(property "Reference" "Q4"
+		(property "Reference" "Q2"
 			(at 98.298 39.116 90)
 			(show_name no)
@@
 			(project "PS-PowerDistributionUnit"
 				(path "/eb16378f-e371-46a9-bfab-b0d9404d0362/e5e6ee2e-1d09-4fff-9eef-bc055f220fc3/b0246900-e267-4919-ada7-b46927cdce75"
-					(reference "Q4")
+					(reference "Q2")
 					(unit 1)
 				)
@@
 		(in_pos_files yes)
 		(dnp no)
-		(property "Reference" "R52"
+		(property "Reference" "R22"
 			(at 114.808 87.884 90)
 			(show_name no)
@@
 			(project "PS-PowerDistributionUnit"
 				(path "/eb16378f-e371-46a9-bfab-b0d9404d0362/e5e6ee2e-1d09-4fff-9eef-bc055f220fc3/b0246900-e267-4919-ada7-b46927cdce75"
-					(reference "R52")
+					(reference "R22")
 					(unit 1)
 				)
@@
 		(in_pos_files yes)
 		(dnp no)
-		(property "Reference" "D49"
+		(property "Reference" "D3"
 			(at 46.228 84.074 90)
 			(show_name no)
@@
 			(project "PS-PowerDistributionUnit"
 				(path "/eb16378f-e371-46a9-bfab-b0d9404d0362/e5e6ee2e-1d09-4fff-9eef-bc055f220fc3/b0246900-e267-4919-ada7-b46927cdce75"
-					(reference "D49")
+					(reference "D3")
 					(unit 1)
 				)
@@
 		(in_pos_files yes)
 		(dnp no)
-		(property "Reference" "C56"
+		(property "Reference" "C8"
 			(at 33.02 80.0099 0)
 			(show_name no)
@@
 			(project "PS-PowerDistributionUnit"
 				(path "/eb16378f-e371-46a9-bfab-b0d9404d0362/e5e6ee2e-1d09-4fff-9eef-bc055f220fc3/b0246900-e267-4919-ada7-b46927cdce75"
-					(reference "C56")
+					(reference "C8")
 					(unit 1)
 				)
@@
 		(in_pos_files yes)
 		(dnp no)
-		(property "Reference" "R51"
+		(property "Reference" "R21"
 			(at 114.3 79.248 90)
 			(show_name no)
@@
 			(project "PS-PowerDistributionUnit"
 				(path "/eb16378f-e371-46a9-bfab-b0d9404d0362/e5e6ee2e-1d09-4fff-9eef-bc055f220fc3/b0246900-e267-4919-ada7-b46927cdce75"
-					(reference "R51")
+					(reference "R21")
 					(unit 1)
 				)

Commit message: changed resistor for spi stuff
Parts:
- renumbered R19 to R27, R20 to R28, R21 to R29, R22 to R30, R23 to R31, R24 to R32
Changed lines of the file:
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@@
 		(dnp no)
 		(fields_autoplaced yes)
-		(property "Reference" "R19"
+		(property "Reference" "R27"
 			(at 45.72 60.9599 0)
 			(show_name no)
@@
 			(project "PS-PowerDistributionUnit"
 				(path "/eb16378f-e371-46a9-bfab-b0d9404d0362/e5e6ee2e-1d09-4fff-9eef-bc055f220fc3/b0246900-e267-4919-ada7-b46927cdce75"
-					(reference "R19")
+					(reference "R27")
 					(unit 1)
 				)
@@
 		(in_pos_files yes)
 		(dnp no)
-		(property "Reference" "R23"
+		(property "Reference" "R31"
 			(at 125.73 77.47 90)
 			(show_name no)
@@
 			(project "PS-PowerDistributionUnit"
 				(path "/eb16378f-e371-46a9-bfab-b0d9404d0362/e5e6ee2e-1d09-4fff-9eef-bc055f220fc3/b0246900-e267-4919-ada7-b46927cdce75"
-					(reference "R23")
+					(reference "R31")
 					(unit 1)
 				)
@@
 		(in_pos_files yes)
 		(dnp no)
-		(property "Reference" "R24"
+		(property "Reference" "R32"
 			(at 125.984 87.63 90)
 			(show_name no)
@@
 			(project "PS-PowerDistributionUnit"
 				(path "/eb16378f-e371-46a9-bfab-b0d9404d0362/e5e6ee2e-1d09-4fff-9eef-bc055f220fc3/b0246900-e267-4919-ada7-b46927cdce75"
-					(reference "R24")
+					(reference "R32")
 					(unit 1)
 				)
@@
 		(in_pos_files yes)
 		(dnp no)
-		(property "Reference" "R20"
+		(property "Reference" "R28"
 			(at 67.31 54.61 90)
 			(show_name no)
@@
 			(project "PS-PowerDistributionUnit"
 				(path "/eb16378f-e371-46a9-bfab-b0d9404d0362/e5e6ee2e-1d09-4fff-9eef-bc055f220fc3/b0246900-e267-4919-ada7-b46927cdce75"
-					(reference "R20")
+					(reference "R28")
 					(unit 1)
 				)
@@
 		(in_pos_files yes)
 		(dnp no)
-		(property "Reference" "R22"
+		(property "Reference" "R30"
 			(at 114.808 87.884 90)
 			(show_name no)
@@
 			(project "PS-PowerDistributionUnit"
 				(path "/eb16378f-e371-46a9-bfab-b0d9404d0362/e5e6ee2e-1d09-4fff-9eef-bc055f220fc3/b0246900-e267-4919-ada7-b46927cdce75"
-					(reference "R22")
+					(reference "R30")
 					(unit 1)
 				)
@@
 		(in_pos_files yes)
 		(dnp no)
-		(property "Reference" "R21"
+		(property "Reference" "R29"
 			(at 114.3 79.248 90)
 			(show_name no)
@@
 			(project "PS-PowerDistributionUnit"
 				(path "/eb16378f-e371-46a9-bfab-b0d9404d0362/e5e6ee2e-1d09-4fff-9eef-bc055f220fc3/b0246900-e267-4919-ada7-b46927cdce75"
-					(reference "R21")
+					(reference "R29")
 					(unit 1)
 				)

Commit message: added p/n and footprints
Parts:
- C10: LCSC P/N MSASH168SB5103KTNA01 -> C6600162; P/N (none) -> MSASH168SB5103KTNA01
Changed lines of the file:
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@@
 			)
 		)
-		(property "LCSC P/N" "MSASH168SB5103KTNA01"
+		(property "LCSC P/N" "C6600162"
 			(at 60.96 63.5 0)
 			(hide yes)
+			(show_name no)
+			(do_not_autoplace no)
+			(effects
+				(font
+					(size 1.27 1.27)
+				)
+			)
+		)
+		(property "P/N" "MSASH168SB5103KTNA01"
+			(at 60.96 63.5 0)
+			(hide yes)

Commit message: added usb
Parts:
- removed D2: SMBJ30CD, Diode_SMD:D_SMB, symbol Device:D_Zener
- removed D3: SMAF4758A, LHRS_Passives:SODFL5026X125N, symbol Device:D_Zener
- removed R31: 10k, Resistor_SMD:R_0603_1608Metric_Pad0.98x0.95mm_HandSolder, symbol Device:R
- removed R32: 137k, Resistor_SMD:R_0603_1608Metric_Pad0.98x0.95mm_HandSolder, symbol Device:R
- added C8, C9: 0.1u, Capacitor_SMD:C_0603_1608Metric_Pad1.08x0.95mm_HandSolder, symbol Device:C
- added D2: SMBJ15CA, Diode_SMD:D_SMB, symbol lhrs_power:SMBJ15CA
- added D3: SMAF4758A, LHRS_Passives:SODFL5026X125N, symbol lhrs_power:SMAF4758A
- added R13: 100k, Resistor_SMD:R_0603_1608Metric_Pad0.98x0.95mm_HandSolder, symbol Device:R_US
- added R14: 15.8k, Resistor_SMD:R_0603_1608Metric_Pad0.98x0.95mm_HandSolder, symbol Device:R_US
- C6: renamed from C10; LCSC P/N C6600162 -> MSASH168SB5103KTNA01; P/N MSASH168SB5103KTNA01 -> (none)
- IC1: symbol LHRS_ICs:LM74502HDDFR -> lhrs_power:LM74502HDDFR
- R10: renamed from R28; symbol Device:R -> Device:R_US
- R11: renamed from R29; value 221k -> 100k; symbol Device:R -> Device:R_US
- R12: renamed from R30; value 10k -> 7.32k; symbol Device:R -> Device:R_US
- R9: renamed from R27; symbol Device:R -> Device:R_US
- renumbered C7 to C3, C8 to C4, C9 to C5, C11 to C7
Connections:
- net EN/UVLO: now also C9.2, R13.2, R14.2
- net GND: now also C8.1, C9.1, D2.1 (A1), D3.2 (A), R14.1
- net OV: now also C8.2
- net Vin: now also D2.2 (A2), R13.1
- net at C4.2, C5.1, IC1.5 (VS)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: now also D3.1 (K)
Other:
- note added: "Output of Python Calulations for Resistor Values"
- note removed: "1.235 is Enable/UVLO falling threshold on data sheet"
- note removed: "Overvoltage Protection: 29.03V Vovr = (R2 * Vov)/(R1 + R2) Vov = Vovr * (R1 + R2) / R2 28.875 = 1.25 * (221k + 10k) / 10k"
- moved on the sheet: C4, Q2

Commit message: layout starte but i want to play codename
Parts:
- C6: LCSC P/N MSASH168SB5103KTNA01 -> C6600162; P/N (none) -> MSASH168SB5103KTNA01
- C8, C9: LCSC P/N (none) -> C14663; P/N (none) -> MLASH168SB7104KTNA01
Changed lines of the file:
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@@
+			)
+		)
+		(property "LCSC P/N" "C14663"
+			(at 129.54 90.17 90)
+			(hide yes)
+			(show_name no)
+			(do_not_autoplace no)
+			(effects
+				(font
+					(size 1.27 1.27)
+				)
+			)
+		)
+		(property "P/N" "MLASH168SB7104KTNA01"
+			(at 129.54 90.17 90)
+			(hide yes)
+			(show_name no)
+			(do_not_autoplace no)
+			(effects
+				(font
+					(size 1.27 1.27)
+				)
 			)
 		)
@@
 			)
 		)
+		(property "LCSC P/N" "C14663"
+			(at 110.49 90.17 90)
+			(hide yes)
+			(show_name no)
+			(do_not_autoplace no)
+			(effects
+				(font
+					(size 1.27 1.27)
+				)
+			)
+		)
+		(property "P/N" "MLASH168SB7104KTNA01"
+			(at 110.49 90.17 90)
+			(hide yes)
+			(show_name no)
+			(do_not_autoplace no)
+			(effects
+				(font
+					(size 1.27 1.27)
+				)
+			)
+		)
 		(pin "2"
 		)
@@
 			)
 		)
-		(property "LCSC P/N" "MSASH168SB5103KTNA01"
+		(property "LCSC P/N" "C6600162"
 			(at 60.96 63.5 0)
 			(hide yes)
+			(show_name no)
+			(do_not_autoplace no)
+			(effects
+				(font
+					(size 1.27 1.27)
+				)
+			)
+		)
+		(property "P/N" "MSASH168SB5103KTNA01"
+			(at 60.96 63.5 0)
+			(hide yes)

Commit message: added pn
Parts:
- C3, C8, C9: LCSC P/N C14663 -> C1591; P/N MLASH168SB7104KTNA01 -> CL10B104KB8NNNC
- C4: P/N MLASU168SB5105KTNA01 -> CC0603KRX7R9BB105
- D3: LCSC P/N (none) -> C183490; P/N (none) -> SMAF4758A
- R11: LCSC P/N C2090661 -> C25803; P/N CRCW0603221KFKEA -> 0603WAF1003T5E
- R13: LCSC P/N C25804 -> C25803; P/N CRCW060310K0FKEI -> 0603WAF1003T5E
- R9: P/N CRCW060310K0FKEI -> 0603WAF1002T5E
Changed lines of the file:
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@@
 			)
 		)
-		(property "LCSC P/N" "C14663"
+		(property "LCSC P/N" "C1591"
 			(at 129.54 90.17 90)
 			(hide yes)
@@
 			)
 		)
-		(property "P/N" "MLASH168SB7104KTNA01"
+		(property "P/N" "CL10B104KB8NNNC"
 			(at 129.54 90.17 90)
 			(hide yes)
@@
 		)
 		(property "Description" "Zener diode"
+			(at 43.18 83.82 0)
+			(hide yes)
+			(show_name no)
+			(do_not_autoplace no)
+			(effects
+				(font
+					(size 1.27 1.27)
+				)
+			)
+		)
+		(property "P/N" "SMAF4758A"
+			(at 43.18 83.82 0)
+			(hide yes)
+			(show_name no)
+			(do_not_autoplace no)
+			(effects
+				(font
+					(size 1.27 1.27)
+				)
+			)
+		)
+		(property "LCSC P/N" "C183490"
 			(at 43.18 83.82 0)
 			(hide yes)
@@
 			)
 		)
-		(property "P/N" "CRCW060310K0FKEI"
+		(property "P/N" "0603WAF1002T5E"
 			(at 43.18 62.23 0)
 			(hide yes)
@@
 			)
 		)
-		(property "P/N" "MLASH168SB7104KTNA01"
+		(property "P/N" "CL10B104KB8NNNC"
 			(at 34.29 50.8 0)
 			(hide yes)
@@
 			)
 		)
-		(property "LCSC P/N" "C14663"
+		(property "LCSC P/N" "C1591"
 			(at 34.29 50.8 0)
 			(hide yes)
@@
 			)
 		)
-		(property "LCSC P/N" "C14663"
+		(property "LCSC P/N" "C1591"
 			(at 110.49 90.17 90)
 			(hide yes)
@@
 			)
 		)
-		(property "P/N" "MLASH168SB7104KTNA01"
+		(property "P/N" "CL10B104KB8NNNC"
 			(at 110.49 90.17 90)
 			(hide yes)
@@
 			)
 		)
-		(property "P/N" "MLASU168SB5105KTNA01"
+		(property "P/N" "CC0603KRX7R9BB105"
 			(at 32.385 86.36 0)
 			(hide yes)
@@
 			)
 		)
-		(property "P/N" "CRCW0603221KFKEA"
+		(property "P/N" "0603WAF1003T5E"
 			(at 115.57 77.47 0)
 			(hide yes)
@@
 			)
 		)
-		(property "LCSC P/N" "C2090661"
+		(property "LCSC P/N" "C25803"
 			(at 115.57 77.47 0)
 			(hide yes)
@@
 			)
 		)
-		(property "P/N" "CRCW060310K0FKEI"
+		(property "P/N" "0603WAF1003T5E"
 			(at 134.62 77.47 0)
 			(hide yes)
@@
 			)
 		)
-		(property "LCSC P/N" "C25804"
+		(property "LCSC P/N" "C25803"
 			(at 134.62 77.47 0)
 			(hide yes)
