File: hardware/48PinMCU.kicad_sch (KiCad schematic)
At the start: 29 parts, among them J1 SWD_Header_02x02, SW1 SW_SPDT, SW2 Reset, U1 STM32G431CBT6, Y1 Crystal

Commit message: discrete cs
Parts:
- renumbered C2 to C10, C9 to C11, C3 to C12, C14 to C13, C4 to C14, C10 to C15, C5 to C16, C12 to C17, C6 to C18, C13 to C19, C7 to C20, C8 to C21, C11 to C22, C15 to C23, C1 to C9, D16 to D19, D2 to D20, FB4 to FB2, J1 to J3, R2 to R10, R3 to R11, R1 to R7, R4 to R8, R5 to R9, SW2 to SW1, SW1 to SW2, U1 to U2
Changed lines of the file:
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@@
 		(dnp no)
 		(fields_autoplaced yes)
-		(property "Reference" "C12"
+		(property "Reference" "C17"
 			(at 204.597 57.4039 0)
 			(show_name no)
@@
 			(project "PS-PowerDistributionUnit"
 				(path "/eb16378f-e371-46a9-bfab-b0d9404d0362/36c8df72-7ede-452e-a2ec-09fdaf0ef78b"
-					(reference "C12")
+					(reference "C17")
 					(unit 1)
 				)
@@
 		(dnp no)
 		(fields_autoplaced yes)
-		(property "Reference" "R1"
+		(property "Reference" "R7"
 			(at 180.34 98.8059 0)
 			(show_name no)
@@
 			(project "PS-PowerDistributionUnit"
 				(path "/eb16378f-e371-46a9-bfab-b0d9404d0362/36c8df72-7ede-452e-a2ec-09fdaf0ef78b"
-					(reference "R1")
+					(reference "R7")
 					(unit 1)
 				)
@@
 		(dnp no)
 		(fields_autoplaced yes)
-		(property "Reference" "D16"
+		(property "Reference" "D19"
 			(at 241.3 106.1719 90)
 			(show_name no)
@@
 			(project "PS-PowerDistributionUnit"
 				(path "/eb16378f-e371-46a9-bfab-b0d9404d0362/36c8df72-7ede-452e-a2ec-09fdaf0ef78b"
-					(reference "D16")
+					(reference "D19")
 					(unit 1)
 				)
@@
 		(in_pos_files yes)
 		(dnp no)
-		(property "Reference" "C11"
+		(property "Reference" "C22"
 			(at 247.142 32.258 0)
 			(show_name no)
@@
 			(project "PS-PowerDistributionUnit"
 				(path "/eb16378f-e371-46a9-bfab-b0d9404d0362/36c8df72-7ede-452e-a2ec-09fdaf0ef78b"
-					(reference "C11")
+					(reference "C22")
 					(unit 1)
 				)
@@
 		(dnp no)
 		(fields_autoplaced yes)
-		(property "Reference" "R4"
+		(property "Reference" "R8"
 			(at 198.628 140.97 90)
 			(show_name no)
@@
 			(project "PS-PowerDistributionUnit"
 				(path "/eb16378f-e371-46a9-bfab-b0d9404d0362/36c8df72-7ede-452e-a2ec-09fdaf0ef78b"
-					(reference "R4")
+					(reference "R8")
 					(unit 1)
 				)
@@
 		(dnp no)
 		(fields_autoplaced yes)
-		(property "Reference" "FB4"
+		(property "Reference" "FB2"
 			(at 249.6312 47.117 90)
 			(show_name no)
@@
 			(project "PS-PowerDistributionUnit"
 				(path "/eb16378f-e371-46a9-bfab-b0d9404d0362/36c8df72-7ede-452e-a2ec-09fdaf0ef78b"
-					(reference "FB4")
+					(reference "FB2")
 					(unit 1)
 				)
@@
 		(dnp no)
 		(fields_autoplaced yes)
-		(property "Reference" "C10"
+		(property "Reference" "C15"
 			(at 189.992 57.4039 0)
 			(show_name no)
@@
 			(project "PS-PowerDistributionUnit"
 				(path "/eb16378f-e371-46a9-bfab-b0d9404d0362/36c8df72-7ede-452e-a2ec-09fdaf0ef78b"
-					(reference "C10")
+					(reference "C15")
 					(unit 1)
 				)
@@
 		(in_pos_files yes)
 		(dnp no)
-		(property "Reference" "R5"
+		(property "Reference" "R9"
 			(at 198.628 153.035 90)
 			(show_name no)
@@
 			(project "PS-PowerDistributionUnit"
 				(path "/eb16378f-e371-46a9-bfab-b0d9404d0362/36c8df72-7ede-452e-a2ec-09fdaf0ef78b"
-					(reference "R5")
+					(reference "R9")
 					(unit 1)
 				)
@@
 		(in_pos_files yes)
 		(dnp no)
-		(property "Reference" "R3"
+		(property "Reference" "R11"
 			(at 261.62 114.808 0)
 			(show_name no)
@@
 			(project "PS-PowerDistributionUnit"
 				(path "/eb16378f-e371-46a9-bfab-b0d9404d0362/36c8df72-7ede-452e-a2ec-09fdaf0ef78b"
-					(reference "R3")
+					(reference "R11")
 					(unit 1)
 				)
@@
 		(in_pos_files yes)
 		(dnp no)
-		(property "Reference" "C4"
+		(property "Reference" "C14"
 			(at 185.166 33.02 0)
 			(show_name no)
@@
 			(project "PS-PowerDistributionUnit"
 				(path "/eb16378f-e371-46a9-bfab-b0d9404d0362/36c8df72-7ede-452e-a2ec-09fdaf0ef78b"
-					(reference "C4")
+					(reference "C14")
 					(unit 1)
 				)
@@
 		(dnp no)
 		(fields_autoplaced yes)
-		(property "Reference" "C9"
+		(property "Reference" "C11"
 			(at 174.752 57.4039 0)
 			(show_name no)
@@
 			(project "PS-PowerDistributionUnit"
 				(path "/eb16378f-e371-46a9-bfab-b0d9404d0362/36c8df72-7ede-452e-a2ec-09fdaf0ef78b"
-					(reference "C9")
+					(reference "C11")
 					(unit 1)
 				)
@@
 		(in_pos_files yes)
 		(dnp no)
-		(property "Reference" "SW1"
+		(property "Reference" "SW2"
 			(at 236.982 99.314 0)
 			(show_name no)
@@
 			(project "PS-PowerDistributionUnit"
 				(path "/eb16378f-e371-46a9-bfab-b0d9404d0362/36c8df72-7ede-452e-a2ec-09fdaf0ef78b"
-					(reference "SW1")
+					(reference "SW2")
 					(unit 1)
 				)
@@
 		(dnp no)
 		(fields_autoplaced yes)
-		(property "Reference" "C15"
+		(property "Reference" "C23"
 			(at 257.937 57.277 0)
 			(show_name no)
@@
 			(project "PS-PowerDistributionUnit"
 				(path "/eb16378f-e371-46a9-bfab-b0d9404d0362/36c8df72-7ede-452e-a2ec-09fdaf0ef78b"
-					(reference "C15")
+					(reference "C23")
 					(unit 1)
 				)
@@
 		(dnp no)
 		(fields_autoplaced yes)
-		(property "Reference" "C1"
+		(property "Reference" "C9"
 			(at 143.002 81.28 90)
 			(show_name no)
@@
 			(project "PS-PowerDistributionUnit"
 				(path "/eb16378f-e371-46a9-bfab-b0d9404d0362/36c8df72-7ede-452e-a2ec-09fdaf0ef78b"
-					(reference "C1")
+					(reference "C9")
 					(unit 1)
 				)
@@
 		(in_pos_files yes)
 		(dnp no)
-		(property "Reference" "C6"
+		(property "Reference" "C18"
 			(at 210.82 32.766 0)
 			(show_name no)
@@
 			(project "PS-PowerDistributionUnit"
 				(path "/eb16378f-e371-46a9-bfab-b0d9404d0362/36c8df72-7ede-452e-a2ec-09fdaf0ef78b"
-					(reference "C6")
+					(reference "C18")
 					(unit 1)
 				)
@@
 		(in_pos_files yes)
 		(dnp no)
-		(property "Reference" "U1"
+		(property "Reference" "U2"
 			(at 74.422 63.5 0)
 			(show_name no)
@@
 			(project "PS-PowerDistributionUnit"
 				(path "/eb16378f-e371-46a9-bfab-b0d9404d0362/36c8df72-7ede-452e-a2ec-09fdaf0ef78b"
-					(reference "U1")
+					(reference "U2")
 					(unit 1)
 				)
@@
 		(dnp no)
 		(fields_autoplaced yes)
-		(property "Reference" "C7"
+		(property "Reference" "C20"
 			(at 224.028 33.0199 0)
 			(show_name no)
@@
 			(project "PS-PowerDistributionUnit"
 				(path "/eb16378f-e371-46a9-bfab-b0d9404d0362/36c8df72-7ede-452e-a2ec-09fdaf0ef78b"
-					(reference "C7")
+					(reference "C20")
 					(unit 1)
 				)
@@
 		(in_pos_files yes)
 		(dnp no)
-		(property "Reference" "C2"
+		(property "Reference" "C10"
 			(at 143.256 100.584 90)
 			(show_name no)
@@
 			(project "PS-PowerDistributionUnit"
 				(path "/eb16378f-e371-46a9-bfab-b0d9404d0362/36c8df72-7ede-452e-a2ec-09fdaf0ef78b"
-					(reference "C2")
+					(reference "C10")
 					(unit 1)
 				)
@@
 		(in_pos_files yes)
 		(dnp no)
-		(property "Reference" "R2"
+		(property "Reference" "R10"
 			(at 250.825 106.1719 0)
 			(show_name no)
@@
 			(project "PS-PowerDistributionUnit"
 				(path "/eb16378f-e371-46a9-bfab-b0d9404d0362/36c8df72-7ede-452e-a2ec-09fdaf0ef78b"
-					(reference "R2")
+					(reference "R10")
 					(unit 1)
 				)
@@
 		(in_pos_files yes)
 		(dnp no)
-		(property "Reference" "C3"
+		(property "Reference" "C12"
 			(at 173.99 33.02 0)
 			(show_name no)
@@
 			(project "PS-PowerDistributionUnit"
 				(path "/eb16378f-e371-46a9-bfab-b0d9404d0362/36c8df72-7ede-452e-a2ec-09fdaf0ef78b"
-					(reference "C3")
+					(reference "C12")
 					(unit 1)
 				)
@@
 		(in_pos_files yes)
 		(dnp no)
-		(property "Reference" "D2"
+		(property "Reference" "D20"
 			(at 265.684 109.982 90)
 			(show_name no)
@@
 			(project "PS-PowerDistributionUnit"
 				(path "/eb16378f-e371-46a9-bfab-b0d9404d0362/36c8df72-7ede-452e-a2ec-09fdaf0ef78b"
-					(reference "D2")
+					(reference "D20")
 					(unit 1)
 				)
@@
 		(dnp no)
 		(fields_autoplaced yes)
-		(property "Reference" "J1"
+		(property "Reference" "J3"
 			(at 185.928 140.97 0)
 			(show_name no)
@@
 			(project "PS-PowerDistributionUnit"
 				(path "/eb16378f-e371-46a9-bfab-b0d9404d0362/36c8df72-7ede-452e-a2ec-09fdaf0ef78b"
-					(reference "J1")
+					(reference "J3")
 					(unit 1)
 				)
@@
 		(in_pos_files yes)
 		(dnp no)
-		(property "Reference" "C13"
+		(property "Reference" "C19"
 			(at 217.17 56.642 0)
 			(show_name no)
@@
 			(project "PS-PowerDistributionUnit"
 				(path "/eb16378f-e371-46a9-bfab-b0d9404d0362/36c8df72-7ede-452e-a2ec-09fdaf0ef78b"
-					(reference "C13")
+					(reference "C19")
 					(unit 1)
 				)
@@
 		(in_pos_files yes)
 		(dnp no)
-		(property "Reference" "SW2"
+		(property "Reference" "SW1"
 			(at 185.8772 110.3376 90)
 			(show_name no)
@@
 			(project "PS-PowerDistributionUnit"
 				(path "/eb16378f-e371-46a9-bfab-b0d9404d0362/36c8df72-7ede-452e-a2ec-09fdaf0ef78b"
-					(reference "SW2")
+					(reference "SW1")
 					(unit 1)
 				)
@@
 		(in_pos_files yes)
 		(dnp no)
-		(property "Reference" "C14"
+		(property "Reference" "C13"
 			(at 169.164 109.728 0)
 			(show_name no)
@@
 			(project "PS-PowerDistributionUnit"
 				(path "/eb16378f-e371-46a9-bfab-b0d9404d0362/36c8df72-7ede-452e-a2ec-09fdaf0ef78b"
-					(reference "C14")
+					(reference "C13")
 					(unit 1)
 				)
@@
 		(in_pos_files yes)
 		(dnp no)
-		(property "Reference" "C5"
+		(property "Reference" "C16"
 			(at 197.358 33.02 0)
 			(show_name no)
@@
 			(project "PS-PowerDistributionUnit"
 				(path "/eb16378f-e371-46a9-bfab-b0d9404d0362/36c8df72-7ede-452e-a2ec-09fdaf0ef78b"
-					(reference "C5")
+					(reference "C16")
 					(unit 1)
 				)
@@
 		(in_pos_files yes)
 		(dnp no)
-		(property "Reference" "C8"
+		(property "Reference" "C21"
 			(at 233.172 32.004 0)
 			(show_name no)
@@
 			(project "PS-PowerDistributionUnit"
 				(path "/eb16378f-e371-46a9-bfab-b0d9404d0362/36c8df72-7ede-452e-a2ec-09fdaf0ef78b"
-					(reference "C8")
+					(reference "C21")
 					(unit 1)
 				)

Commit message: some reviews done
Parts:
- removed D19: D_TVS, Diode_SMD:D_SOD-323, symbol Device:D_TVS
- removed D20: LED, LED_SMD:LED_0201_0603Metric, symbol Device:LED
- removed R8: 22, Resistor_SMD:R_0603_1608Metric_Pad0.98x0.95mm_HandSolder, symbol Device:R
- removed U2: STM32G431CBT6, UTSVT_Special:48PinMCU, symbol 48PinMCU_Symbols:STM32G431CBT6
- added D19: RGB_LED, LHRS_Special:RGB_LED, symbol lhrs_special:RGB_LED
- added D20: TVS, Diode_SMD:D_SOD-323, symbol lhrs_misc:Boot_TVS
- added D60: LED, LED_SMD:LED_0603_1608Metric, symbol lhrs_misc:Blue_LED
- added J5: SWD, Connector_PinHeader_2.54mm:PinHeader_1x04_P2.54mm_Vertical, symbol Connector_Generic:Conn_01x04
- added R7, R93: 1k, Resistor_SMD:R_0603_1608Metric_Pad0.98x0.95mm_HandSolder, symbol Device:R
- added R91: 22, Resistor_SMD:R_0603_1608Metric_Pad0.98x0.95mm_HandSolder, symbol Device:R
- added R92: 10k, Resistor_SMD:R_0603_1608Metric_Pad0.98x0.95mm_HandSolder, symbol Device:R
- added U2: STM32G473CETx, LHRS_Special:48PinMCU, symbol lhrs_special:STM32G473CET6
- J3: value SWD_Header_02x02 -> SWD_Header; footprint 878320406:CONN04_878320406_MOL -> LHRS_Connectors:SWD_Conn; LSCS P/N (none) -> C17492485
- R10: value 10k -> 1k; LCSC P/N C25804 -> C21190; Mouser Part Number CRCW060310K0FKEI -> (none); P/N CRCW060310K0FKEI -> CRCW06031K00FKEI
- R11: value 1k -> 22; LCSC P/N C21190 -> C2930077; P/N CRCW06031K00FKEI -> FRC0603F22R0TS
- R9: value 22 -> 1k; LCSC P/N C2930077 -> C21190; P/N FRC0603F22R0TS -> CRCW06031K00FKEI
- SW1: footprint UTSVT_Special:BootSW -> LHRS_Special:TL3365AF180QG
- SW2: footprint BootSW:BootSW -> LHRS_Special:BootSW
- Y1: footprint Crystal:Crystal_SMD_Abracon_ABM3-2Pin_5.0x3.2mm -> LHRS_Passives:Crystal_SMD_Abracon_ABM3-2Pin_5.0x3.2mm
- renumbered R7 to R8
Connections:
- net BOOT0: now also R92.1, U2.45 (PB8-BOOT0); no longer R10.1
- net GND: now also C10.2, C9.1, R10.2, R9.2, D20.1 (A1), J5.2 (Pin_2), R7.2, R93.2, U2.23 (VSS), U2.35 (VSS), U2.47 (VSS); no longer C10.1, C9.2, R11.2
- net GNDA: now also U2.19 (VSSA)
- net PA0: now also D19.5, U2.8 (PA0-GPIO_BLUE)
- net PA1: now also D19.3, U2.9 (PA1_GPIO_RED)
- net PA10: now also U2.32 (PA10)
- net PA15: now also U2.39 (PA15)
- net PA2: now also D19.1, U2.10 (PA2-GPIO_GREEN)
- net PA3: now also U2.11 (PA3)
- net PA4: now also U2.12 (PA4)
- net PA5: now also U2.13 (PA5)
- net PA6: now also U2.14 (PA6)
- net PA7: now also U2.15 (PA7)
- net PA8: now also U2.30 (PA8)
- net PA9: now also U2.31 (PA9)
- net PB0: now also U2.16 (PB0)
- net PB1: now also U2.17 (PB1)
- net PB10: now also U2.22 (PB10)
- net PB11: now also U2.25 (PB11)
- net PB12: now also U2.26 (PB12)
- net PB13: now also U2.27 (PB13)
- net PB14: now also U2.28 (PB14)
- net PB15: now also U2.29 (PB15)
- net PB2: now also U2.18 (PB2)
- net PB3: now also U2.40 (PB3)
- net PB4: now also U2.41 (PB4)
- net PB5: now also U2.42 (PB5)
- net PB6: now also U2.43 (PB6)
- net PB7: now also U2.44 (PB7)
- net PB9: now also U2.46 (PB9)
- net PC13: now also U2.2 (PC13)
- net PC14: now also U2.3 (PC14-OSC32_IN)
- net PC15: now also U2.4 (PC15-OSC32_OUT)
- net SWCLK: now also R11.1, U2.38 (PA14)
- net SWDIO: now also R91.1, U2.37 (PA13); no longer R9.1
- net USB_DM: now also U2.33 (PA11)
- net USB_DP: now also U2.34 (PA12)
- net VDDA: now also U2.20 (VREF+), U2.21 (VDDA)
- net at Y1.1: now also C9.2, U2.5 (PF0-OSC_IN); no longer C10.2
- net at Y1.2: now also C10.1, U2.6 (PF1-OSC_OUT); no longer C9.1
- net at SW2.2 (B): now also D20.2 (A2), D60.2 (A), R92.2; no longer R10.2
- net at J3.3 (Pin_3): now also R11.2, J5.3 (Pin_3)
- net at J3.4 (Pin_4): now also J5.4 (Pin_4), R91.2; no longer R9.2
- net +3.3V renamed +3V3
- net +3V3: now also J5.1 (Pin_1), U2.1 (VBAT), U2.24 (VDD), U2.36 (VDD), U2.48 (VDD)
- net PG10-NRST renamed NRST
- net NRST: now also U2.7 (PG10-NRST)
- new net: D19.4, R9.1
- new net: D19.2, R7.1
- new net: D19.6, R10.1
- new net: D60.1 (K), R93.1
Other:
- note added: "*Place oscillator circuitry close to MCU"
- note added: "48 Pin MCU"
- note added: "BLUE"
- note added: "BOOT0 low -> Load into app BOOT0 high -> Load into bootloader"
- note added: "Beware, using PC13 - 15 as GPIOs ..."
- note added: "CLK"
- note added: "Conn"
- note added: "GREEN"
- note added: "IO"
- note added: "Pin Headers"
- note added: "Place these decoupling caps as close as possible to their respective leads."
- note added: "RED"
- note added: "RGB LED"
- note added: "Use PA0, PA1, PA2 to PWM RGB LED (TIM2_CH1, TIM2_CH2, TIM2_CH3)"
- note removed: "Place these decoupling caps as close as possible to their respective leads.(i.e. at C3-C8 at VDD, C11 at VBAT, C15 at VDDA, and C9-10 & C12-C13 at VDDA)."
- moved on the sheet: C13, R8, SW1

Commit message: comments addressed
Changed lines of the file:
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@@
 	(wire
 		(pts
-			(xy 132.08 36.83) (xy 121.92 36.83)
-		)
-		(stroke
-			(width 0)
-			(type default)
-		)
-	)
-	(wire
-		(pts
 			(xy 172.72 41.148) (xy 182.372 41.148)
 		)
@@
 	(wire
 		(pts
+			(xy 121.92 36.83) (xy 125.73 36.83)
+		)
+		(stroke
+			(width 0)
+			(type default)
+		)
+	)
+	(wire
+		(pts
 			(xy 100.33 21.59) (xy 101.6 21.59)
 		)
@@
 		)
 	)
-	(label "PA0"
-		(at 132.08 36.83 0)
-		(effects
-			(font
-				(size 1.27 1.27)
-			)
-			(justify left bottom)
-		)
-	)
 	(label "SWCLK"
 		(at 130.81 72.39 0)
@@
 		)
 	)
+	(hierarchical_label "PA0"
+		(shape bidirectional)
+		(at 125.73 36.83 0)
+		(effects
+			(font
+				(size 1.27 1.27)
+			)
+			(justify left)
+		)
+	)

Commit message: maybe added tvs
Parts:
- renumbered C9 to C16, C10 to C17, C11 to C18, C12 to C19, C13 to C20, C14 to C21, C15 to C22, C16 to C23, C17 to C24, C18 to C25, C19 to C26, C20 to C27, C21 to C28, C22 to C29, C23 to C30, D19 to D5, D20 to D6, D60 to D7, J3 to J7, J5 to J8, R7 to R28, R8 to R29, R9 to R30, R10 to R31, R11 to R32, R91 to R33, R92 to R34, R93 to R35, U2 to U3
