File: hardware/48PinMCU.kicad_sch (KiCad schematic)
At the start: 34 parts, among them J7 SWD_Header, J8 SWD, SW1 Reset, SW2 SW_SPDT, U3 STM32G473CETx, Y1 Crystal

Commit message: added p/n and footprints
Parts:
- J8: LCSC P/N (none) -> C2691448; P/N (none) -> PZ254V-11-04P
Changed lines of the file:
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@@
+			)
+		)
+		(property "LCSC P/N" "C2691448"
+			(at 250.19 153.67 0)
+			(hide yes)
+			(show_name no)
+			(do_not_autoplace no)
+			(effects
+				(font
+					(size 1.27 1.27)
+				)
+			)
+		)
+		(property "P/N" "PZ254V-11-04P"
+			(at 250.19 153.67 0)
+			(hide yes)
+			(show_name no)
+			(do_not_autoplace no)
+			(effects
+				(font
+					(size 1.27 1.27)
+				)
 			)
 		)

Commit message: added usb
Parts:
- R24: renamed from R40; LCSC P/N C2930077 -> C107701; P/N FRC0603F22R0TS -> RC0603FR-0722RL
- R25: renamed from R41; LCSC P/N C2930077 -> C107701; P/N FRC0603F22R0TS -> RC0603FR-0722RL
- renumbered J7 to J12, J8 to J13, R36 to R20, R37 to R21, R38 to R22, R39 to R23, R42 to R26, R43 to R27
Changed lines of the file:
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@@
 		(in_pos_files yes)
 		(dnp no)
-		(property "Reference" "R38"
+		(property "Reference" "R22"
 			(at 183.388 154.686 0)
 			(show_name no)
@@
 			(project "PS-PowerDistributionUnit"
 				(path "/eb16378f-e371-46a9-bfab-b0d9404d0362/293adb11-be79-4700-a618-5d6ae719b8c4"
-					(reference "R38")
+					(reference "R22")
 					(unit 1)
 				)
@@
 		(dnp no)
 		(fields_autoplaced yes)
-		(property "Reference" "R37"
+		(property "Reference" "R21"
 			(at 180.848 96.0119 0)
 			(show_name no)
@@
 			(project "PS-PowerDistributionUnit"
 				(path "/eb16378f-e371-46a9-bfab-b0d9404d0362/293adb11-be79-4700-a618-5d6ae719b8c4"
-					(reference "R37")
+					(reference "R21")
 					(unit 1)
 				)
@@
 		(in_pos_files yes)
 		(dnp no)
-		(property "Reference" "J7"
+		(property "Reference" "J12"
 			(at 259.334 135.89 0)
 			(show_name no)
@@
 			(project "PS-PowerDistributionUnit"
 				(path "/eb16378f-e371-46a9-bfab-b0d9404d0362/293adb11-be79-4700-a618-5d6ae719b8c4"
-					(reference "J7")
+					(reference "J12")
 					(unit 1)
 				)
@@
 		(in_pos_files yes)
 		(dnp no)
-		(property "Reference" "R39"
+		(property "Reference" "R23"
 			(at 191.008 154.686 0)
 			(show_name no)
@@
 			(project "PS-PowerDistributionUnit"
 				(path "/eb16378f-e371-46a9-bfab-b0d9404d0362/293adb11-be79-4700-a618-5d6ae719b8c4"
-					(reference "R39")
+					(reference "R23")
 					(unit 1)
 				)
@@
 		(in_pos_files yes)
 		(dnp no)
-		(property "Reference" "R43"
+		(property "Reference" "R27"
 			(at 259.588 110.236 0)
 			(show_name no)
@@
 			(project "PS-PowerDistributionUnit"
 				(path "/eb16378f-e371-46a9-bfab-b0d9404d0362/293adb11-be79-4700-a618-5d6ae719b8c4"
-					(reference "R43")
+					(reference "R27")
 					(unit 1)
 				)
@@
 		(in_pos_files yes)
 		(dnp no)
-		(property "Reference" "R36"
+		(property "Reference" "R20"
 			(at 175.768 154.686 0)
 			(show_name no)
@@
 			(project "PS-PowerDistributionUnit"
 				(path "/eb16378f-e371-46a9-bfab-b0d9404d0362/293adb11-be79-4700-a618-5d6ae719b8c4"
-					(reference "R36")
+					(reference "R20")
 					(unit 1)
 				)
@@
 		(in_pos_files yes)
 		(dnp no)
-		(property "Reference" "R41"
+		(property "Reference" "R25"
 			(at 226.06 149.225 90)
 			(show_name no)
@@
 			)
 		)
-		(property "LCSC P/N" "C2930077"
+		(property "LCSC P/N" "C107701"
 			(at 226.06 146.05 90)
 			(hide yes)
@@
 			)
 		)
-		(property "P/N" "FRC0603F22R0TS"
+		(property "P/N" "RC0603FR-0722RL"
 			(at 226.06 146.05 90)
 			(hide yes)
@@
 			(project "PS-PowerDistributionUnit"
 				(path "/eb16378f-e371-46a9-bfab-b0d9404d0362/293adb11-be79-4700-a618-5d6ae719b8c4"
-					(reference "R41")
+					(reference "R25")
 					(unit 1)
 				)
@@
 		(in_pos_files yes)
 		(dnp no)
-		(property "Reference" "R42"
+		(property "Reference" "R26"
 			(at 248.285 101.5999 0)
 			(show_name no)
@@
 			(project "PS-PowerDistributionUnit"
 				(path "/eb16378f-e371-46a9-bfab-b0d9404d0362/293adb11-be79-4700-a618-5d6ae719b8c4"
-					(reference "R42")
+					(reference "R26")
 					(unit 1)
 				)
@@
 		(in_pos_files yes)
 		(dnp no)
-		(property "Reference" "J8"
+		(property "Reference" "J13"
 			(at 254 151.384 0)
 			(show_name no)
@@
 			(project "PS-PowerDistributionUnit"
 				(path "/eb16378f-e371-46a9-bfab-b0d9404d0362/293adb11-be79-4700-a618-5d6ae719b8c4"
-					(reference "J8")
+					(reference "J13")
 					(unit 1)
 				)
@@
 		(dnp no)
 		(fields_autoplaced yes)
-		(property "Reference" "R40"
+		(property "Reference" "R24"
 			(at 226.06 137.795 90)
 			(show_name no)
@@
 			)
 		)
-		(property "LCSC P/N" "C2930077"
+		(property "LCSC P/N" "C107701"
 			(at 226.06 143.51 90)
 			(hide yes)
@@
 			)
 		)
-		(property "P/N" "FRC0603F22R0TS"
+		(property "P/N" "RC0603FR-0722RL"
 			(at 226.06 143.51 90)
 			(hide yes)
@@
 			(project "PS-PowerDistributionUnit"
 				(path "/eb16378f-e371-46a9-bfab-b0d9404d0362/293adb11-be79-4700-a618-5d6ae719b8c4"
-					(reference "R40")
+					(reference "R24")
 					(unit 1)
 				)
