File: hardware/5VBuck.kicad_sch (KiCad schematic)
At the start: 12 parts, among them U1 LMR51635XDDCR

Commit message: progress
Parts:
- L1: footprint Inductor_SMD:L_TDK_VLP8040 -> LHRS_Passives:SRN8040-101M; LCSC P/N C354639 -> C54563397; P/N CKCS8040-10uH/M -> SRN8040-101M
- U1: footprint utsvt_ics:DDC0006A-MFG -> LHRS_ICs:DDC0006A-MFG
- renumbered TP15 to TP?, TP13 to TP?, TP16 to TP?, TP14 to TP?
Changed lines of the file:
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@@
 			)
 		)
-		(property "Footprint" "Inductor_SMD:L_TDK_VLP8040"
+		(property "Footprint" "LHRS_Passives:SRN8040-101M"
 			(at 106.68 46.99 0)
 			(effects
@@
 			)
 		)
-		(property "LCSC P/N" "C354639"
+		(property "LCSC P/N" "C54563397"
 			(at 106.68 46.99 90)
 			(effects
@@
 			)
 		)
-		(property "P/N" "CKCS8040-10uH/M"
+		(property "P/N" "SRN8040-101M"
 			(at 106.68 46.99 90)
 			(effects
@@
 			)
 			(project "5VBuck"
-				(path "/ad6c7df0-eb90-4670-9aa8-3e2007aefc2d/ae63f0a9-78b8-4efb-b2ee-a2699a24d705"
-					(reference "L2")
-					(unit 1)
-				)
-			)
-			(project "5VBuck"
-				(path "/eb16378f-e371-46a9-bfab-b0d9404d0362/ed2d1a41-bb36-4dea-9776-a72024efc9f4"
+				(path "/eb16378f-e371-46a9-bfab-b0d9404d0362/c1ab43bd-83f5-4478-8cd1-f36b80c9eb92"
 					(reference "L1")
 					(unit 1)
@@
 			)
 			(project "5VBuck"
-				(path "/ad6c7df0-eb90-4670-9aa8-3e2007aefc2d/ae63f0a9-78b8-4efb-b2ee-a2699a24d705"
-					(reference "R33")
-					(unit 1)
-				)
-			)
-			(project "5VBuck"
-				(path "/eb16378f-e371-46a9-bfab-b0d9404d0362/ed2d1a41-bb36-4dea-9776-a72024efc9f4"
+				(path "/eb16378f-e371-46a9-bfab-b0d9404d0362/c1ab43bd-83f5-4478-8cd1-f36b80c9eb92"
 					(reference "R2")
 					(unit 1)
@@
 			)
 			(project "5VBuck"
-				(path "/ad6c7df0-eb90-4670-9aa8-3e2007aefc2d/ae63f0a9-78b8-4efb-b2ee-a2699a24d705"
-					(reference "C12")
-					(unit 1)
-				)
-			)
-			(project "5VBuck"
-				(path "/eb16378f-e371-46a9-bfab-b0d9404d0362/ed2d1a41-bb36-4dea-9776-a72024efc9f4"
+				(path "/eb16378f-e371-46a9-bfab-b0d9404d0362/c1ab43bd-83f5-4478-8cd1-f36b80c9eb92"
 					(reference "C1")
 					(unit 1)
@@
 		(on_board yes)
 		(dnp no)
-		(property "Reference" "TP15"
+		(property "Reference" "TP?"
 			(at 184.15 80.5179 0)
 			(effects
@@
 		)
 		(instances
+			(project "5VBuck"
+				(path "/1a7db697-3478-4f8f-a838-af5608c43196"
+					(reference "TP?")
+					(unit 1)
+				)
+			)
 			(project "PowerPath"
 				(path "/ad6c7df0-eb90-4670-9aa8-3e2007aefc2d/ae63f0a9-78b8-4efb-b2ee-a2699a24d705"
@@
 				)
 			)
-			(project "PowerPath"
-				(path "/eb16378f-e371-46a9-bfab-b0d9404d0362/ed2d1a41-bb36-4dea-9776-a72024efc9f4"
-					(reference "TP15")
+			(project "5VBuck"
+				(path "/eb16378f-e371-46a9-bfab-b0d9404d0362/c1ab43bd-83f5-4478-8cd1-f36b80c9eb92"
+					(reference "TP?")
 					(unit 1)
 				)
@@
 			)
 			(project "5VBuck"
-				(path "/ad6c7df0-eb90-4670-9aa8-3e2007aefc2d/ae63f0a9-78b8-4efb-b2ee-a2699a24d705"
-					(reference "C13")
-					(unit 1)
-				)
-			)
-			(project "5VBuck"
-				(path "/eb16378f-e371-46a9-bfab-b0d9404d0362/ed2d1a41-bb36-4dea-9776-a72024efc9f4"
+				(path "/eb16378f-e371-46a9-bfab-b0d9404d0362/c1ab43bd-83f5-4478-8cd1-f36b80c9eb92"
 					(reference "C2")
 					(unit 1)
@@
 			)
 		)
-		(property "Footprint" "utsvt_ics:DDC0006A-MFG"
+		(property "Footprint" "LHRS_ICs:DDC0006A-MFG"
 			(at 58.42 41.91 0)
 			(effects
@@
 			)
 			(project "5VBuck"
-				(path "/ad6c7df0-eb90-4670-9aa8-3e2007aefc2d/ae63f0a9-78b8-4efb-b2ee-a2699a24d705"
-					(reference "U4")
-					(unit 1)
-				)
-			)
-			(project "5VBuck"
-				(path "/eb16378f-e371-46a9-bfab-b0d9404d0362/ed2d1a41-bb36-4dea-9776-a72024efc9f4"
+				(path "/eb16378f-e371-46a9-bfab-b0d9404d0362/c1ab43bd-83f5-4478-8cd1-f36b80c9eb92"
 					(reference "U1")
 					(unit 1)
@@
 		(on_board yes)
 		(dnp no)
-		(property "Reference" "TP13"
+		(property "Reference" "TP?"
 			(at 171.45 80.5179 0)
 			(effects
@@
 		)
 		(instances
+			(project "5VBuck"
+				(path "/1a7db697-3478-4f8f-a838-af5608c43196"
+					(reference "TP?")
+					(unit 1)
+				)
+			)
 			(project ""
 				(path "/ad6c7df0-eb90-4670-9aa8-3e2007aefc2d/ae63f0a9-78b8-4efb-b2ee-a2699a24d705"
@@
 				)
 			)
-			(project ""
-				(path "/eb16378f-e371-46a9-bfab-b0d9404d0362/ed2d1a41-bb36-4dea-9776-a72024efc9f4"
-					(reference "TP13")
+			(project "5VBuck"
+				(path "/eb16378f-e371-46a9-bfab-b0d9404d0362/c1ab43bd-83f5-4478-8cd1-f36b80c9eb92"
+					(reference "TP?")
 					(unit 1)
 				)
@@
 			)
 			(project "5VBuck"
-				(path "/ad6c7df0-eb90-4670-9aa8-3e2007aefc2d/ae63f0a9-78b8-4efb-b2ee-a2699a24d705"
-					(reference "#FLG010")
-					(unit 1)
-				)
-			)
-			(project "5VBuck"
-				(path "/eb16378f-e371-46a9-bfab-b0d9404d0362/ed2d1a41-bb36-4dea-9776-a72024efc9f4"
+				(path "/eb16378f-e371-46a9-bfab-b0d9404d0362/c1ab43bd-83f5-4478-8cd1-f36b80c9eb92"
 					(reference "#FLG01")
 					(unit 1)
@@
 		(on_board yes)
 		(dnp no)
-		(property "Reference" "TP16"
+		(property "Reference" "TP?"
 			(at 184.15 93.2179 0)
 			(effects
@@
 		)
 		(instances
+			(project "5VBuck"
+				(path "/1a7db697-3478-4f8f-a838-af5608c43196"
+					(reference "TP?")
+					(unit 1)
+				)
+			)
 			(project "PowerPath"
 				(path "/ad6c7df0-eb90-4670-9aa8-3e2007aefc2d/ae63f0a9-78b8-4efb-b2ee-a2699a24d705"
@@
 				)
 			)
-			(project "PowerPath"
-				(path "/eb16378f-e371-46a9-bfab-b0d9404d0362/ed2d1a41-bb36-4dea-9776-a72024efc9f4"
-					(reference "TP16")
+			(project "5VBuck"
+				(path "/eb16378f-e371-46a9-bfab-b0d9404d0362/c1ab43bd-83f5-4478-8cd1-f36b80c9eb92"
+					(reference "TP?")
 					(unit 1)
 				)
@@
 			)
 			(project "5VBuck"
-				(path "/ad6c7df0-eb90-4670-9aa8-3e2007aefc2d/ae63f0a9-78b8-4efb-b2ee-a2699a24d705"
-					(reference "C15")
-					(unit 1)
-				)
-			)
-			(project "5VBuck"
-				(path "/eb16378f-e371-46a9-bfab-b0d9404d0362/ed2d1a41-bb36-4dea-9776-a72024efc9f4"
+				(path "/eb16378f-e371-46a9-bfab-b0d9404d0362/c1ab43bd-83f5-4478-8cd1-f36b80c9eb92"
 					(reference "C4")
 					(unit 1)
@@
 			)
 			(project "5VBuck"
-				(path "/ad6c7df0-eb90-4670-9aa8-3e2007aefc2d/ae63f0a9-78b8-4efb-b2ee-a2699a24d705"
-					(reference "#FLG011")
-					(unit 1)
-				)
-			)
-			(project "5VBuck"
-				(path "/eb16378f-e371-46a9-bfab-b0d9404d0362/ed2d1a41-bb36-4dea-9776-a72024efc9f4"
+				(path "/eb16378f-e371-46a9-bfab-b0d9404d0362/c1ab43bd-83f5-4478-8cd1-f36b80c9eb92"
 					(reference "#FLG02")
 					(unit 1)
@@
 			)
 			(project "5VBuck"
-				(path "/ad6c7df0-eb90-4670-9aa8-3e2007aefc2d/ae63f0a9-78b8-4efb-b2ee-a2699a24d705"
-					(reference "R32")
-					(unit 1)
-				)
-			)
-			(project "5VBuck"
-				(path "/eb16378f-e371-46a9-bfab-b0d9404d0362/ed2d1a41-bb36-4dea-9776-a72024efc9f4"
+				(path "/eb16378f-e371-46a9-bfab-b0d9404d0362/c1ab43bd-83f5-4478-8cd1-f36b80c9eb92"
 					(reference "R1")
 					(unit 1)
@@
 			)
 			(project "5VBuck"
-				(path "/ad6c7df0-eb90-4670-9aa8-3e2007aefc2d/ae63f0a9-78b8-4efb-b2ee-a2699a24d705"
-					(reference "C14")
-					(unit 1)
-				)
-			)
-			(project "5VBuck"
-				(path "/eb16378f-e371-46a9-bfab-b0d9404d0362/ed2d1a41-bb36-4dea-9776-a72024efc9f4"
+				(path "/eb16378f-e371-46a9-bfab-b0d9404d0362/c1ab43bd-83f5-4478-8cd1-f36b80c9eb92"
 					(reference "C3")
 					(unit 1)
@@
 		(on_board yes)
 		(dnp no)
-		(property "Reference" "TP14"
+		(property "Reference" "TP?"
 			(at 171.45 93.2179 0)
 			(effects
@@
 		)
 		(instances
+			(project "5VBuck"
+				(path "/1a7db697-3478-4f8f-a838-af5608c43196"
+					(reference "TP?")
+					(unit 1)
+				)
+			)
 			(project "PowerPath"
 				(path "/ad6c7df0-eb90-4670-9aa8-3e2007aefc2d/ae63f0a9-78b8-4efb-b2ee-a2699a24d705"
@@
 				)
 			)
-			(project "PowerPath"
-				(path "/eb16378f-e371-46a9-bfab-b0d9404d0362/ed2d1a41-bb36-4dea-9776-a72024efc9f4"
-					(reference "TP14")
-					(unit 1)
-				)
+			(project "5VBuck"
+				(path "/eb16378f-e371-46a9-bfab-b0d9404d0362/c1ab43bd-83f5-4478-8cd1-f36b80c9eb92"
+					(reference "TP?")
+					(unit 1)
+				)

Commit message: discrete cs
Parts:
- gave numbers to parts that had none: 4
- renumbered R1 to R3, R2 to R4
Changed lines of the file:
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@@
 		(dnp no)
 		(fields_autoplaced yes)
-		(property "Reference" "R2"
+		(property "Reference" "R4"
 			(at 170.18 49.5299 0)
 			(show_name no)
@@
 			(project "PS-PowerDistributionUnit"
 				(path "/eb16378f-e371-46a9-bfab-b0d9404d0362/c1ab43bd-83f5-4478-8cd1-f36b80c9eb92"
-					(reference "R2")
+					(reference "R4")
 					(unit 1)
 				)
@@
 		(in_pos_files yes)
 		(dnp no)
-		(property "Reference" "TP?"
+		(property "Reference" "TP4"
 			(at 184.15 80.5179 0)
 			(hide yes)
@@
 			(project "PS-PowerDistributionUnit"
 				(path "/eb16378f-e371-46a9-bfab-b0d9404d0362/c1ab43bd-83f5-4478-8cd1-f36b80c9eb92"
-					(reference "TP?")
+					(reference "TP4")
 					(unit 1)
 				)
@@
 		(in_pos_files yes)
 		(dnp no)
-		(property "Reference" "TP?"
+		(property "Reference" "TP2"
 			(at 171.45 80.5179 0)
 			(hide yes)
@@
 			(project "PS-PowerDistributionUnit"
 				(path "/eb16378f-e371-46a9-bfab-b0d9404d0362/c1ab43bd-83f5-4478-8cd1-f36b80c9eb92"
-					(reference "TP?")
+					(reference "TP2")
 					(unit 1)
 				)
@@
 		(in_pos_files yes)
 		(dnp no)
-		(property "Reference" "TP?"
+		(property "Reference" "TP5"
 			(at 184.15 93.2179 0)
 			(hide yes)
@@
 			(project "PS-PowerDistributionUnit"
 				(path "/eb16378f-e371-46a9-bfab-b0d9404d0362/c1ab43bd-83f5-4478-8cd1-f36b80c9eb92"
-					(reference "TP?")
+					(reference "TP5")
 					(unit 1)
 				)
@@
 		(dnp no)
 		(fields_autoplaced yes)
-		(property "Reference" "R1"
+		(property "Reference" "R3"
 			(at 170.18 41.9099 0)
 			(show_name no)
@@
 			(project "PS-PowerDistributionUnit"
 				(path "/eb16378f-e371-46a9-bfab-b0d9404d0362/c1ab43bd-83f5-4478-8cd1-f36b80c9eb92"
-					(reference "R1")
+					(reference "R3")
 					(unit 1)
 				)
@@
 		(in_pos_files yes)
 		(dnp no)
-		(property "Reference" "TP?"
+		(property "Reference" "TP3"
 			(at 171.45 93.2179 0)
 			(hide yes)
@@
 			(project "PS-PowerDistributionUnit"
 				(path "/eb16378f-e371-46a9-bfab-b0d9404d0362/c1ab43bd-83f5-4478-8cd1-f36b80c9eb92"
-					(reference "TP?")
-					(unit 1)
-				)
+					(reference "TP3")
+					(unit 1)
+				)

Commit message: maybe added tvs
Parts:
- renumbered C1 to C3, C2 to C4, C3 to C5, C4 to C6, R3 to R17, R4 to R18, U1 to U2
Changed lines of the file:
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@@
 		(dnp no)
 		(fields_autoplaced yes)
-		(property "Reference" "R4"
+		(property "Reference" "R18"
 			(at 170.18 49.5299 0)
 			(show_name no)
@@
 			(project "PS-PowerDistributionUnit"
 				(path "/eb16378f-e371-46a9-bfab-b0d9404d0362/e5e6ee2e-1d09-4fff-9eef-bc055f220fc3/e1446a70-7bd0-4041-85fa-90922de295c9"
-					(reference "R4")
+					(reference "R18")
 					(unit 1)
 				)
@@
 		(dnp no)
 		(fields_autoplaced yes)
-		(property "Reference" "C1"
+		(property "Reference" "C3"
 			(at 40.64 45.7262 0)
 			(show_name no)
@@
 			(project "PS-PowerDistributionUnit"
 				(path "/eb16378f-e371-46a9-bfab-b0d9404d0362/e5e6ee2e-1d09-4fff-9eef-bc055f220fc3/e1446a70-7bd0-4041-85fa-90922de295c9"
-					(reference "C1")
+					(reference "C3")
 					(unit 1)
 				)
@@
 		(in_pos_files yes)
 		(dnp no)
-		(property "Reference" "C2"
+		(property "Reference" "C4"
 			(at 100.838 40.64 0)
 			(show_name no)
@@
 			(project "PS-PowerDistributionUnit"
 				(path "/eb16378f-e371-46a9-bfab-b0d9404d0362/e5e6ee2e-1d09-4fff-9eef-bc055f220fc3/e1446a70-7bd0-4041-85fa-90922de295c9"
-					(reference "C2")
+					(reference "C4")
 					(unit 1)
 				)
@@
 		(dnp no)
 		(fields_autoplaced yes)
-		(property "Reference" "U1"
+		(property "Reference" "U2"
 			(at 73.66 31.75 0)
 			(show_name no)
@@
 			(project "PS-PowerDistributionUnit"
 				(path "/eb16378f-e371-46a9-bfab-b0d9404d0362/e5e6ee2e-1d09-4fff-9eef-bc055f220fc3/e1446a70-7bd0-4041-85fa-90922de295c9"
-					(reference "U1")
+					(reference "U2")
 					(unit 1)
 				)
@@
 		(dnp no)
 		(fields_autoplaced yes)
-		(property "Reference" "C4"
+		(property "Reference" "C6"
 			(at 129.54 49.5362 0)
 			(show_name no)
@@
 			(project "PS-PowerDistributionUnit"
 				(path "/eb16378f-e371-46a9-bfab-b0d9404d0362/e5e6ee2e-1d09-4fff-9eef-bc055f220fc3/e1446a70-7bd0-4041-85fa-90922de295c9"
-					(reference "C4")
+					(reference "C6")
 					(unit 1)
 				)
@@
 		(dnp no)
 		(fields_autoplaced yes)
-		(property "Reference" "R3"
+		(property "Reference" "R17"
 			(at 170.18 41.9099 0)
 			(show_name no)
@@
 			(project "PS-PowerDistributionUnit"
 				(path "/eb16378f-e371-46a9-bfab-b0d9404d0362/e5e6ee2e-1d09-4fff-9eef-bc055f220fc3/e1446a70-7bd0-4041-85fa-90922de295c9"
-					(reference "R3")
+					(reference "R17")
 					(unit 1)
 				)
@@
 		(dnp no)
 		(fields_autoplaced yes)
-		(property "Reference" "C3"
+		(property "Reference" "C5"
 			(at 118.11 49.5362 0)
 			(show_name no)
@@
 			(project "PS-PowerDistributionUnit"
 				(path "/eb16378f-e371-46a9-bfab-b0d9404d0362/e5e6ee2e-1d09-4fff-9eef-bc055f220fc3/e1446a70-7bd0-4041-85fa-90922de295c9"
-					(reference "C3")
-					(unit 1)
-				)
+					(reference "C5")
+					(unit 1)
+				)

Commit message: changed resistor for spi stuff
Parts:
- renumbered R17 to R25, R18 to R26
Changed lines of the file:
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@@
 		(dnp no)
 		(fields_autoplaced yes)
-		(property "Reference" "R18"
+		(property "Reference" "R26"
 			(at 170.18 49.5299 0)
 			(show_name no)
@@
 			(project "PS-PowerDistributionUnit"
 				(path "/eb16378f-e371-46a9-bfab-b0d9404d0362/e5e6ee2e-1d09-4fff-9eef-bc055f220fc3/e1446a70-7bd0-4041-85fa-90922de295c9"
-					(reference "R18")
+					(reference "R26")
 					(unit 1)
 				)
@@
 		(dnp no)
 		(fields_autoplaced yes)
-		(property "Reference" "R17"
+		(property "Reference" "R25"
 			(at 170.18 41.9099 0)
 			(show_name no)
@@
 			(project "PS-PowerDistributionUnit"
 				(path "/eb16378f-e371-46a9-bfab-b0d9404d0362/e5e6ee2e-1d09-4fff-9eef-bc055f220fc3/e1446a70-7bd0-4041-85fa-90922de295c9"
-					(reference "R17")
-					(unit 1)
-				)
+					(reference "R25")
+					(unit 1)
+				)
