File: hardware/CAN_Transceiver.kicad_sch (KiCad schematic)
At the start: 9 parts, among them IC1 TCAN3413DR

Commit message: discrete cs
Parts:
- renumbered D8 to D18, JP2 to JP1, R22 to R5, R23 to R6
Changed lines of the file:
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@@
 			)
 			(project "PS-PowerDistributionUnit"
-				(path "/eb16378f-e371-46a9-bfab-b0d9404d0362/9cd8cb49-32eb-4950-9e07-61b751a85545"
+				(path "/eb16378f-e371-46a9-bfab-b0d9404d0362/c3c07a99-aad4-4609-b9c8-47e591430794"
 					(reference "C6")
 					(unit 1)
@@
 			)
 			(project "PS-PowerDistributionUnit"
-				(path "/eb16378f-e371-46a9-bfab-b0d9404d0362/9cd8cb49-32eb-4950-9e07-61b751a85545"
+				(path "/eb16378f-e371-46a9-bfab-b0d9404d0362/c3c07a99-aad4-4609-b9c8-47e591430794"
 					(reference "C8")
 					(unit 1)
@@
 		(dnp no)
 		(fields_autoplaced yes)
-		(property "Reference" "JP2"
+		(property "Reference" "JP1"
 			(at 215.9 78.74 0)
 			(show_name no)
@@
 			)
 			(project "PS-PowerDistributionUnit"
-				(path "/eb16378f-e371-46a9-bfab-b0d9404d0362/9cd8cb49-32eb-4950-9e07-61b751a85545"
-					(reference "JP2")
+				(path "/eb16378f-e371-46a9-bfab-b0d9404d0362/c3c07a99-aad4-4609-b9c8-47e591430794"
+					(reference "JP1")
 					(unit 1)
 				)
@@
 			)
 			(project "PS-PowerDistributionUnit"
-				(path "/eb16378f-e371-46a9-bfab-b0d9404d0362/9cd8cb49-32eb-4950-9e07-61b751a85545"
+				(path "/eb16378f-e371-46a9-bfab-b0d9404d0362/c3c07a99-aad4-4609-b9c8-47e591430794"
 					(reference "C7")
 					(unit 1)
@@
 			)
 			(project "PS-PowerDistributionUnit"
-				(path "/eb16378f-e371-46a9-bfab-b0d9404d0362/9cd8cb49-32eb-4950-9e07-61b751a85545"
+				(path "/eb16378f-e371-46a9-bfab-b0d9404d0362/c3c07a99-aad4-4609-b9c8-47e591430794"
 					(reference "C5")
 					(unit 1)
@@
 		(in_pos_files yes)
 		(dnp no)
-		(property "Reference" "R23"
+		(property "Reference" "R6"
 			(at 201.93 80.01 90)
 			(show_name no)
@@
 			)
 			(project "PS-PowerDistributionUnit"
-				(path "/eb16378f-e371-46a9-bfab-b0d9404d0362/9cd8cb49-32eb-4950-9e07-61b751a85545"
-					(reference "R23")
+				(path "/eb16378f-e371-46a9-bfab-b0d9404d0362/c3c07a99-aad4-4609-b9c8-47e591430794"
+					(reference "R6")
 					(unit 1)
 				)
@@
 		(dnp no)
 		(fields_autoplaced yes)
-		(property "Reference" "D8"
+		(property "Reference" "D18"
 			(at 196.85 46.99 0)
 			(show_name no)
@@
 			)
 			(project "PS-PowerDistributionUnit"
-				(path "/eb16378f-e371-46a9-bfab-b0d9404d0362/9cd8cb49-32eb-4950-9e07-61b751a85545"
-					(reference "D8")
+				(path "/eb16378f-e371-46a9-bfab-b0d9404d0362/c3c07a99-aad4-4609-b9c8-47e591430794"
+					(reference "D18")
 					(unit 1)
 				)
@@
 			)
 			(project "PS-PowerDistributionUnit"
-				(path "/eb16378f-e371-46a9-bfab-b0d9404d0362/9cd8cb49-32eb-4950-9e07-61b751a85545"
+				(path "/eb16378f-e371-46a9-bfab-b0d9404d0362/c3c07a99-aad4-4609-b9c8-47e591430794"
 					(reference "IC1")
 					(unit 1)
@@
 		(in_pos_files yes)
 		(dnp no)
-		(property "Reference" "R22"
+		(property "Reference" "R5"
 			(at 176.53 80.01 90)
 			(show_name no)
@@
 			)
 			(project "PS-PowerDistributionUnit"
-				(path "/eb16378f-e371-46a9-bfab-b0d9404d0362/9cd8cb49-32eb-4950-9e07-61b751a85545"
-					(reference "R22")
-					(unit 1)
-				)
+				(path "/eb16378f-e371-46a9-bfab-b0d9404d0362/c3c07a99-aad4-4609-b9c8-47e591430794"
+					(reference "R5")
+					(unit 1)
+				)

Commit message: surahbi comment mostly done except led
Parts:
- renumbered C5 to C50, C6 to C51, C7 to C52, C8 to C53, D18 to D46, IC1 to IC10, JP1 to JP2, R5 to R18, R6 to R20
Changed lines of the file:
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@@
 		(in_pos_files yes)
 		(dnp no)
-		(property "Reference" "C6"
+		(property "Reference" "C51"
 			(at 76.2 73.66 0)
 			(show_name no)
@@
 		)
 		(instances
-			(project ""
-				(path "/69b823fd-c065-40ff-9bb9-c5835555f3eb/9d9eae1e-c713-4323-9845-a569cff8d5d3"
-					(reference "C6")
-					(unit 1)
-				)
-			)
-			(project "CAN_Transceiver"
-				(path "/a09f9696-80ee-4697-8aaa-225f287b667b"
-					(reference "C2")
-					(unit 1)
-				)
-			)
 			(project "PS-PowerDistributionUnit"
-				(path "/eb16378f-e371-46a9-bfab-b0d9404d0362/c3c07a99-aad4-4609-b9c8-47e591430794"
-					(reference "C6")
+				(path "/eb16378f-e371-46a9-bfab-b0d9404d0362/2ee5fe6f-603f-4929-8596-ad2cbd26bff6/94c71f3c-d4af-48d6-8a1b-560875efeb40"
+					(reference "C51")
 					(unit 1)
 				)
@@
 		(in_pos_files yes)
 		(dnp no)
-		(property "Reference" "C8"
+		(property "Reference" "C53"
 			(at 194.564 88.646 0)
 			(show_name no)
@@
 		)
 		(instances
-			(project ""
-				(path "/69b823fd-c065-40ff-9bb9-c5835555f3eb/9d9eae1e-c713-4323-9845-a569cff8d5d3"
-					(reference "C8")
-					(unit 1)
-				)
-			)
-			(project "CAN_Transceiver"
-				(path "/a09f9696-80ee-4697-8aaa-225f287b667b"
-					(reference "C4")
-					(unit 1)
-				)
-			)
 			(project "PS-PowerDistributionUnit"
-				(path "/eb16378f-e371-46a9-bfab-b0d9404d0362/c3c07a99-aad4-4609-b9c8-47e591430794"
-					(reference "C8")
+				(path "/eb16378f-e371-46a9-bfab-b0d9404d0362/2ee5fe6f-603f-4929-8596-ad2cbd26bff6/94c71f3c-d4af-48d6-8a1b-560875efeb40"
+					(reference "C53")
 					(unit 1)
 				)
@@
 		(dnp no)
 		(fields_autoplaced yes)
-		(property "Reference" "JP1"
+		(property "Reference" "JP2"
 			(at 215.9 78.74 0)
 			(show_name no)
@@
 		)
 		(instances
-			(project ""
-				(path "/69b823fd-c065-40ff-9bb9-c5835555f3eb/9d9eae1e-c713-4323-9845-a569cff8d5d3"
+			(project "PS-PowerDistributionUnit"
+				(path "/eb16378f-e371-46a9-bfab-b0d9404d0362/2ee5fe6f-603f-4929-8596-ad2cbd26bff6/94c71f3c-d4af-48d6-8a1b-560875efeb40"
 					(reference "JP2")
-					(unit 1)
-				)
-			)
-			(project ""
-				(path "/81d906df-a099-480a-8398-28a8e913d125"
-					(reference "JP1")
-					(unit 1)
-				)
-			)
-			(project "CAN_Transceiver"
-				(path "/a09f9696-80ee-4697-8aaa-225f287b667b"
-					(reference "JP1")
-					(unit 1)
-				)
-			)
-			(project "PS-PowerDistributionUnit"
-				(path "/eb16378f-e371-46a9-bfab-b0d9404d0362/c3c07a99-aad4-4609-b9c8-47e591430794"
-					(reference "JP1")
 					(unit 1)
 				)
@@
 		(in_pos_files yes)
 		(dnp no)
-		(property "Reference" "C7"
+		(property "Reference" "C52"
 			(at 88.138 73.66 0)
 			(show_name no)
@@
 		)
 		(instances
-			(project ""
-				(path "/69b823fd-c065-40ff-9bb9-c5835555f3eb/9d9eae1e-c713-4323-9845-a569cff8d5d3"
-					(reference "C7")
-					(unit 1)
-				)
-			)
-			(project "CAN_Transceiver"
-				(path "/a09f9696-80ee-4697-8aaa-225f287b667b"
-					(reference "C3")
-					(unit 1)
-				)
-			)
 			(project "PS-PowerDistributionUnit"
-				(path "/eb16378f-e371-46a9-bfab-b0d9404d0362/c3c07a99-aad4-4609-b9c8-47e591430794"
-					(reference "C7")
+				(path "/eb16378f-e371-46a9-bfab-b0d9404d0362/2ee5fe6f-603f-4929-8596-ad2cbd26bff6/94c71f3c-d4af-48d6-8a1b-560875efeb40"
+					(reference "C52")
 					(unit 1)
 				)
@@
 		(in_pos_files yes)
 		(dnp no)
-		(property "Reference" "C5"
+		(property "Reference" "C50"
 			(at 65.278 73.66 0)
 			(show_name no)
@@
 		)
 		(instances
-			(project ""
-				(path "/69b823fd-c065-40ff-9bb9-c5835555f3eb/9d9eae1e-c713-4323-9845-a569cff8d5d3"
-					(reference "C5")
-					(unit 1)
-				)
-			)
-			(project ""
-				(path "/81d906df-a099-480a-8398-28a8e913d125"
-					(reference "C1")
-					(unit 1)
-				)
-			)
-			(project "CAN_Transceiver"
-				(path "/a09f9696-80ee-4697-8aaa-225f287b667b"
-					(reference "C1")
-					(unit 1)
-				)
-			)
 			(project "PS-PowerDistributionUnit"
-				(path "/eb16378f-e371-46a9-bfab-b0d9404d0362/c3c07a99-aad4-4609-b9c8-47e591430794"
-					(reference "C5")
+				(path "/eb16378f-e371-46a9-bfab-b0d9404d0362/2ee5fe6f-603f-4929-8596-ad2cbd26bff6/94c71f3c-d4af-48d6-8a1b-560875efeb40"
+					(reference "C50")
 					(unit 1)
 				)
@@
 		(in_pos_files yes)
 		(dnp no)
-		(property "Reference" "R6"
+		(property "Reference" "R20"
 			(at 201.93 80.01 90)
 			(show_name no)
@@
 		)
 		(instances
-			(project "kk36984"
-				(path "/69b823fd-c065-40ff-9bb9-c5835555f3eb/9d9eae1e-c713-4323-9845-a569cff8d5d3"
-					(reference "R23")
-					(unit 1)
-				)
-			)
-			(project "CAN_Transceiver"
-				(path "/a09f9696-80ee-4697-8aaa-225f287b667b"
-					(reference "R2")
-					(unit 1)
-				)
-			)
 			(project "PS-PowerDistributionUnit"
-				(path "/eb16378f-e371-46a9-bfab-b0d9404d0362/c3c07a99-aad4-4609-b9c8-47e591430794"
-					(reference "R6")
+				(path "/eb16378f-e371-46a9-bfab-b0d9404d0362/2ee5fe6f-603f-4929-8596-ad2cbd26bff6/94c71f3c-d4af-48d6-8a1b-560875efeb40"
+					(reference "R20")
 					(unit 1)
 				)
@@
 		(dnp no)
 		(fields_autoplaced yes)
-		(property "Reference" "D18"
+		(property "Reference" "D46"
 			(at 196.85 46.99 0)
 			(show_name no)
@@
 		)
 		(instances
-			(project ""
-				(path "/69b823fd-c065-40ff-9bb9-c5835555f3eb/9d9eae1e-c713-4323-9845-a569cff8d5d3"
-					(reference "D8")
-					(unit 1)
-				)
-			)
-			(project "CAN_Transceiver"
-				(path "/a09f9696-80ee-4697-8aaa-225f287b667b"
-					(reference "D1")
-					(unit 1)
-				)
-			)
 			(project "PS-PowerDistributionUnit"
-				(path "/eb16378f-e371-46a9-bfab-b0d9404d0362/c3c07a99-aad4-4609-b9c8-47e591430794"
-					(reference "D18")
+				(path "/eb16378f-e371-46a9-bfab-b0d9404d0362/2ee5fe6f-603f-4929-8596-ad2cbd26bff6/94c71f3c-d4af-48d6-8a1b-560875efeb40"
+					(reference "D46")
 					(unit 1)
 				)
@@
 		(dnp no)
 		(fields_autoplaced yes)
-		(property "Reference" "IC1"
+		(property "Reference" "IC10"
 			(at 128.27 63.5 0)
 			(show_name no)
@@
 		)
 		(instances
-			(project ""
-				(path "/69b823fd-c065-40ff-9bb9-c5835555f3eb/9d9eae1e-c713-4323-9845-a569cff8d5d3"
-					(reference "IC1")
-					(unit 1)
-				)
-			)
-			(project "CAN_Transceiver"
-				(path "/a09f9696-80ee-4697-8aaa-225f287b667b"
-					(reference "IC1")
-					(unit 1)
-				)
-			)
 			(project "PS-PowerDistributionUnit"
-				(path "/eb16378f-e371-46a9-bfab-b0d9404d0362/c3c07a99-aad4-4609-b9c8-47e591430794"
-					(reference "IC1")
+				(path "/eb16378f-e371-46a9-bfab-b0d9404d0362/2ee5fe6f-603f-4929-8596-ad2cbd26bff6/94c71f3c-d4af-48d6-8a1b-560875efeb40"
+					(reference "IC10")
 					(unit 1)
 				)
@@
 		(in_pos_files yes)
 		(dnp no)
-		(property "Reference" "R5"
+		(property "Reference" "R18"
 			(at 176.53 80.01 90)
 			(show_name no)
@@
 		)
 		(instances
-			(project ""
-				(path "/69b823fd-c065-40ff-9bb9-c5835555f3eb/9d9eae1e-c713-4323-9845-a569cff8d5d3"
-					(reference "R22")
+			(project "PS-PowerDistributionUnit"
+				(path "/eb16378f-e371-46a9-bfab-b0d9404d0362/2ee5fe6f-603f-4929-8596-ad2cbd26bff6/94c71f3c-d4af-48d6-8a1b-560875efeb40"
+					(reference "R18")
 					(unit 1)
 				)
-			)
-			(project ""
-				(path "/81d906df-a099-480a-8398-28a8e913d125"
-					(reference "R1")
-					(unit 1)
-				)
-			)
-			(project "CAN_Transceiver"
-				(path "/a09f9696-80ee-4697-8aaa-225f287b667b"
-					(reference "R1")
-					(unit 1)
-				)
-			)
-			(project "PS-PowerDistributionUnit"
-				(path "/eb16378f-e371-46a9-bfab-b0d9404d0362/c3c07a99-aad4-4609-b9c8-47e591430794"
-					(reference "R5")
-					(unit 1)
-				)

Commit message: maybe added tvs
Parts:
- renumbered C50 to C12, C51 to C13, C52 to C14, C53 to C15, D46 to D4, IC10 to IC2, JP2 to JP1, R18 to R26, R20 to R27
Changed lines of the file:
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@@
 		(in_pos_files yes)
 		(dnp no)
-		(property "Reference" "C51"
+		(property "Reference" "C13"
 			(at 76.2 73.66 0)
 			(show_name no)
@@
 			(project "PS-PowerDistributionUnit"
 				(path "/eb16378f-e371-46a9-bfab-b0d9404d0362/2ee5fe6f-603f-4929-8596-ad2cbd26bff6/94c71f3c-d4af-48d6-8a1b-560875efeb40"
-					(reference "C51")
+					(reference "C13")
 					(unit 1)
 				)
@@
 		(in_pos_files yes)
 		(dnp no)
-		(property "Reference" "C53"
+		(property "Reference" "C15"
 			(at 194.564 88.646 0)
 			(show_name no)
@@
 			(project "PS-PowerDistributionUnit"
 				(path "/eb16378f-e371-46a9-bfab-b0d9404d0362/2ee5fe6f-603f-4929-8596-ad2cbd26bff6/94c71f3c-d4af-48d6-8a1b-560875efeb40"
-					(reference "C53")
+					(reference "C15")
 					(unit 1)
 				)
@@
 		(dnp no)
 		(fields_autoplaced yes)
-		(property "Reference" "JP2"
+		(property "Reference" "JP1"
 			(at 215.9 78.74 0)
 			(show_name no)
@@
 			(project "PS-PowerDistributionUnit"
 				(path "/eb16378f-e371-46a9-bfab-b0d9404d0362/2ee5fe6f-603f-4929-8596-ad2cbd26bff6/94c71f3c-d4af-48d6-8a1b-560875efeb40"
-					(reference "JP2")
+					(reference "JP1")
 					(unit 1)
 				)
@@
 		(in_pos_files yes)
 		(dnp no)
-		(property "Reference" "C52"
+		(property "Reference" "C14"
 			(at 88.138 73.66 0)
 			(show_name no)
@@
 			(project "PS-PowerDistributionUnit"
 				(path "/eb16378f-e371-46a9-bfab-b0d9404d0362/2ee5fe6f-603f-4929-8596-ad2cbd26bff6/94c71f3c-d4af-48d6-8a1b-560875efeb40"
-					(reference "C52")
+					(reference "C14")
 					(unit 1)
 				)
@@
 		(in_pos_files yes)
 		(dnp no)
-		(property "Reference" "C50"
+		(property "Reference" "C12"
 			(at 65.278 73.66 0)
 			(show_name no)
@@
 			(project "PS-PowerDistributionUnit"
 				(path "/eb16378f-e371-46a9-bfab-b0d9404d0362/2ee5fe6f-603f-4929-8596-ad2cbd26bff6/94c71f3c-d4af-48d6-8a1b-560875efeb40"
-					(reference "C50")
+					(reference "C12")
 					(unit 1)
 				)
@@
 		(in_pos_files yes)
 		(dnp no)
-		(property "Reference" "R20"
+		(property "Reference" "R27"
 			(at 201.93 80.01 90)
 			(show_name no)
@@
 			(project "PS-PowerDistributionUnit"
 				(path "/eb16378f-e371-46a9-bfab-b0d9404d0362/2ee5fe6f-603f-4929-8596-ad2cbd26bff6/94c71f3c-d4af-48d6-8a1b-560875efeb40"
-					(reference "R20")
+					(reference "R27")
 					(unit 1)
 				)
@@
 		(dnp no)
 		(fields_autoplaced yes)
-		(property "Reference" "D46"
+		(property "Reference" "D4"
 			(at 196.85 46.99 0)
 			(show_name no)
@@
 			(project "PS-PowerDistributionUnit"
 				(path "/eb16378f-e371-46a9-bfab-b0d9404d0362/2ee5fe6f-603f-4929-8596-ad2cbd26bff6/94c71f3c-d4af-48d6-8a1b-560875efeb40"
-					(reference "D46")
+					(reference "D4")
 					(unit 1)
 				)
@@
 		(dnp no)
 		(fields_autoplaced yes)
-		(property "Reference" "IC10"
+		(property "Reference" "IC2"
 			(at 128.27 63.5 0)
 			(show_name no)
@@
 			(project "PS-PowerDistributionUnit"
 				(path "/eb16378f-e371-46a9-bfab-b0d9404d0362/2ee5fe6f-603f-4929-8596-ad2cbd26bff6/94c71f3c-d4af-48d6-8a1b-560875efeb40"
-					(reference "IC10")
+					(reference "IC2")
 					(unit 1)
 				)
@@
 		(in_pos_files yes)
 		(dnp no)
-		(property "Reference" "R18"
+		(property "Reference" "R26"
 			(at 176.53 80.01 90)
 			(show_name no)
@@
 			(project "PS-PowerDistributionUnit"
 				(path "/eb16378f-e371-46a9-bfab-b0d9404d0362/2ee5fe6f-603f-4929-8596-ad2cbd26bff6/94c71f3c-d4af-48d6-8a1b-560875efeb40"
-					(reference "R18")
+					(reference "R26")
 					(unit 1)
 				)

Commit message: changed resistor for spi stuff
Parts:
- renumbered R26 to R34, R27 to R35
Changed lines of the file:
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@@
 		(in_pos_files yes)
 		(dnp no)
-		(property "Reference" "R27"
+		(property "Reference" "R35"
 			(at 201.93 80.01 90)
 			(show_name no)
@@
 			(project "PS-PowerDistributionUnit"
 				(path "/eb16378f-e371-46a9-bfab-b0d9404d0362/2ee5fe6f-603f-4929-8596-ad2cbd26bff6/94c71f3c-d4af-48d6-8a1b-560875efeb40"
-					(reference "R27")
+					(reference "R35")
 					(unit 1)
 				)
@@
 		(in_pos_files yes)
 		(dnp no)
-		(property "Reference" "R26"
+		(property "Reference" "R34"
 			(at 176.53 80.01 90)
 			(show_name no)
@@
 			(project "PS-PowerDistributionUnit"
 				(path "/eb16378f-e371-46a9-bfab-b0d9404d0362/2ee5fe6f-603f-4929-8596-ad2cbd26bff6/94c71f3c-d4af-48d6-8a1b-560875efeb40"
-					(reference "R26")
+					(reference "R34")
 					(unit 1)
 				)
