File: hardware/CAN_Transceiver.kicad_sch (KiCad schematic)
At the start: 9 parts, among them IC2 TCAN3413DR

Commit message: added p/n and footprints
Parts:
- JP1: LCSC P/N (none) -> C492401; P/N (none) -> PZ254V-11-02P
Changed lines of the file:
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@@
+			)
+		)
+		(property "LCSC P/N" "C492401"
+			(at 215.9 85.09 0)
+			(hide yes)
+			(show_name no)
+			(do_not_autoplace no)
+			(effects
+				(font
+					(size 1.27 1.27)
+				)
+			)
+		)
+		(property "P/N" "PZ254V-11-02P"
+			(at 215.9 85.09 0)
+			(hide yes)
+			(show_name no)
+			(do_not_autoplace no)
+			(effects
+				(font
+					(size 1.27 1.27)
+				)
 			)
 		)

Commit message: added usb
Parts:
- D4: footprint UTSVT_Passives:CDSOT23-T24CAN -> LHRS_Passives:CDSOT23-T24CAN
- IC2: footprint UTSVT_Passives:TCAN3413DR -> LHRS_Passives:TCAN3413DR
- renumbered R34 to R18, R35 to R19
Changed lines of the file:
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@@
 		(in_pos_files yes)
 		(dnp no)
-		(property "Reference" "R35"
+		(property "Reference" "R19"
 			(at 201.93 80.01 90)
 			(show_name no)
@@
 			(project "PS-PowerDistributionUnit"
 				(path "/eb16378f-e371-46a9-bfab-b0d9404d0362/2ee5fe6f-603f-4929-8596-ad2cbd26bff6/94c71f3c-d4af-48d6-8a1b-560875efeb40"
-					(reference "R35")
+					(reference "R19")
 					(unit 1)
 				)
@@
 			)
 		)
-		(property "Footprint" "UTSVT_Passives:CDSOT23-T24CAN"
+		(property "Footprint" "LHRS_Passives:CDSOT23-T24CAN"
 			(at 204.47 149.53 0)
 			(hide yes)
@@
 			)
 		)
-		(property "Footprint" "UTSVT_Passives:TCAN3413DR"
+		(property "Footprint" "LHRS_Passives:TCAN3413DR"
 			(at 140.97 166.04 0)
 			(hide yes)
@@
 		(in_pos_files yes)
 		(dnp no)
-		(property "Reference" "R34"
+		(property "Reference" "R18"
 			(at 176.53 80.01 90)
 			(show_name no)
@@
 			(project "PS-PowerDistributionUnit"
 				(path "/eb16378f-e371-46a9-bfab-b0d9404d0362/2ee5fe6f-603f-4929-8596-ad2cbd26bff6/94c71f3c-d4af-48d6-8a1b-560875efeb40"
-					(reference "R34")
+					(reference "R18")
 					(unit 1)
 				)

Commit message: layout starte but i want to play codename
Parts:
- renumbered C12 to C14, C13 to C15, C14 to C16, C15 to C17, R18 to R17, R19 to R18
Changed lines of the file:
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@@
 		(in_pos_files yes)
 		(dnp no)
-		(property "Reference" "C13"
+		(property "Reference" "C15"
 			(at 76.2 73.66 0)
 			(show_name no)
@@
 			(project "PS-PowerDistributionUnit"
 				(path "/eb16378f-e371-46a9-bfab-b0d9404d0362/2ee5fe6f-603f-4929-8596-ad2cbd26bff6/94c71f3c-d4af-48d6-8a1b-560875efeb40"
-					(reference "C13")
+					(reference "C15")
 					(unit 1)
 				)
@@
 		(in_pos_files yes)
 		(dnp no)
-		(property "Reference" "C15"
+		(property "Reference" "C17"
 			(at 194.564 88.646 0)
 			(show_name no)
@@
 			(project "PS-PowerDistributionUnit"
 				(path "/eb16378f-e371-46a9-bfab-b0d9404d0362/2ee5fe6f-603f-4929-8596-ad2cbd26bff6/94c71f3c-d4af-48d6-8a1b-560875efeb40"
-					(reference "C15")
+					(reference "C17")
 					(unit 1)
 				)
@@
 		(in_pos_files yes)
 		(dnp no)
-		(property "Reference" "C14"
+		(property "Reference" "C16"
 			(at 88.138 73.66 0)
 			(show_name no)
@@
 			(project "PS-PowerDistributionUnit"
 				(path "/eb16378f-e371-46a9-bfab-b0d9404d0362/2ee5fe6f-603f-4929-8596-ad2cbd26bff6/94c71f3c-d4af-48d6-8a1b-560875efeb40"
-					(reference "C14")
+					(reference "C16")
 					(unit 1)
 				)
@@
 		(in_pos_files yes)
 		(dnp no)
-		(property "Reference" "C12"
+		(property "Reference" "C14"
 			(at 65.278 73.66 0)
 			(show_name no)
@@
 			(project "PS-PowerDistributionUnit"
 				(path "/eb16378f-e371-46a9-bfab-b0d9404d0362/2ee5fe6f-603f-4929-8596-ad2cbd26bff6/94c71f3c-d4af-48d6-8a1b-560875efeb40"
-					(reference "C12")
+					(reference "C14")
 					(unit 1)
 				)
@@
 		(in_pos_files yes)
 		(dnp no)
-		(property "Reference" "R19"
+		(property "Reference" "R18"
 			(at 201.93 80.01 90)
 			(show_name no)
@@
 			(project "PS-PowerDistributionUnit"
 				(path "/eb16378f-e371-46a9-bfab-b0d9404d0362/2ee5fe6f-603f-4929-8596-ad2cbd26bff6/94c71f3c-d4af-48d6-8a1b-560875efeb40"
-					(reference "R19")
+					(reference "R18")
 					(unit 1)
 				)
@@
 		(in_pos_files yes)
 		(dnp no)
-		(property "Reference" "R18"
+		(property "Reference" "R17"
 			(at 176.53 80.01 90)
 			(show_name no)
@@
 			(project "PS-PowerDistributionUnit"
 				(path "/eb16378f-e371-46a9-bfab-b0d9404d0362/2ee5fe6f-603f-4929-8596-ad2cbd26bff6/94c71f3c-d4af-48d6-8a1b-560875efeb40"
-					(reference "R18")
+					(reference "R17")
 					(unit 1)
 				)

Commit message: added pn
Parts:
- C15, C16, C17: LCSC P/N C14663 -> C1591; P/N MLASH168SB7104KTNA01 -> CL10B104KB8NNNC
Changed lines of the file:
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@@
 			)
 		)
-		(property "LCSC P/N" "C14663"
+		(property "LCSC P/N" "C1591"
 			(at 73.66 74.93 0)
 			(hide yes)
@@
 			)
 		)
-		(property "P/N" "MLASH168SB7104KTNA01"
+		(property "P/N" "CL10B104KB8NNNC"
 			(at 73.66 74.93 0)
 			(hide yes)
@@
 			)
 		)
-		(property "LCSC P/N" "C14663"
+		(property "LCSC P/N" "C1591"
 			(at 189.23 88.9 0)
 			(hide yes)
@@
 			)
 		)
-		(property "P/N" "MLASH168SB7104KTNA01"
+		(property "P/N" "CL10B104KB8NNNC"
 			(at 189.23 88.9 0)
 			(hide yes)
@@
 			)
 		)
-		(property "LCSC P/N" "C14663"
+		(property "LCSC P/N" "C1591"
 			(at 85.09 74.93 0)
 			(hide yes)
@@
 			)
 		)
-		(property "P/N" "MLASH168SB7104KTNA01"
+		(property "P/N" "CL10B104KB8NNNC"
 			(at 85.09 74.93 0)
 			(hide yes)
