File: hardware/HSS_Pair.kicad_sch (KiCad schematic)
At the start: 23 parts, among them IC8 TPS2HCS08AQPWPRQ1

Commit message: maybe added tvs
Parts:
- C31: renamed from C28; LCSC P/N (none) -> C106851
- C32: renamed from C6; LCSC P/N (none) -> C100040
- C33: renamed from C47; LCSC P/N (none) -> C696901
- C34: renamed from C32; LCSC P/N (none) -> C5254613
- C35: renamed from C62; LCSC P/N (none) -> C14663
- C36: renamed from C67; LCSC P/N (none) -> C14663
- D10: renamed from D39; footprint (none) -> LED_SMD:LED_0201_0603Metric; LCSC P/N (none) -> C84263
- D11: renamed from D26; LCSC P/N (none) -> C428853
- D12: renamed from D24; LCSC P/N (none) -> C428853
- D8: renamed from D41; LCSC P/N (none) -> C428853
- D9: renamed from D61; footprint (none) -> LED_SMD:LED_0201_0603Metric; LCSC P/N (none) -> C84263
- R36: renamed from R77; LCSC P/N (none) -> C313648
- R37: renamed from R15; LCSC P/N (none) -> C25804
- R42: renamed from R70; LCSC P/N (none) -> C21190
- R43: renamed from R96; LCSC P/N (none) -> C23162
- R44: renamed from R12; LCSC P/N (none) -> C23162
- renumbered F3 to F2, F6 to F3, IC8 to IC3, R28 to R38, R35 to R39, R47 to R40, R58 to R41

Commit message: changed resistor for spi stuff
Parts:
- removed R38, R40, R41: 22, symbol Device:R
- renumbered R36 to R44, R37 to R45, R39 to R46, R42 to R47, R43 to R48, R44 to R49
Connections:
- net SPI_CS: now also IC3.15 (NCS)
- net SPI_MOSI: now also IC3.13 (SDI)
- net SPI_SCLK: now also IC3.16 (SCLK)

Commit message: what i did during matrices made it pretty
Parts:
- added R11: 4.7k, symbol Device:R
- added R12, R80: 10k, symbol Device:R
- added R81: 22, symbol Device:R
- added TP11: TestPoint, symbol Connector:TestPoint
Connections:
- net +24V_HSS: now also TP11.1
- net +3V3: now also R11.1, R80.1
- net FLT_WAKE: now also R11.2, R12.1, R12.2
- net SPI_CS: now also R80.2, R81.1, R81.2
- net SPI_MISO renamed MISO
- net SPI_MOSI renamed MOSI
- net SPI_SCLK renamed SCLK
Other:
- note added: "CS protection"
- note added: "FLT_WAKE protection"
- note added: "Resistor should be placed close to where it is driven for SPI whether its near the MCU or HSS"
- moved on the sheet: C31, C32, C33, C35, C36, D10, D11, D12, D8, D9, F2, F3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

Commit message: before update design block
Parts:
- added TP33, TP39: 24VOUT, TestPoint:TestPoint_THTPad_D3.0mm_Drill1.5mm, symbol Connector:TestPoint
- TP11: value TestPoint -> 24V_VBB; footprint (none) -> TestPoint:TestPoint_THTPad_D3.0mm_Drill1.5mm
Connections:
- net VOUT1: now also TP33.1
- net VOUT2: now also TP39.1
Changed lines of the file:
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@@
 	)
 	(junction
+		(at 177.165 84.455)
+		(diameter 0)
+		(color 0 0 0 0)
+	)
+	(junction
+		(at 173.99 84.455)
+		(diameter 0)
+		(color 0 0 0 0)
+	)
+	(junction
 		(at 35.56 163.195)
 		(diameter 0)
@@
 	)
 	(junction
+		(at 177.165 92.075)
+		(diameter 0)
+		(color 0 0 0 0)
+	)
+	(junction
 		(at 138.43 151.13)
 		(diameter 0)
@@
 	)
 	(junction
+		(at 173.99 92.075)
+		(diameter 0)
+		(color 0 0 0 0)
+	)
+	(junction
 		(at 139.7 41.275)
 		(diameter 0)
@@
 	)
 	(junction
-		(at 173.99 84.455)
-		(diameter 0)
-		(color 0 0 0 0)
-	)
-	(junction
 		(at 193.04 99.695)
 		(diameter 0)
@@
 		(color 0 0 0 0)
 	)
-	(junction
-		(at 173.99 92.075)
-		(diameter 0)
-		(color 0 0 0 0)
-	)
 	(bus_entry
 		(at 89.535 102.235)
@@
 	(wire
 		(pts
+			(xy 177.165 84.455) (xy 173.99 84.455)
+		)
+		(stroke
+			(width 0)
+			(type default)
+		)
+	)
+	(wire
+		(pts
 			(xy 71.755 137.16) (xy 60.96 137.16)
 		)
@@
 	(wire
 		(pts
-			(xy 182.88 84.455) (xy 173.99 84.455)
+			(xy 186.055 84.455) (xy 177.165 84.455)
 		)
 		(stroke
@@
 	(wire
 		(pts
+			(xy 177.165 92.075) (xy 173.99 92.075)
+		)
+		(stroke
+			(width 0)
+			(type default)
+		)
+	)
+	(wire
+		(pts
 			(xy 173.99 86.995) (xy 170.815 86.995)
 		)
@@
 	(wire
 		(pts
-			(xy 182.88 92.075) (xy 173.99 92.075)
+			(xy 186.055 92.075) (xy 177.165 92.075)
 		)
 		(stroke
@@
 	)
 	(label "VOUT1"
-		(at 182.88 84.455 180)
+		(at 186.055 84.455 180)
 		(effects
 			(font
@@
 	)
 	(label "VOUT2"
-		(at 182.88 92.075 180)
+		(at 186.055 92.075 180)
 		(effects
 			(font
@@
 	)
 	(symbol
+		(lib_id "Connector:TestPoint")
+		(at 177.165 92.075 0)
+		(unit 1)
+		(body_style 1)
+		(exclude_from_sim no)
+		(in_bom yes)
+		(on_board yes)
+		(in_pos_files yes)
+		(dnp no)
+		(property "Reference" "TP39"
+			(at 178.054 93.98 0)
+			(show_name no)
+			(do_not_autoplace no)
+			(effects
+				(font
+					(size 1.27 1.27)
+				)
+				(justify left)
+			)
+		)
+		(property "Value" "24VOUT"
+			(at 176.022 96.266 0)
+			(show_name no)
+			(do_not_autoplace no)
+			(effects
+				(font
+					(size 1.27 1.27)
+				)
+				(justify left)
+			)
+		)
+		(property "Footprint" "TestPoint:TestPoint_THTPad_D3.0mm_Drill1.5mm"
+			(at 182.245 92.075 0)
+			(hide yes)
+			(show_name no)
+			(do_not_autoplace no)
+			(effects
+				(font
+					(size 1.27 1.27)
+				)
+			)
+		)
+		(property "Datasheet" ""
+			(at 182.245 92.075 0)
+			(hide yes)
+			(show_name no)
+			(do_not_autoplace no)
+			(effects
+				(font
+					(size 1.27 1.27)
+				)
+			)
+		)
+		(property "Description" "test point"
+			(at 177.165 92.075 0)
+			(hide yes)
+			(show_name no)
+			(do_not_autoplace no)
+			(effects
+				(font
+					(size 1.27 1.27)
+				)
+			)
+		)
+		(pin "1"
+		)
+		(instances
+			(project "PS-PowerDistributionUnit"
+				(path "/eb16378f-e371-46a9-bfab-b0d9404d0362/2ab77bb0-369b-4fa2-b5e4-9072d062af22"
+					(reference "TP43")
+					(unit 1)
+				)
+				(path "/eb16378f-e371-46a9-bfab-b0d9404d0362/3e1dda67-cc99-4912-9b53-77c688c0b444"
+					(reference "TP39")
+					(unit 1)
+				)
+				(path "/eb16378f-e371-46a9-bfab-b0d9404d0362/4e29a9cd-f4f8-4556-90cc-d0fc24ec852e"
+					(reference "TP44")
+					(unit 1)
+				)
+				(path "/eb16378f-e371-46a9-bfab-b0d9404d0362/581c2176-fcdd-45dc-ac95-481314f75eaa"
+					(reference "TP41")
+					(unit 1)
+				)
+				(path "/eb16378f-e371-46a9-bfab-b0d9404d0362/7fd95c3c-7bef-4d5e-8058-7407405c1287"
+					(reference "TP40")
+					(unit 1)
+				)
+				(path "/eb16378f-e371-46a9-bfab-b0d9404d0362/ceeb953c-7a8e-4ff4-89fb-4a85a671b5e4"
+					(reference "TP42")
+					(unit 1)
+				)
+			)
+		)
+	)
+	(symbol
 		(lib_id "Device:C")
 		(at 64.77 53.34 0)
@@
 			)
 		)
-		(property "Value" "TestPoint"
+		(property "Value" "24V_VBB"
 			(at 109.728 78.486 0)
 			(show_name no)
@@
 			)
 		)
-		(property "Footprint" ""
+		(property "Footprint" "TestPoint:TestPoint_THTPad_D3.0mm_Drill1.5mm"
 			(at 118.745 84.455 0)
 			(hide yes)
@@
 					(unit 1)
 				)
+			)
+		)
+	)
+	(symbol
+		(lib_id "Connector:TestPoint")
+		(at 177.165 84.455 0)
+		(unit 1)
+		(body_style 1)
+		(exclude_from_sim no)
+		(in_bom yes)
+		(on_board yes)
+		(in_pos_files yes)
+		(dnp no)
+		(property "Reference" "TP33"
+			(at 175.26 76.2 0)
+			(show_name no)
+			(do_not_autoplace no)
+			(effects
+				(font
+					(size 1.27 1.27)
+				)
+				(justify left)
+			)
+		)
+		(property "Value" "24VOUT"
+			(at 173.228 78.486 0)
+			(show_name no)
+			(do_not_autoplace no)
+			(effects
+				(font
+					(size 1.27 1.27)
+				)
+				(justify left)
+			)
+		)
+		(property "Footprint" "TestPoint:TestPoint_THTPad_D3.0mm_Drill1.5mm"
+			(at 182.245 84.455 0)
+			(hide yes)
+			(show_name no)
+			(do_not_autoplace no)
+			(effects
+				(font
+					(size 1.27 1.27)
+				)
+			)
+		)
+		(property "Datasheet" ""
+			(at 182.245 84.455 0)
+			(hide yes)
+			(show_name no)
+			(do_not_autoplace no)
+			(effects
+				(font
+					(size 1.27 1.27)
+				)
+			)
+		)
+		(property "Description" "test point"
+			(at 177.165 84.455 0)
+			(hide yes)
+			(show_name no)
+			(do_not_autoplace no)
+			(effects
+				(font
+					(size 1.27 1.27)
+				)
+			)
+		)
+		(pin "1"
+		)
+		(instances
+			(project "PS-PowerDistributionUnit"
+				(path "/eb16378f-e371-46a9-bfab-b0d9404d0362/2ab77bb0-369b-4fa2-b5e4-9072d062af22"
+					(reference "TP37")
+					(unit 1)
+				)
+				(path "/eb16378f-e371-46a9-bfab-b0d9404d0362/3e1dda67-cc99-4912-9b53-77c688c0b444"
+					(reference "TP33")
+					(unit 1)
+				)
+				(path "/eb16378f-e371-46a9-bfab-b0d9404d0362/4e29a9cd-f4f8-4556-90cc-d0fc24ec852e"
+					(reference "TP38")
+					(unit 1)
+				)
+				(path "/eb16378f-e371-46a9-bfab-b0d9404d0362/581c2176-fcdd-45dc-ac95-481314f75eaa"
+					(reference "TP35")
+					(unit 1)
+				)
+				(path "/eb16378f-e371-46a9-bfab-b0d9404d0362/7fd95c3c-7bef-4d5e-8058-7407405c1287"
+					(reference "TP34")
+					(unit 1)
+				)
+				(path "/eb16378f-e371-46a9-bfab-b0d9404d0362/ceeb953c-7a8e-4ff4-89fb-4a85a671b5e4"
+					(reference "TP36")
+					(unit 1)
+				)

Commit message: added p/n and footprints
Parts:
- C31: footprint (none) -> Capacitor_SMD:C_0603_1608Metric_Pad1.08x0.95mm_HandSolder; P/N (none) -> CC0603KRX7R7BB474
- C32: footprint (none) -> Capacitor_SMD:C_0603_1608Metric_Pad1.08x0.95mm_HandSolder; P/N (none) -> CC0603KRX7R9BB102
- C33: footprint (none) -> Capacitor_SMD:C_0603_1608Metric_Pad1.08x0.95mm_HandSolder; P/N (none) -> TCC0603X5R105K160CT
- C34: footprint (none) -> Capacitor_SMD:C_0603_1608Metric_Pad1.08x0.95mm_HandSolder; P/N (none) -> CSA0603X7R222K101JT
- C35, C36: footprint (none) -> Capacitor_SMD:C_0603_1608Metric_Pad1.08x0.95mm_HandSolder; P/N (none) -> CC0603KRX7R9BB104
- D10, D9: P/N (none) -> NCD0603R1
- D11, D12, D8: footprint (none) -> Diode_SMD:D_SMB; P/N (none) -> TPSMB39CA
- R11, R48, R49: footprint (none) -> Resistor_SMD:R_0603_1608Metric; P/N (none) -> CRCW06034K70FKEA
- R12, R45, R80: footprint (none) -> Resistor_SMD:R_0603_1608Metric; P/N (none) -> CRCW060310K0FKEI
- R44: footprint (none) -> Resistor_SMD:R_0603_1608Metric_Pad0.98x0.95mm_HandSolder; P/N (none) -> CRCW060310R0FKEE
- R46, R81: footprint (none) -> Resistor_SMD:R_0603_1608Metric; LCSC P/N (none) -> C107701; P/N (none) -> RC0603FR-0722RL
- R47: footprint (none) -> Resistor_SMD:R_0603_1608Metric_Pad0.98x0.95mm_HandSolder; P/N (none) -> CRCW06031K00FKEI

Commit message: added usb
Parts:
- IC3: footprint TPS2HCS08AQPWPRQ1 -> PDU_TPS2HCS08AQPWPRQ1:TSSOP16_4P5X5P1_2P78X3P313_TEX
- renumbered C35 to C32, C36 to C33, C32 to C34, C33 to C35, C34 to C36, D11 to D10, D12 to D11, D8 to D12, D9 to D8, D10 to D9, R48 to R28, R49 to R29, R80 to R30, R44 to R31, R81 to R32, R45 to R33, R46 to R34, R11 to R35, R12 to R36, R47 to R37, TP11 to TP33, TP33 to TP34, TP39 to TP35
Connections:
- net +24V_HSS renamed +12V_HSS

Commit message: layout starte but i want to play codename
Parts:
- renumbered C31 to C33, C32 to C34, C33 to C35, C34 to C36, C35 to C37, C36 to C38, R28 to R27, R29 to R28, R30 to R29, R31 to R30, R32 to R31, R33 to R32, R34 to R33, R35 to R34, R36 to R35, R37 to R36, TP33 to TP30, TP34 to TP31, TP35 to TP32
