File: hardware/HSS_Pair.kicad_sch (KiCad schematic)
At the start: 27 parts, among them IC3 TPS2HCS08AQPWPRQ1

Commit message: son...
Other:
- moved on the sheet: R32
Changed lines of the file:
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@@
 	(wire
 		(pts
-			(xy 116.84 89.535) (xy 125.095 89.535)
+			(xy 121.285 89.535) (xy 125.095 89.535)
 		)
 		(stroke
@@
 	(wire
 		(pts
-			(xy 92.075 89.535) (xy 109.22 89.535)
+			(xy 92.075 89.535) (xy 113.665 89.535)
 		)
 		(stroke
@@
 	(symbol
 		(lib_id "Device:R")
-		(at 113.03 89.535 90)
+		(at 117.475 89.535 90)
 		(unit 1)
 		(body_style 1)
@@
 		(dnp no)
 		(property "Reference" "R32"
-			(at 113.03 86.868 90)
+			(at 117.475 86.868 90)
 			(show_name no)
 			(do_not_autoplace no)
@@
 		)
 		(property "Value" "10k"
-			(at 118.364 88.646 90)
+			(at 122.809 88.646 90)
 			(show_name no)
 			(do_not_autoplace no)
@@
 		)
 		(property "Footprint" "Resistor_SMD:R_0603_1608Metric"
-			(at 113.03 91.313 90)
+			(at 117.475 91.313 90)
 			(hide yes)
 			(show_name no)
@@
 		)
 		(property "Datasheet" ""
-			(at 113.03 89.535 0)
+			(at 117.475 89.535 0)
 			(hide yes)
 			(show_name no)
@@
 		)
 		(property "Description" "Resistor"
-			(at 113.03 89.535 0)
+			(at 117.475 89.535 0)
 			(hide yes)
 			(show_name no)
@@
 		)
 		(property "LCSC P/N" "C25804"
-			(at 113.03 89.535 90)
+			(at 117.475 89.535 90)
 			(hide yes)
 			(show_name no)
@@
 		)
 		(property "P/N" "CRCW060310K0FKEI "
-			(at 113.03 89.535 90)
+			(at 117.475 89.535 90)
 			(hide yes)
 			(show_name no)

Commit message: done w HSS and PP
Parts:
- D8, D9: footprint LED_SMD:LED_0201_0603Metric -> LED_SMD:LED_0603_1608Metric
Changed lines of the file:
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@@
 			)
 		)
-		(property "Footprint" "LED_SMD:LED_0201_0603Metric"
+		(property "Footprint" "LED_SMD:LED_0603_1608Metric"
 			(at 53.975 173.355 0)
 			(hide yes)
@@
 			)
 		)
-		(property "Footprint" "LED_SMD:LED_0201_0603Metric"
+		(property "Footprint" "LED_SMD:LED_0603_1608Metric"
 			(at 54.61 147.32 0)
 			(hide yes)

Commit message: booooom not done tho
Parts:
- renumbered R33 to R32, R32 to R33
Changed lines of the file:
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@@
 		(in_pos_files yes)
 		(dnp no)
-		(property "Reference" "R33"
+		(property "Reference" "R32"
 			(at 108.458 98.552 90)
 			(show_name no)
@@
 			(project "PS-PowerDistributionUnit"
 				(path "/eb16378f-e371-46a9-bfab-b0d9404d0362/1d57fdee-2418-4435-ae97-d28030158467"
-					(reference "R63")
+					(reference "R62")
 					(unit 1)
 				)
 				(path "/eb16378f-e371-46a9-bfab-b0d9404d0362/3e1dda67-cc99-4912-9b53-77c688c0b444"
-					(reference "R33")
+					(reference "R32")
 					(unit 1)
 				)
 				(path "/eb16378f-e371-46a9-bfab-b0d9404d0362/83a4b0dc-4f87-423f-8cff-81ec7b69755b"
-					(reference "R53")
+					(reference "R52")
 					(unit 1)
 				)
 				(path "/eb16378f-e371-46a9-bfab-b0d9404d0362/9a4fed0a-9cad-414c-a2d7-99084feee164"
-					(reference "R83")
+					(reference "R82")
 					(unit 1)
 				)
 				(path "/eb16378f-e371-46a9-bfab-b0d9404d0362/b569e97f-7cae-4639-b563-894389ffb9b1"
-					(reference "R73")
+					(reference "R72")
 					(unit 1)
 				)
 				(path "/eb16378f-e371-46a9-bfab-b0d9404d0362/e1779edd-9750-42d0-8bd9-b7615dff1a3e"
-					(reference "R43")
+					(reference "R42")
 					(unit 1)
 				)
@@
 		(in_pos_files yes)
 		(dnp no)
-		(property "Reference" "R32"
+		(property "Reference" "R33"
 			(at 117.475 86.868 90)
 			(show_name no)
@@
 			(project "PS-PowerDistributionUnit"
 				(path "/eb16378f-e371-46a9-bfab-b0d9404d0362/1d57fdee-2418-4435-ae97-d28030158467"
-					(reference "R62")
+					(reference "R63")
 					(unit 1)
 				)
 				(path "/eb16378f-e371-46a9-bfab-b0d9404d0362/3e1dda67-cc99-4912-9b53-77c688c0b444"
-					(reference "R32")
+					(reference "R33")
 					(unit 1)
 				)
 				(path "/eb16378f-e371-46a9-bfab-b0d9404d0362/83a4b0dc-4f87-423f-8cff-81ec7b69755b"
-					(reference "R52")
+					(reference "R53")
 					(unit 1)
 				)
 				(path "/eb16378f-e371-46a9-bfab-b0d9404d0362/9a4fed0a-9cad-414c-a2d7-99084feee164"
-					(reference "R82")
+					(reference "R83")
 					(unit 1)
 				)
 				(path "/eb16378f-e371-46a9-bfab-b0d9404d0362/b569e97f-7cae-4639-b563-894389ffb9b1"
-					(reference "R72")
+					(reference "R73")
 					(unit 1)
 				)
 				(path "/eb16378f-e371-46a9-bfab-b0d9404d0362/e1779edd-9750-42d0-8bd9-b7615dff1a3e"
-					(reference "R42")
-					(unit 1)
-				)
+					(reference "R43")
+					(unit 1)
+				)

Commit message: added pn
Parts:
- C34, C35: LCSC P/N C14663 -> C1591; P/N CC0603KRX7R9BB104 -> CL10B104KB8NNNC
- C37: LCSC P/N C696901 -> C15849; P/N TCC0603X5R105K160CT -> CC0603KRX7R9BB105
- R27, R28, R34: P/N CRCW06034K70FKEA -> 0603WAF4701T5E
- R29, R33, R35: P/N CRCW060310K0FKEI -> 0603WAF1002T5E
- R36: P/N CRCW06031K00FKEI -> 0603WAF1001T5E
Changed lines of the file:
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@@
 			)
 		)
-		(property "LCSC P/N" "C696901"
+		(property "LCSC P/N" "C15849"
 			(at 120.65 46.99 0)
 			(hide yes)
@@
 			)
 		)
-		(property "P/N" "TCC0603X5R105K160CT"
+		(property "P/N" "CC0603KRX7R9BB105"
 			(at 120.65 46.99 0)
 			(hide yes)
@@
 			)
 		)
-		(property "P/N" "CRCW06031K00FKEI "
+		(property "P/N" "0603WAF1001T5E"
 			(at 180.975 106.045 0)
 			(hide yes)
@@
 			)
 		)
-		(property "P/N" "CRCW06034K70FKEA"
+		(property "P/N" "0603WAF4701T5E"
 			(at 138.43 144.145 0)
 			(hide yes)
@@
 			)
 		)
-		(property "P/N" "CRCW06034K70FKEA"
+		(property "P/N" "0603WAF4701T5E"
 			(at 43.18 173.355 90)
 			(hide yes)
@@
 			)
 		)
-		(property "P/N" "CRCW06034K70FKEA"
+		(property "P/N" "0603WAF4701T5E"
 			(at 43.815 147.32 90)
 			(hide yes)
@@
 			)
 		)
-		(property "LCSC P/N" "C14663"
+		(property "LCSC P/N" "C1591"
 			(at 82.55 169.545 0)
 			(hide yes)
@@
 			)
 		)
-		(property "P/N" "CC0603KRX7R9BB104"
+		(property "P/N" "CL10B104KB8NNNC"
 			(at 82.55 169.545 0)
 			(hide yes)
@@
 			)
 		)
-		(property "P/N" "CRCW060310K0FKEI "
+		(property "P/N" "0603WAF1002T5E"
 			(at 50.8 99.06 0)
 			(hide yes)
@@
 			)
 		)
-		(property "LCSC P/N" "C14663"
+		(property "LCSC P/N" "C1591"
 			(at 83.185 143.51 0)
 			(hide yes)
@@
 			)
 		)
-		(property "P/N" "CC0603KRX7R9BB104"
+		(property "P/N" "CL10B104KB8NNNC"
 			(at 83.185 143.51 0)
 			(hide yes)
@@
 			)
 		)
-		(property "P/N" "CRCW060310K0FKEI "
+		(property "P/N" "0603WAF1002T5E"
 			(at 117.475 89.535 90)
 			(hide yes)
@@
 			)
 		)
-		(property "P/N" "CRCW060310K0FKEI "
+		(property "P/N" "0603WAF1002T5E"
 			(at 146.685 151.13 90)
 			(hide yes)

Commit message: need to study matrices:
Parts:
- R27, R28, R29, R31, R32, R33, R34, R35: footprint Resistor_SMD:R_0603_1608Metric -> Resistor_SMD:R_0603_1608Metric_Pad0.98x0.95mm_HandSolder
Changed lines of the file:
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@@
 			)
 		)
-		(property "Footprint" "Resistor_SMD:R_0603_1608Metric"
+		(property "Footprint" "Resistor_SMD:R_0603_1608Metric_Pad0.98x0.95mm_HandSolder"
 			(at 140.208 144.145 90)
 			(hide yes)
@@
 			)
 		)
-		(property "Footprint" "Resistor_SMD:R_0603_1608Metric"
+		(property "Footprint" "Resistor_SMD:R_0603_1608Metric_Pad0.98x0.95mm_HandSolder"
 			(at 43.18 175.133 90)
 			(hide yes)
@@
 			)
 		)
-		(property "Footprint" "Resistor_SMD:R_0603_1608Metric"
+		(property "Footprint" "Resistor_SMD:R_0603_1608Metric_Pad0.98x0.95mm_HandSolder"
 			(at 113.665 101.473 90)
 			(hide yes)
@@
 			)
 		)
-		(property "Footprint" "Resistor_SMD:R_0603_1608Metric"
+		(property "Footprint" "Resistor_SMD:R_0603_1608Metric_Pad0.98x0.95mm_HandSolder"
 			(at 43.815 149.098 90)
 			(hide yes)
@@
 			)
 		)
-		(property "Footprint" "Resistor_SMD:R_0603_1608Metric"
+		(property "Footprint" "Resistor_SMD:R_0603_1608Metric_Pad0.98x0.95mm_HandSolder"
 			(at 59.055 105.918 90)
 			(hide yes)
@@
 			)
 		)
-		(property "Footprint" "Resistor_SMD:R_0603_1608Metric"
+		(property "Footprint" "Resistor_SMD:R_0603_1608Metric_Pad0.98x0.95mm_HandSolder"
 			(at 52.578 99.06 90)
 			(hide yes)
@@
 			)
 		)
-		(property "Footprint" "Resistor_SMD:R_0603_1608Metric"
+		(property "Footprint" "Resistor_SMD:R_0603_1608Metric_Pad0.98x0.95mm_HandSolder"
 			(at 117.475 91.313 90)
 			(hide yes)
@@
 			)
 		)
-		(property "Footprint" "Resistor_SMD:R_0603_1608Metric"
+		(property "Footprint" "Resistor_SMD:R_0603_1608Metric_Pad0.98x0.95mm_HandSolder"
 			(at 146.685 152.908 90)
 			(hide yes)
