File: hardware/USB-C Connector.kicad_sch (KiCad schematic)
At the start: 6 parts, among them J14 USB_C_Receptacle_USB2.0_16P

Commit message: layout starte but i want to play codename
Parts:
- J14: footprint LHRS_ICs:USB_C_Receptacle_GCT_USB4105-xx-A_16P_TopMnt_Horizontal -> LHRS_Connectors:USB_C_Receptacle_GCT_USB4105-xx-A_16P_TopMnt_Horizontal
- renumbered C79 to C73, D60 to D55, D61 to D56, R16 to R89, R100 to R90
Changed lines of the file:
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@@
 		(in_pos_files yes)
 		(dnp no)
-		(property "Reference" "R16"
+		(property "Reference" "R89"
 			(at 86.106 48.26 90)
 			(show_name no)
@@
 			(project "PS-PowerDistributionUnit"
 				(path "/eb16378f-e371-46a9-bfab-b0d9404d0362/e5e6ee2e-1d09-4fff-9eef-bc055f220fc3/f81579d2-7db1-4332-bf6b-3f69d0bc1a0d"
-					(reference "R16")
+					(reference "R89")
 					(unit 1)
 				)
@@
 		(in_pos_files yes)
 		(dnp no)
-		(property "Reference" "R100"
+		(property "Reference" "R90"
 			(at 93.726 48.26 90)
 			(show_name no)
@@
 			(project "PS-PowerDistributionUnit"
 				(path "/eb16378f-e371-46a9-bfab-b0d9404d0362/e5e6ee2e-1d09-4fff-9eef-bc055f220fc3/f81579d2-7db1-4332-bf6b-3f69d0bc1a0d"
-					(reference "R100")
+					(reference "R90")
 					(unit 1)
 				)
@@
 			)
 		)
-		(property "Footprint" "LHRS_ICs:USB_C_Receptacle_GCT_USB4105-xx-A_16P_TopMnt_Horizontal"
+		(property "Footprint" "LHRS_Connectors:USB_C_Receptacle_GCT_USB4105-xx-A_16P_TopMnt_Horizontal"
 			(at 39.37 45.72 0)
 			(hide yes)
@@
 		(dnp no)
 		(fields_autoplaced yes)
-		(property "Reference" "#FLG01"
+		(property "Reference" "#FLG05"
 			(at 71.755 30.48 0)
 			(hide yes)
@@
 			(project "PS-PowerDistributionUnit"
 				(path "/eb16378f-e371-46a9-bfab-b0d9404d0362/e5e6ee2e-1d09-4fff-9eef-bc055f220fc3/f81579d2-7db1-4332-bf6b-3f69d0bc1a0d"
-					(reference "#FLG01")
+					(reference "#FLG05")
 					(unit 1)
 				)
@@
 		(in_pos_files yes)
 		(dnp no)
-		(property "Reference" "D60"
+		(property "Reference" "D55"
 			(at 59.69 24.765 0)
 			(show_name no)
@@
 			(project "PS-PowerDistributionUnit"
 				(path "/eb16378f-e371-46a9-bfab-b0d9404d0362/e5e6ee2e-1d09-4fff-9eef-bc055f220fc3/f81579d2-7db1-4332-bf6b-3f69d0bc1a0d"
-					(reference "D60")
+					(reference "D55")
 					(unit 1)
 				)
@@
 		(in_pos_files yes)
 		(dnp no)
-		(property "Reference" "C79"
+		(property "Reference" "C73"
 			(at 64.3128 37.9984 0)
 			(show_name no)
@@
 			(project "PS-PowerDistributionUnit"
 				(path "/eb16378f-e371-46a9-bfab-b0d9404d0362/e5e6ee2e-1d09-4fff-9eef-bc055f220fc3/f81579d2-7db1-4332-bf6b-3f69d0bc1a0d"
-					(reference "C79")
+					(reference "C73")
 					(unit 1)
 				)
@@
 		(in_pos_files yes)
 		(dnp no)
-		(property "Reference" "D61"
+		(property "Reference" "D56"
 			(at 82.55 71.12 0)
 			(show_name no)
@@
 			(project "PS-PowerDistributionUnit"
 				(path "/eb16378f-e371-46a9-bfab-b0d9404d0362/e5e6ee2e-1d09-4fff-9eef-bc055f220fc3/f81579d2-7db1-4332-bf6b-3f69d0bc1a0d"
-					(reference "D61")
+					(reference "D56")
 					(unit 1)
 				)
