File: hardware/USB-C Connector.kicad_sch (KiCad schematic)
At the start: 6 parts, among them J8 USB_C_Receptacle_USB2.0_16P

Commit message: gerb bom
Parts:
- J8: P/N (none) -> USB4105-GF-A-120
Changed lines of the file:
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@@
+			)
+		)
+		(property "P/N" "USB4105-GF-A-120"
+			(at 35.56 45.72 0)
+			(hide yes)
+			(show_name no)
+			(do_not_autoplace no)
+			(effects
+				(font
+					(size 1.27 1.27)
+				)
 			)
 		)
