File: hardware/PS-PowerDistributionUnit.kicad_pcb (KiCad board)
At the start: 2 copper layers, 324 parts, among them IC1 LM74502DDFR, IC2 TCAN3413DR, IC3 TPS2HCS08AQPWPRQ1, IC4 TPS2HCS08AQPWPRQ1, IC5 TPS2HCS08AQPWPRQ1, IC6 TPS2HCS08AQPWPRQ1, IC7 TPS2HCS08AQPWPRQ1, IC8 TPS2HCS08AQPWPRQ1, J1 LV_IN, J10 CAN2, J11 CAN_DEBUG, J12 SWD_Header, J13 SWD, J14 USB_C_Receptacle_USB2.0_16P, J2 Conn_01x02, J3 Conn_01x02, J4 Conn_01x02, J5 LV_0UT2, J6 Conn_01x02, J7 Conn_01x02, J8 Conn_01x02, J9 CAN1, Q1 PSMN012-100YS, Q2 PSMN012-100YS, SW1 Reset, SW2 SW_SPDT, U1 MCP1826S, U2 TPS2117DRLR, U3 STM32G473CETx, U4 LMR51635XDDCR, Y1 Crystal

Commit message: done w HSS and PP
Parts:
- D13, D14, D18, D19, D23, D24, D28, D29, D33, D34, D8, D9: value LED -> BFuse; footprint LED_SMD:LED_0201_0603Metric -> LED_SMD:LED_0603_1608Metric
- R1, R2, R27, R28, R29, R3, R31, R32, R33, R34, R35, R37, R38, R39, R4, R41, R42, R43, R44, R45, R47, R48, R49, R5, R51, R52, R53, R54, R55, R57, R58, R59, R6, R61, R62, R63, R64, R65, R67, R68, R69, R7, R71, R72, R73, R74, R75, R77, R78, R79, R8, R81, R82, R83, R84, R85, R87, R88: footprint Resistor_SMD:R_0603_1608Metric -> Resistor_SMD:R_0603_1608Metric_Pad0.98x0.95mm_HandSolder
- moved J7 434.6 mm to (281.8, 121.2)
- moved J8 434.6 mm to (281.8, 129.2)
- moved J6 431.8 mm to (281.8, 92.8)
- moved J4 431.5 mm to (281.5, 84.0)
- moved J2 430.7 mm to (282.8, 43.8)
- moved J3 430.5 mm to (282.5, 52.8)
- moved C23 296.1 mm to (191.9, 104.7), turned to 180 degrees
- moved R1 294.1 mm to (174.3, 64.4)
- moved R2 294.1 mm to (174.3, 67.0)
- moved R3 294.1 mm to (174.3, 69.5)
- moved R4 294.1 mm to (174.3, 72.0)
- moved R5 294.1 mm to (174.3, 74.5)
- moved R6 294.1 mm to (174.3, 77.0)
- moved R7 294.1 mm to (174.3, 79.5)
- moved C20 292.4 mm to (188.1, 102.3), turned to 180 degrees
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Routing:
- added copper zone on F.Cu, net /+12V_HSS

Commit message: my baby is in groups
Parts:
- C21, C73: footprint Capacitor_SMD:C_0805_2012Metric -> Capacitor_SMD:C_0805_2012Metric_Pad1.18x1.45mm_HandSolder
- C71: footprint Capacitor_SMD:C_0603_1608Metric -> Capacitor_SMD:C_0603_1608Metric_Pad1.08x0.95mm_HandSolder
- D13, D14, D18, D19, D23, D24, D28, D29, D33, D34, D8, D9: value BFuse -> LED
- R1, R2, R27, R28, R29, R3, R31, R32, R33, R34, R35, R37, R38, R39, R4, R41, R42, R43, R44, R45, R47, R48, R49, R5, R51, R52, R53, R54, R55, R57, R58, R59, R6, R61, R62, R63, R64, R65, R67, R68, R69, R7, R71, R72, R73, R74, R75, R77, R78, R79, R8, R81, R82, R83, R84, R85, R87, R88: footprint Resistor_SMD:R_0603_1608Metric_Pad0.98x0.95mm_HandSolder -> Resistor_SMD:R_0603_1608Metric
- moved C22 269.5 mm to (164.6, 116.8)
- moved D5 269.5 mm to (184.1, 135.9)
- moved D6 269.5 mm to (164.6, 136.4)
- moved D7 269.5 mm to (168.8, 136.2)
- moved J12 269.5 mm to (185.3, 112.3)
- moved J13 269.5 mm to (188.8, 125.3)
- moved R19 269.5 mm to (173.3, 119.3)
- moved R20 269.5 mm to (173.3, 121.8)
- moved R21 269.5 mm to (177.7, 109.2)
- moved R22 269.5 mm to (177.7, 111.8)
- moved R23 269.5 mm to (177.7, 114.3)
- moved R24 269.5 mm to (177.7, 116.8)
- moved R25 269.5 mm to (177.7, 119.3)
- moved R26 269.5 mm to (177.7, 121.8)
- moved SW1 269.5 mm to (184.2, 119.8)
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