File: hardware/PS-PowerDistributionUnit.kicad_pcb (KiCad board)
At the start: 2 copper layers, 324 parts, among them IC1 LM74502DDFR, IC2 TCAN3413DR, IC3 TPS2HCS08AQPWPRQ1, IC4 TPS2HCS08AQPWPRQ1, IC5 TPS2HCS08AQPWPRQ1, IC6 TPS2HCS08AQPWPRQ1, IC7 TPS2HCS08AQPWPRQ1, IC8 TPS2HCS08AQPWPRQ1, J1 LV_IN, J10 CAN2, J11 CAN_DEBUG, J12 SWD_Header, J13 SWD, J14 USB_C_Receptacle_USB2.0_16P, J2 Conn_01x02, J3 Conn_01x02, J4 Conn_01x02, J5 LV_0UT2, J6 Conn_01x02, J7 Conn_01x02, J8 Conn_01x02, J9 CAN1, Q1 PSMN012-100YS, Q2 PSMN012-100YS, SW1 Reset, SW2 SW_SPDT, U1 MCP1826S, U2 TPS2117DRLR, U3 STM32G473CETx, U4 LMR51635XDDCR, Y1 Crystal

Commit message: two of my ugly babies r somewhat routed
Parts:
- moved C45 50.9 mm to (197.0, 115.2)
- moved C49 50.9 mm to (188.1, 102.5)
- moved R54 50.9 mm to (200.1, 95.7)
- moved C48 50.9 mm to (188.1, 105.0)
- moved D20 50.9 mm to (220.1, 94.8)
- moved D21 50.9 mm to (220.2, 117.6)
- moved F7 50.9 mm to (215.4, 102.0)
- moved R47 50.9 mm to (209.4, 96.0)
- moved R48 50.9 mm to (209.4, 116.0)
- moved C46 50.9 mm to (226.6, 101.1)
- moved C47 50.9 mm to (226.6, 109.5)
- moved C50 50.9 mm to (194.3, 112.4)
- moved D18 50.9 mm to (213.8, 96.0)
- moved D19 50.9 mm to (213.8, 116.0)
- moved D22 50.9 mm to (192.6, 105.4)
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Routing:
- net /Pair4/VDD: track 0.00 -> 7.79 mm
- net Net-(IC3-DI): track 0.00 -> 6.81 mm
- net /Pair4/SPI_CS: track 0.00 -> 6.39 mm
- net /Pair1/VDD: track 0.00 -> 6.26 mm
- net Net-(IC6-DI): track 0.00 -> 5.70 mm
- net /Pair1/SPI_CS: track 0.00 -> 4.71 mm
- net /Pair1/FLT_WAKE: track 0.00 -> 4.58 mm
- net Net-(IC6-SNS): track 0.00 -> 4.21 mm
- net /Pair4/FLT_WAKE: track 0.00 -> 4.20 mm
- net Net-(IC3-SNS): track 0.00 -> 3.87 mm
- net Net-(IC3-SDO): track 0.00 -> 2.74 mm
- net Net-(D9-A): track 0.00 -> 2.50 mm
- net Net-(D24-A): track 0.00 -> 2.42 mm
- net Net-(IC6-SDO): track 0.00 -> 2.40 mm
- net Net-(D23-A): track 0.00 -> 2.35 mm
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- added copper zone on F.Cu, net /OUTPUT2
- added copper zone on F.Cu, net /OUTPUT7
- added copper zone on F.Cu, net /OUTPUT8
- added copper zone on F.Cu, net /Pair1/VOUT1
- added copper zone on F.Cu, net /Pair1/VOUT2
- added copper zone on F.Cu, net /Pair4/VOUT1
- added copper zone on F.Cu, net /Pair4/VOUT2

Commit message: more ugly babies
Parts:
- moved R20 87.7 mm to (165.7, 60.9), turned to 180 degrees
- moved SW1 87.5 mm to (159.5, 63.3)
- moved C22 81.9 mm to (169.3, 60.9), turned to 180 degrees
- moved C25 27.4 mm to (168.8, 50.5), turned to 90 degrees
- moved C33 25.6 mm to (190.4, 35.9)
- moved C34 25.6 mm to (214.2, 25.0)
- moved C35 25.6 mm to (213.9, 34.1)
- moved C36 25.6 mm to (183.4, 28.6)
- moved C37 25.6 mm to (185.2, 28.6)
- moved C38 25.6 mm to (186.8, 36.8)
- moved D10 25.6 mm to (207.2, 18.9)
- moved D11 25.6 mm to (207.2, 42.1)
- moved D12 25.6 mm to (179.9, 28.1)
- moved D8 25.6 mm to (200.3, 19.9)
- moved F2 25.6 mm to (202.7, 34.9)
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