File: hardware/USB-C Connector.recovered.2026-09-09_232641.kicad_sch (KiCad schematic)
At the start: 6 parts, among them J14 USB_C_Receptacle_USB2.0_16P

Commit message: my baby is in groups
Parts:
- C73: footprint Capacitor_SMD:C_0805_2012Metric_Pad1.18x1.45mm_HandSolder -> Capacitor_SMD:C_0805_2012Metric
Changed lines of the file:
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@@
 			)
 		)
-		(property "Footprint" "Capacitor_SMD:C_0805_2012Metric_Pad1.18x1.45mm_HandSolder"
+		(property "Footprint" "Capacitor_SMD:C_0805_2012Metric"
 			(at 66.3448 33.02 0)
 			(hide yes)
