File: hardware/Power_Mux.kicad_sch (KiCad schematic)
At the start: 6 parts, among them U2 TPS2117DRLR

Commit message: layout starte but i want to play codename
Parts:
- renumbered C77 to C12, C78 to C13
Changed lines of the file:
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@@
 		(in_pos_files yes)
 		(dnp no)
-		(property "Reference" "C78"
+		(property "Reference" "C13"
 			(at 91.8972 57.2516 0)
 			(show_name no)
@@
 			(project "PS-PowerDistributionUnit"
 				(path "/eb16378f-e371-46a9-bfab-b0d9404d0362/e5e6ee2e-1d09-4fff-9eef-bc055f220fc3/e9da0216-1649-4300-a983-3b0c0f99c133"
-					(reference "C78")
+					(reference "C13")
 					(unit 1)
 				)
@@
 		(in_pos_files yes)
 		(dnp no)
-		(property "Reference" "C77"
+		(property "Reference" "C12"
 			(at 42.3672 67.4116 0)
 			(show_name no)
@@
 			(project "PS-PowerDistributionUnit"
 				(path "/eb16378f-e371-46a9-bfab-b0d9404d0362/e5e6ee2e-1d09-4fff-9eef-bc055f220fc3/e9da0216-1649-4300-a983-3b0c0f99c133"
-					(reference "C77")
+					(reference "C12")
 					(unit 1)
 				)

Commit message: added pn
Parts:
- C10, C11, C12, C13: LCSC P/N (none) -> C1591; P/N MLASH168SB7104KTNA01 -> CL10B104KB8NNNC
- R15: LCSC P/N (none) -> C25804; P/N CRCW060310K0FKEI -> 0603WAF1002T5E
- U2: LCSC P/N (none) -> C22399676
Changed lines of the file:
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@@
 			)
 		)
-		(property "P/N" "MLASH168SB7104KTNA01"
+		(property "P/N" "CL10B104KB8NNNC"
 			(at 88.9 58.42 0)
 			(hide yes)
@@
 		)
 		(property "Mfg" "MLASH168SB7104KTNA01"
+			(at 88.9 58.42 0)
+			(hide yes)
+			(show_name no)
+			(do_not_autoplace no)
+			(effects
+				(font
+					(size 1.27 1.27)
+				)
+			)
+		)
+		(property "LCSC P/N" "C1591"
 			(at 88.9 58.42 0)
 			(hide yes)
@@
 			)
 		)
-		(property "P/N" "CRCW060310K0FKEI "
+		(property "P/N" "0603WAF1002T5E"
 			(at 76.2 68.58 90)
+			(hide yes)
+			(show_name no)
+			(do_not_autoplace no)
+			(effects
+				(font
+					(size 1.27 1.27)
+				)
+			)
+		)
+		(property "LCSC P/N" "C25804"
+			(at 76.2 68.58 0)
 			(hide yes)
 			(show_name no)
@@
 			)
 		)
-		(property "P/N" "MLASH168SB7104KTNA01"
+		(property "P/N" "CL10B104KB8NNNC"
 			(at 21.59 45.72 0)
 			(hide yes)
@@
 		)
 		(property "Mfg" "MLASH168SB7104KTNA01"
+			(at 21.59 45.72 0)
+			(hide yes)
+			(show_name no)
+			(do_not_autoplace no)
+			(effects
+				(font
+					(size 1.27 1.27)
+				)
+			)
+		)
+		(property "LCSC P/N" "C1591"
 			(at 21.59 45.72 0)
 			(hide yes)
@@
 			)
 		)
+		(property "LCSC P/N" "C22399676"
+			(at 60.96 62.23 0)
+			(hide yes)
+			(show_name no)
+			(do_not_autoplace no)
+			(effects
+				(font
+					(size 1.27 1.27)
+				)
+			)
+		)
 		(pin "6"
 		)
@@
 			)
 		)
-		(property "P/N" "MLASH168SB7104KTNA01"
+		(property "P/N" "CL10B104KB8NNNC"
 			(at 39.37 68.58 0)
 			(hide yes)
@@
 		)
 		(property "Mfg" "MLASH168SB7104KTNA01"
+			(at 39.37 68.58 0)
+			(hide yes)
+			(show_name no)
+			(do_not_autoplace no)
+			(effects
+				(font
+					(size 1.27 1.27)
+				)
+			)
+		)
+		(property "LCSC P/N" "C1591"
 			(at 39.37 68.58 0)
 			(hide yes)
@@
 			)
 		)
-		(property "P/N" "MLASH168SB7104KTNA01"
+		(property "P/N" "CL10B104KB8NNNC"
 			(at 35.56 45.72 0)
 			(hide yes)
@@
 			(at 35.56 45.72 0)
 			(hide yes)
+			(show_name no)
+			(do_not_autoplace no)
+			(effects
+				(font
+					(size 1.27 1.27)
+				)
+			)
+		)
+		(property "LCSC P/N" "C1591"
+			(at 35.56 45.72 0)
+			(hide yes)
