File: hardware/USB-C Connector.recovered.2026-09-13_235320.kicad_sch (KiCad schematic)
At the start: 6 parts, among them J8 USB_C_Receptacle_USB2.0_16P

Commit message: added pn
Parts:
- C75: P/N GRM21BR61H106KE43K -> TMK212BBJ106MGHT
- R89, R90: P/N CRCW06035K10FKEC -> (none)
Changed lines of the file:
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@@
+		)
+	)
+	(label "D-"
+		(at 52.07 44.45 0)
+		(effects
+			(font
+				(size 1.27 1.27)
+			)
+			(justify left bottom)
+		)
+	)
+	(label "D+"
+		(at 52.07 49.53 0)
+		(effects
+			(font
+				(size 1.27 1.27)
+			)
+			(justify left bottom)
 		)
 	)
@@
 			)
 		)
-		(property "P/N" "CRCW06035K10FKEC"
-			(at 90.17 48.26 90)
-			(hide yes)
-			(show_name no)
-			(do_not_autoplace no)
-			(effects
-				(font
-					(size 1.27 1.27)
-				)
-			)
-		)
 		(pin "1"
 		)
@@
 		)
 		(property "LCSC P/N" "C23186"
-			(at 97.79 48.26 90)
-			(hide yes)
-			(show_name no)
-			(do_not_autoplace no)
-			(effects
-				(font
-					(size 1.27 1.27)
-				)
-			)
-		)
-		(property "P/N" "CRCW06035K10FKEC"
 			(at 97.79 48.26 90)
 			(hide yes)
@@
 			)
 		)
-		(property "P/N" "GRM21BR61H106KE43K"
+		(property "P/N" "TMK212BBJ106MGHT"
 			(at 67.31 36.83 0)
 			(hide yes)
