File: hardware/CAN.kicad_sch (KiCad schematic)
At the start: 4 parts, among them J10 CAN2, J11 CAN_DEBUG, J9 CAN1

Commit message: need to study matrices:
Parts:
- R16: P/N (none) -> CRCW06030000Z0EE
Changed lines of the file:
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@@
+			)
+		)
+		(property "P/N" "CRCW06030000Z0EE"
+			(at 85.725 73.66 0)
+			(hide yes)
+			(show_name no)
+			(do_not_autoplace no)
+			(effects
+				(font
+					(size 1.27 1.27)
+				)
 			)
 		)
