File: hardware/12VBuck.kicad_sch (KiCad schematic)
At the start: 12 parts, among them U4 LMR51635XDDCR

Commit message: layout starte but i want to play codename
Parts:
- renumbered C67 to C69, C68 to C70, C69 to C71, C70 to C72, L2 to L1, R88 to R87, R89 to R88, TP51 to TP48, TP52 to TP49, TP53 to TP50, TP54 to TP51
Changed lines of the file:
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@@
 		(dnp no)
 		(fields_autoplaced yes)
-		(property "Reference" "#FLG04"
+		(property "Reference" "#FLG02"
 			(at 149.86 79.375 0)
 			(hide yes)
@@
 			(project "PS-PowerDistributionUnit"
 				(path "/eb16378f-e371-46a9-bfab-b0d9404d0362/e5e6ee2e-1d09-4fff-9eef-bc055f220fc3/327cca63-c9b6-4c56-8c6f-1a607730f7cc"
-					(reference "#FLG04")
+					(reference "#FLG02")
 					(unit 1)
 				)
@@
 		(dnp no)
 		(fields_autoplaced yes)
-		(property "Reference" "C67"
+		(property "Reference" "C69"
 			(at 96.52 85.0962 0)
 			(show_name no)
@@
 			(project "PS-PowerDistributionUnit"
 				(path "/eb16378f-e371-46a9-bfab-b0d9404d0362/e5e6ee2e-1d09-4fff-9eef-bc055f220fc3/327cca63-c9b6-4c56-8c6f-1a607730f7cc"
-					(reference "C67")
+					(reference "C69")
 					(unit 1)
 				)
@@
 		(in_pos_files yes)
 		(dnp no)
-		(property "Reference" "TP51"
+		(property "Reference" "TP48"
 			(at 229.87 123.6979 0)
 			(hide yes)
@@
 			(project "PS-PowerDistributionUnit"
 				(path "/eb16378f-e371-46a9-bfab-b0d9404d0362/e5e6ee2e-1d09-4fff-9eef-bc055f220fc3/327cca63-c9b6-4c56-8c6f-1a607730f7cc"
-					(reference "TP51")
+					(reference "TP48")
 					(unit 1)
 				)
@@
 		(in_pos_files yes)
 		(dnp no)
-		(property "Reference" "L2"
+		(property "Reference" "L1"
 			(at 161.29 87.884 90)
 			(show_name no)
@@
 			(project "PS-PowerDistributionUnit"
 				(path "/eb16378f-e371-46a9-bfab-b0d9404d0362/e5e6ee2e-1d09-4fff-9eef-bc055f220fc3/327cca63-c9b6-4c56-8c6f-1a607730f7cc"
-					(reference "L2")
+					(reference "L1")
 					(unit 1)
 				)
@@
 		(in_pos_files yes)
 		(dnp no)
-		(property "Reference" "TP53"
+		(property "Reference" "TP50"
 			(at 242.57 123.6979 0)
 			(hide yes)
@@
 			(project "PS-PowerDistributionUnit"
 				(path "/eb16378f-e371-46a9-bfab-b0d9404d0362/e5e6ee2e-1d09-4fff-9eef-bc055f220fc3/327cca63-c9b6-4c56-8c6f-1a607730f7cc"
-					(reference "TP53")
+					(reference "TP50")
 					(unit 1)
 				)
@@
 		(in_pos_files yes)
 		(dnp no)
-		(property "Reference" "TP52"
+		(property "Reference" "TP49"
 			(at 229.87 136.3979 0)
 			(hide yes)
@@
 			(project "PS-PowerDistributionUnit"
 				(path "/eb16378f-e371-46a9-bfab-b0d9404d0362/e5e6ee2e-1d09-4fff-9eef-bc055f220fc3/327cca63-c9b6-4c56-8c6f-1a607730f7cc"
-					(reference "TP52")
+					(reference "TP49")
 					(unit 1)
 				)
@@
 		(in_pos_files yes)
 		(dnp no)
-		(property "Reference" "TP54"
+		(property "Reference" "TP51"
 			(at 242.57 136.3979 0)
 			(hide yes)
@@
 			(project "PS-PowerDistributionUnit"
 				(path "/eb16378f-e371-46a9-bfab-b0d9404d0362/e5e6ee2e-1d09-4fff-9eef-bc055f220fc3/327cca63-c9b6-4c56-8c6f-1a607730f7cc"
-					(reference "TP54")
+					(reference "TP51")
 					(unit 1)
 				)
@@
 		(dnp no)
 		(fields_autoplaced yes)
-		(property "Reference" "C70"
+		(property "Reference" "C72"
 			(at 184.15 88.9062 0)
 			(show_name no)
@@
 			(project "PS-PowerDistributionUnit"
 				(path "/eb16378f-e371-46a9-bfab-b0d9404d0362/e5e6ee2e-1d09-4fff-9eef-bc055f220fc3/327cca63-c9b6-4c56-8c6f-1a607730f7cc"
-					(reference "C70")
+					(reference "C72")
 					(unit 1)
 				)
@@
 		(dnp no)
 		(fields_autoplaced yes)
-		(property "Reference" "#FLG06"
+		(property "Reference" "#FLG04"
 			(at 181.61 84.455 0)
 			(hide yes)
@@
 			(project "PS-PowerDistributionUnit"
 				(path "/eb16378f-e371-46a9-bfab-b0d9404d0362/e5e6ee2e-1d09-4fff-9eef-bc055f220fc3/327cca63-c9b6-4c56-8c6f-1a607730f7cc"
-					(reference "#FLG06")
+					(reference "#FLG04")
 					(unit 1)
 				)
@@
 		(dnp no)
 		(fields_autoplaced yes)
-		(property "Reference" "#FLG03"
+		(property "Reference" "#FLG01"
 			(at 88.9 79.375 0)
 			(hide yes)
@@
 			(project "PS-PowerDistributionUnit"
 				(path "/eb16378f-e371-46a9-bfab-b0d9404d0362/e5e6ee2e-1d09-4fff-9eef-bc055f220fc3/327cca63-c9b6-4c56-8c6f-1a607730f7cc"
-					(reference "#FLG03")
+					(reference "#FLG01")
 					(unit 1)
 				)
@@
 		(in_pos_files yes)
 		(dnp no)
-		(property "Reference" "C69"
+		(property "Reference" "C71"
 			(at 156.718 80.01 0)
 			(show_name no)
@@
 			(project "PS-PowerDistributionUnit"
 				(path "/eb16378f-e371-46a9-bfab-b0d9404d0362/e5e6ee2e-1d09-4fff-9eef-bc055f220fc3/327cca63-c9b6-4c56-8c6f-1a607730f7cc"
-					(reference "C69")
+					(reference "C71")
 					(unit 1)
 				)
@@
 		(in_pos_files yes)
 		(dnp no)
-		(property "Reference" "#FLG05"
+		(property "Reference" "#FLG03"
 			(at 149.86 84.455 0)
 			(hide yes)
@@
 			(project "PS-PowerDistributionUnit"
 				(path "/eb16378f-e371-46a9-bfab-b0d9404d0362/e5e6ee2e-1d09-4fff-9eef-bc055f220fc3/327cca63-c9b6-4c56-8c6f-1a607730f7cc"
-					(reference "#FLG05")
+					(reference "#FLG03")
 					(unit 1)
 				)
@@
 		(dnp no)
 		(fields_autoplaced yes)
-		(property "Reference" "R88"
+		(property "Reference" "R87"
 			(at 227.33 85.0899 0)
 			(show_name no)
@@
 			(project "PS-PowerDistributionUnit"
 				(path "/eb16378f-e371-46a9-bfab-b0d9404d0362/e5e6ee2e-1d09-4fff-9eef-bc055f220fc3/327cca63-c9b6-4c56-8c6f-1a607730f7cc"
-					(reference "R88")
+					(reference "R87")
 					(unit 1)
 				)
@@
 		(dnp no)
 		(fields_autoplaced yes)
-		(property "Reference" "C68"
+		(property "Reference" "C70"
 			(at 105.41 87.6362 0)
 			(show_name no)
@@
 			(project "PS-PowerDistributionUnit"
 				(path "/eb16378f-e371-46a9-bfab-b0d9404d0362/e5e6ee2e-1d09-4fff-9eef-bc055f220fc3/327cca63-c9b6-4c56-8c6f-1a607730f7cc"
-					(reference "C68")
+					(reference "C70")
 					(unit 1)
 				)
@@
 		(dnp no)
 		(fields_autoplaced yes)
-		(property "Reference" "R89"
+		(property "Reference" "R88"
 			(at 227.33 92.7099 0)
 			(show_name no)
@@
 			(project "PS-PowerDistributionUnit"
 				(path "/eb16378f-e371-46a9-bfab-b0d9404d0362/e5e6ee2e-1d09-4fff-9eef-bc055f220fc3/327cca63-c9b6-4c56-8c6f-1a607730f7cc"
-					(reference "R89")
-					(unit 1)
-				)
+					(reference "R88")
+					(unit 1)
+				)

Commit message: chud fresh
Parts:
- removed C72: 47u, Capacitor_SMD:C_1210_3225Metric_Pad1.33x2.70mm_HandSolder, symbol Device:C_Small
- added C4, C5: 22u, Capacitor_SMD:C_1210_3225Metric_Pad1.33x2.70mm_HandSolder, symbol Device:C
- added C6: 3.3u, Capacitor_SMD:C_0805_2012Metric_Pad1.18x1.45mm_HandSolder, symbol Device:C
- C1: renamed from C69; LCSC P/N (none) -> C6962403; P/N MSASL168SB5475KTNA01 -> 08055D475KAT4A
- C2: renamed from C70; footprint Capacitor_SMD:C_0805_2012Metric_Pad1.18x1.45mm_HandSolder -> Capacitor_SMD:C_0603_1608Metric_Pad1.08x0.95mm_HandSolder; LCSC P/N (none) -> C6666325
- C3: renamed from C71; LCSC P/N (none) -> C6666325
- L1: footprint LHRS_Passives:SRN8040-150M -> LHRS_Passives:74439369082
- R1: renamed from R87; LCSC P/N (none) -> C25803; P/N AE1206BR-07100KL -> CRCW0603100KFKEE
- R2: renamed from R88; LCSC P/N (none) -> C844132; P/N ERA-2ARB1912X -> CRCW060319K1FKEAHP
- renumbered TP48 to TP1, TP49 to TP2, TP50 to TP3, TP51 to TP4, U4 to U1
Connections:
- net GND: now also C4.2, C5.2, C6.2
- net V_out_5V: now also C4.1, C5.1, C6.1

Commit message: done w HSS and PP
Parts:
- renumbered C1 to C69, C2 to C70, C3 to C71, C4 to C72, C5 to C74, C6 to C75, R1 to R87, R2 to R88, TP1 to TP48, TP2 to TP49, TP3 to TP50, TP4 to TP51, U1 to U4
Changed lines of the file:
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@@
+				)
+			)
+			(project "PS-PowerDistributionUnit"
+				(path "/eb16378f-e371-46a9-bfab-b0d9404d0362/e5e6ee2e-1d09-4fff-9eef-bc055f220fc3/77a6ec5c-8e09-4a13-82a9-b08f1d53f7e4"
+					(reference "#FLG02")
+					(unit 1)
 				)
 			)
@@
 		(dnp no)
 		(fields_autoplaced yes)
-		(property "Reference" "C1"
+		(property "Reference" "C69"
 			(at 96.52 85.0962 0)
 			(show_name no)
@@
 				(path "/ad6c7df0-eb90-4670-9aa8-3e2007aefc2d/41c72b07-cf60-4ca9-96a7-6ae96aaa0c90"
 					(reference "C8")
+					(unit 1)
+				)
+			)
+			(project "PS-PowerDistributionUnit"
+				(path "/eb16378f-e371-46a9-bfab-b0d9404d0362/e5e6ee2e-1d09-4fff-9eef-bc055f220fc3/77a6ec5c-8e09-4a13-82a9-b08f1d53f7e4"
+					(reference "C69")
 					(unit 1)
 				)
@@
 		(in_pos_files yes)
 		(dnp no)
-		(property "Reference" "TP1"
+		(property "Reference" "TP48"
 			(at 229.87 123.6979 0)
 			(hide yes)
@@
 				(path "/ad6c7df0-eb90-4670-9aa8-3e2007aefc2d/41c72b07-cf60-4ca9-96a7-6ae96aaa0c90"
 					(reference "TP9")
+					(unit 1)
+				)
+			)
+			(project "PS-PowerDistributionUnit"
+				(path "/eb16378f-e371-46a9-bfab-b0d9404d0362/e5e6ee2e-1d09-4fff-9eef-bc055f220fc3/77a6ec5c-8e09-4a13-82a9-b08f1d53f7e4"
+					(reference "TP48")
 					(unit 1)
 				)
@@
 				)
 			)
+			(project "PS-PowerDistributionUnit"
+				(path "/eb16378f-e371-46a9-bfab-b0d9404d0362/e5e6ee2e-1d09-4fff-9eef-bc055f220fc3/77a6ec5c-8e09-4a13-82a9-b08f1d53f7e4"
+					(reference "L1")
+					(unit 1)
+				)
+			)
 			(project "12VBuck"
 				(path "/f2a6729b-b8d5-4133-ae64-a5e680928255"
@@
 		(in_pos_files yes)
 		(dnp no)
-		(property "Reference" "TP3"
+		(property "Reference" "TP50"
 			(at 242.57 123.6979 0)
 			(hide yes)
@@
 				(path "/ad6c7df0-eb90-4670-9aa8-3e2007aefc2d/41c72b07-cf60-4ca9-96a7-6ae96aaa0c90"
 					(reference "TP11")
+					(unit 1)
+				)
+			)
+			(project "PS-PowerDistributionUnit"
+				(path "/eb16378f-e371-46a9-bfab-b0d9404d0362/e5e6ee2e-1d09-4fff-9eef-bc055f220fc3/77a6ec5c-8e09-4a13-82a9-b08f1d53f7e4"
+					(reference "TP50")
 					(unit 1)
 				)
@@
 		(in_pos_files yes)
 		(dnp no)
-		(property "Reference" "TP2"
+		(property "Reference" "TP49"
 			(at 229.87 136.3979 0)
 			(hide yes)
@@
 				(path "/ad6c7df0-eb90-4670-9aa8-3e2007aefc2d/41c72b07-cf60-4ca9-96a7-6ae96aaa0c90"
 					(reference "TP10")
+					(unit 1)
+				)
+			)
+			(project "PS-PowerDistributionUnit"
+				(path "/eb16378f-e371-46a9-bfab-b0d9404d0362/e5e6ee2e-1d09-4fff-9eef-bc055f220fc3/77a6ec5c-8e09-4a13-82a9-b08f1d53f7e4"
+					(reference "TP49")
 					(unit 1)
 				)
@@
 		(dnp no)
 		(fields_autoplaced yes)
-		(property "Reference" "U1"
+		(property "Reference" "U4"
 			(at 129.54 71.12 0)
 			(show_name no)
@@
 				(path "/ad6c7df0-eb90-4670-9aa8-3e2007aefc2d/41c72b07-cf60-4ca9-96a7-6ae96aaa0c90"
 					(reference "U3")
+					(unit 1)
+				)
+			)
+			(project "PS-PowerDistributionUnit"
+				(path "/eb16378f-e371-46a9-bfab-b0d9404d0362/e5e6ee2e-1d09-4fff-9eef-bc055f220fc3/77a6ec5c-8e09-4a13-82a9-b08f1d53f7e4"
+					(reference "U4")
 					(unit 1)
 				)
@@
 		(in_pos_files yes)
 		(dnp no)
-		(property "Reference" "TP4"
+		(property "Reference" "TP51"
 			(at 242.57 136.3979 0)
 			(hide yes)
@@
 				(path "/ad6c7df0-eb90-4670-9aa8-3e2007aefc2d/41c72b07-cf60-4ca9-96a7-6ae96aaa0c90"
 					(reference "TP12")
+					(unit 1)
+				)
+			)
+			(project "PS-PowerDistributionUnit"
+				(path "/eb16378f-e371-46a9-bfab-b0d9404d0362/e5e6ee2e-1d09-4fff-9eef-bc055f220fc3/77a6ec5c-8e09-4a13-82a9-b08f1d53f7e4"
+					(reference "TP51")
 					(unit 1)
 				)
@@
 				)
 			)
+			(project "PS-PowerDistributionUnit"
+				(path "/eb16378f-e371-46a9-bfab-b0d9404d0362/e5e6ee2e-1d09-4fff-9eef-bc055f220fc3/77a6ec5c-8e09-4a13-82a9-b08f1d53f7e4"
+					(reference "#FLG04")
+					(unit 1)
+				)
+			)
 			(project "12VBuck"
 				(path "/f2a6729b-b8d5-4133-ae64-a5e680928255"
@@
 				)
 			)
+			(project "PS-PowerDistributionUnit"
+				(path "/eb16378f-e371-46a9-bfab-b0d9404d0362/e5e6ee2e-1d09-4fff-9eef-bc055f220fc3/77a6ec5c-8e09-4a13-82a9-b08f1d53f7e4"
+					(reference "#FLG01")
+					(unit 1)
+				)
+			)
 			(project "12VBuck"
 				(path "/f2a6729b-b8d5-4133-ae64-a5e680928255"
@@
 		(in_pos_files yes)
 		(dnp no)
-		(property "Reference" "C4"
+		(property "Reference" "C72"
 			(at 164.084 93.98 0)
 			(show_name no)
@@
 				(path "/0fbc6656-132d-42e4-bdc9-f0a11468b104/973e334b-57f3-4378-b197-420dc86c33e2"
 					(reference "C4")
+					(unit 1)
+				)
+			)
+			(project "PS-PowerDistributionUnit"
+				(path "/eb16378f-e371-46a9-bfab-b0d9404d0362/e5e6ee2e-1d09-4fff-9eef-bc055f220fc3/77a6ec5c-8e09-4a13-82a9-b08f1d53f7e4"
+					(reference "C72")
 					(unit 1)
 				)
@@
 		(in_pos_files yes)
 		(dnp no)
-		(property "Reference" "C6"
+		(property "Reference" "C75"
 			(at 189.992 93.98 0)
 			(show_name no)
@@
 				(path "/0fbc6656-132d-42e4-bdc9-f0a11468b104/973e334b-57f3-4378-b197-420dc86c33e2"
 					(reference "C6")
+					(unit 1)
+				)
+			)
+			(project "PS-PowerDistributionUnit"
+				(path "/eb16378f-e371-46a9-bfab-b0d9404d0362/e5e6ee2e-1d09-4fff-9eef-bc055f220fc3/77a6ec5c-8e09-4a13-82a9-b08f1d53f7e4"
+					(reference "C75")
 					(unit 1)
 				)
@@
 		(in_pos_files yes)
 		(dnp no)
-		(property "Reference" "C3"
+		(property "Reference" "C71"
 			(at 156.718 80.01 0)
 			(show_name no)
@@
 				(path "/ad6c7df0-eb90-4670-9aa8-3e2007aefc2d/41c72b07-cf60-4ca9-96a7-6ae96aaa0c90"
 					(reference "C9")
+					(unit 1)
+				)
+			)
+			(project "PS-PowerDistributionUnit"
+				(path "/eb16378f-e371-46a9-bfab-b0d9404d0362/e5e6ee2e-1d09-4fff-9eef-bc055f220fc3/77a6ec5c-8e09-4a13-82a9-b08f1d53f7e4"
+					(reference "C71")
 					(unit 1)
 				)
@@
 				)
 			)
+			(project "PS-PowerDistributionUnit"
+				(path "/eb16378f-e371-46a9-bfab-b0d9404d0362/e5e6ee2e-1d09-4fff-9eef-bc055f220fc3/77a6ec5c-8e09-4a13-82a9-b08f1d53f7e4"
+					(reference "#FLG03")
+					(unit 1)
+				)
+			)
 			(project "12VBuck"
 				(path "/f2a6729b-b8d5-4133-ae64-a5e680928255"
@@
 		(dnp no)
 		(fields_autoplaced yes)
-		(property "Reference" "R1"
+		(property "Reference" "R87"
 			(at 227.33 85.0899 0)
 			(show_name no)
@@
 				(path "/ad6c7df0-eb90-4670-9aa8-3e2007aefc2d/41c72b07-cf60-4ca9-96a7-6ae96aaa0c90"
 					(reference "R30")
+					(unit 1)
+				)
+			)
+			(project "PS-PowerDistributionUnit"
+				(path "/eb16378f-e371-46a9-bfab-b0d9404d0362/e5e6ee2e-1d09-4fff-9eef-bc055f220fc3/77a6ec5c-8e09-4a13-82a9-b08f1d53f7e4"
+					(reference "R87")
 					(unit 1)
 				)
@@
 		(dnp no)
 		(fields_autoplaced yes)
-		(property "Reference" "C2"
+		(property "Reference" "C70"
 			(at 105.41 87.6362 0)
 			(show_name no)
@@
 				(path "/0fbc6656-132d-42e4-bdc9-f0a11468b104/973e334b-57f3-4378-b197-420dc86c33e2"
 					(reference "C2")
+					(unit 1)
+				)
+			)
+			(project "PS-PowerDistributionUnit"
+				(path "/eb16378f-e371-46a9-bfab-b0d9404d0362/e5e6ee2e-1d09-4fff-9eef-bc055f220fc3/77a6ec5c-8e09-4a13-82a9-b08f1d53f7e4"
+					(reference "C70")
 					(unit 1)
 				)
@@
 		(dnp no)
 		(fields_autoplaced yes)
-		(property "Reference" "R2"
+		(property "Reference" "R88"
 			(at 227.33 92.7099 0)
 			(show_name no)
@@
 				(path "/ad6c7df0-eb90-4670-9aa8-3e2007aefc2d/41c72b07-cf60-4ca9-96a7-6ae96aaa0c90"
 					(reference "R31")
+					(unit 1)
+				)
+			)
+			(project "PS-PowerDistributionUnit"
+				(path "/eb16378f-e371-46a9-bfab-b0d9404d0362/e5e6ee2e-1d09-4fff-9eef-bc055f220fc3/77a6ec5c-8e09-4a13-82a9-b08f1d53f7e4"
+					(reference "R88")
 					(unit 1)
 				)
@@
 		(in_pos_files yes)
 		(dnp no)
-		(property "Reference" "C5"
+		(property "Reference" "C74"
 			(at 173.482 94.234 0)
 			(show_name no)
@@
 					(unit 1)
 				)
+			)
+			(project "PS-PowerDistributionUnit"
+				(path "/eb16378f-e371-46a9-bfab-b0d9404d0362/e5e6ee2e-1d09-4fff-9eef-bc055f220fc3/77a6ec5c-8e09-4a13-82a9-b08f1d53f7e4"
+					(reference "C74")
+					(unit 1)
+				)

Commit message: my baby is in groups
Parts:
- C71: footprint Capacitor_SMD:C_0603_1608Metric -> Capacitor_SMD:C_0603_1608Metric_Pad1.08x0.95mm_HandSolder
Changed lines of the file:
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@@
 			)
 		)
-		(property "Footprint" "Capacitor_SMD:C_0603_1608Metric"
+		(property "Footprint" "Capacitor_SMD:C_0603_1608Metric_Pad1.08x0.95mm_HandSolder"
 			(at 153.67 83.82 0)
 			(hide yes)

Commit message: booooom not done tho
Parts:
- renumbered C74 to C73, C75 to C74
Changed lines of the file:
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@@
 		(in_pos_files yes)
 		(dnp no)
-		(property "Reference" "C75"
+		(property "Reference" "C74"
 			(at 189.992 93.98 0)
 			(show_name no)
@@
 			(project "PS-PowerDistributionUnit"
 				(path "/eb16378f-e371-46a9-bfab-b0d9404d0362/e5e6ee2e-1d09-4fff-9eef-bc055f220fc3/77a6ec5c-8e09-4a13-82a9-b08f1d53f7e4"
-					(reference "C75")
+					(reference "C74")
 					(unit 1)
 				)
@@
 		(in_pos_files yes)
 		(dnp no)
-		(property "Reference" "C74"
+		(property "Reference" "C73"
 			(at 173.482 94.234 0)
 			(show_name no)
@@
 			(project "PS-PowerDistributionUnit"
 				(path "/eb16378f-e371-46a9-bfab-b0d9404d0362/e5e6ee2e-1d09-4fff-9eef-bc055f220fc3/77a6ec5c-8e09-4a13-82a9-b08f1d53f7e4"
-					(reference "C74")
-					(unit 1)
-				)
+					(reference "C73")
+					(unit 1)
+				)

Commit message: added pn
Parts:
- C69: LCSC P/N C6962403 -> C105911; P/N 08055D475KAT4A -> C0805B475K050T
- C70, C71: LCSC P/N C6666325 -> C1591; P/N MLASH168SB7104KTNA01 -> CL10B104KB8NNNC
- C72, C73: LCSC P/N C778721 -> C5448976; P/N GMK325BJ226MM-P -> GGM31CD70J226KE02L
- L1: LCSC P/N (none) -> C1870586
- R87: P/N CRCW0603100KFKEE -> 0603WAF1003T5E
Changed lines of the file:
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@@
 			)
 		)
-		(property "LCSC P/N" "C6962403"
+		(property "LCSC P/N" "C105911"
 			(at 93.98 86.36 0)
 			(hide yes)
@@
 			)
 		)
-		(property "P/N" "08055D475KAT4A"
+		(property "P/N" "C0805B475K050T"
 			(at 93.98 86.36 0)
 			(hide yes)
@@
 			)
 		)
-		(property "LCSC P/N" ""
+		(property "LCSC P/N" "C1870586"
 			(at 161.29 86.36 90)
 			(hide yes)
@@
 			)
 		)
-		(property "P/N" "GMK325BJ226MM-P"
+		(property "P/N" "GGM31CD70J226KE02L"
 			(at 170.18 95.25 0)
 			(hide yes)
@@
 			)
 		)
-		(property "LCSC P/N" "C778721"
+		(property "LCSC P/N" "C5448976"
 			(at 170.18 95.25 0)
 			(hide yes)
@@
 			)
 		)
-		(property "P/N" "MLASH168SB7104KTNA01"
+		(property "P/N" "CL10B104KB8NNNC"
 			(at 153.67 83.82 0)
 			(hide yes)
@@
 			)
 		)
-		(property "LCSC P/N" "C6666325"
+		(property "LCSC P/N" "C1591"
 			(at 153.67 83.82 0)
 			(hide yes)
@@
 			)
 		)
-		(property "P/N" "CRCW0603100KFKEE"
+		(property "P/N" "0603WAF1003T5E"
 			(at 224.79 86.36 0)
 			(hide yes)
@@
 			)
 		)
-		(property "LCSC P/N" "C6666325"
+		(property "LCSC P/N" "C1591"
 			(at 102.87 88.9 0)
 			(hide yes)
@@
 			)
 		)
-		(property "P/N" "MLASH168SB7104KTNA01"
+		(property "P/N" "CL10B104KB8NNNC"
 			(at 102.87 88.9 0)
 			(hide yes)
@@
 			)
 		)
-		(property "P/N" "GMK325BJ226MM-P"
+		(property "P/N" "GGM31CD70J226KE02L"
 			(at 179.07 95.25 0)
 			(hide yes)
@@
 			)
 		)
-		(property "LCSC P/N" "C778721"
+		(property "LCSC P/N" "C5448976"
 			(at 179.07 95.25 0)
 			(hide yes)

Commit message: need to study matrices:
Parts:
- R87, R88: footprint Resistor_SMD:R_0603_1608Metric -> Resistor_SMD:R_0603_1608Metric_Pad0.98x0.95mm_HandSolder
Changed lines of the file:
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@@
 			)
 		)
-		(property "Footprint" "Resistor_SMD:R_0603_1608Metric"
+		(property "Footprint" "Resistor_SMD:R_0603_1608Metric_Pad0.98x0.95mm_HandSolder"
 			(at 224.79 86.36 0)
 			(hide yes)
@@
 			)
 		)
-		(property "Footprint" "Resistor_SMD:R_0603_1608Metric"
+		(property "Footprint" "Resistor_SMD:R_0603_1608Metric_Pad0.98x0.95mm_HandSolder"
 			(at 224.79 93.98 0)
 			(hide yes)
