File: hardware/LDO.kicad_sch (KiCad schematic)
At the start: 5 parts, among them U3 MCP1826S

Commit message: maybe added tvs
Parts:
- renumbered C36 to C1, C37 to C2, D33 to D1, U3 to U1
Changed lines of the file:
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@@
 		(dnp no)
 		(fields_autoplaced yes)
-		(property "Reference" "C37"
+		(property "Reference" "C2"
 			(at 168.275 68.5735 0)
 			(show_name no)
@@
 			(project "PS-PowerDistributionUnit"
 				(path "/eb16378f-e371-46a9-bfab-b0d9404d0362/e5e6ee2e-1d09-4fff-9eef-bc055f220fc3/b3ece65c-a1bc-4529-9ff0-e7f39b9d1f6a"
-					(reference "C37")
+					(reference "C2")
 					(unit 1)
 				)
@@
 		(dnp no)
 		(fields_autoplaced yes)
-		(property "Reference" "U3"
+		(property "Reference" "U1"
 			(at 152.4 56.515 0)
 			(show_name no)
@@
 			(project "PS-PowerDistributionUnit"
 				(path "/eb16378f-e371-46a9-bfab-b0d9404d0362/e5e6ee2e-1d09-4fff-9eef-bc055f220fc3/b3ece65c-a1bc-4529-9ff0-e7f39b9d1f6a"
-					(reference "U3")
+					(reference "U1")
 					(unit 1)
 				)
@@
 		(dnp no)
 		(fields_autoplaced yes)
-		(property "Reference" "D33"
+		(property "Reference" "D1"
 			(at 133.604 57.15 0)
 			(show_name no)
@@
 			(project "PS-PowerDistributionUnit"
 				(path "/eb16378f-e371-46a9-bfab-b0d9404d0362/e5e6ee2e-1d09-4fff-9eef-bc055f220fc3/b3ece65c-a1bc-4529-9ff0-e7f39b9d1f6a"
-					(reference "D33")
+					(reference "D1")
 					(unit 1)
 				)
@@
 		(dnp no)
 		(fields_autoplaced yes)
-		(property "Reference" "C36"
+		(property "Reference" "C1"
 			(at 142.875 68.5735 0)
 			(show_name no)
@@
 			(project "PS-PowerDistributionUnit"
 				(path "/eb16378f-e371-46a9-bfab-b0d9404d0362/e5e6ee2e-1d09-4fff-9eef-bc055f220fc3/b3ece65c-a1bc-4529-9ff0-e7f39b9d1f6a"
-					(reference "C36")
+					(reference "C1")
 					(unit 1)
 				)

Commit message: added p/n and footprints
Parts:
- C1, C2: P/N (none) -> GRM21BR61H106KE43K
Changed lines of the file:
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@@
+			)
+		)
+		(property "P/N" "GRM21BR61H106KE43K"
+			(at 165.1 69.85 0)
+			(hide yes)
+			(show_name no)
+			(do_not_autoplace no)
+			(effects
+				(font
+					(size 1.27 1.27)
+				)
 			)
 		)
@@
 			(at 139.7 69.85 0)
 			(hide yes)
+			(show_name no)
+			(do_not_autoplace no)
+			(effects
+				(font
+					(size 1.27 1.27)
+				)
+			)
+		)
+		(property "P/N" "GRM21BR61H106KE43K"
+			(at 139.7 69.85 0)
+			(hide yes)

Commit message: gerb bom
Parts:
- TP_3.3V1: footprint TestPoint:TestPoint_Loop_D1.80mm_Drill1.0mm_Beaded -> TestPoint:TestPoint_THTPad_D3.0mm_Drill1.5mm
Changed lines of the file:
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@@
 			)
 		)
-		(property "Footprint" "TestPoint:TestPoint_Loop_D1.80mm_Drill1.0mm_Beaded"
+		(property "Footprint" "TestPoint:TestPoint_THTPad_D3.0mm_Drill1.5mm"
 			(at 170.18 63.5 0)
 			(hide yes)
